File: mntcomp-keyboard/mntcomp-keyboard.kicad_pcb (KiCad board)
At the start: 2 copper layers, 275.2 x 114.1 mm, 167 parts, among them J1 Conn_01x02, J2 Conn_01x06, J3 Conn_01x04, SW1 ML, SW10 ML, SW11 ML, SW12 ML, SW13 ML, SW14 ML, SW15 ML, SW16 ML, SW17 ML, SW18 ML, SW19 ML, SW2 ML, SW20 ML, SW21 ML, SW22 ML, SW23 ML, SW24 ML, SW25 ML, SW26 ML, SW27 ML, SW28 ML, SW29 ML, SW3 ML, SW30 ML, SW31 ML, SW32 ML, SW33 ML, SW34 ML, SW35 ML, SW36 ML, SW37 ML, SW38 ML, SW39 ML, SW4 ML, SW40 ML, SW41 ML, SW42 ML, SW43 ML, SW44 ML, SW45 ML, SW46 ML, SW47 ML, SW48 ML, SW49 ML, SW5 ML, SW50 ML, SW51 ML, SW52 ML, SW53 ML, SW54 ML, SW55 ML, SW56 ML, SW57 ML, SW58 ML, SW59 ML, SW6 ML, SW60 ML, SW61 ML, SW62 ML, SW63 ML, SW64 ML, SW65 ML, SW66 ML, SW67 ML, SW68 ML, SW69 ML, SW7 ML, SW70 ML, SW71 ML, SW72 ML, SW73 ML, SW74 ML, SW75 ML, SW76 ML, SW77 ML, SW8 ML, SW9 ML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

Commit message: 0.2 snapshot before starting new battery mgmt
Parts:
- added D78: D_Small, Diodes_SMD:D_1206, B.Cu at (95.2, 137.7)
- added D79: D_Small, Diodes_SMD:D_1206, B.Cu at (189.9, 137.7)
- added D80: LED, LEDs:LED_0805_HandSoldering, F.Cu at (152.4, 131.7)
- added G***: LOGO, mnt:mnt, B.Cu at (156.2, 131.2)
- added G***: LOGO, mnt:reform02, B.Cu at (170.7, 128.9)
- added MH1: Hole, Mounting_Holes:MountingHole_3mm, F.Cu at (85.7, 37.6)
- added MH2: Hole, Mounting_Holes:MountingHole_3mm, F.Cu at (211.6, 37.6)
- added MH3: Hole, Mounting_Holes:MountingHole_3mm, F.Cu at (13.2, 126.8)
- added MH4: Hole, Mounting_Holes:MountingHole_3mm, F.Cu at (284.1, 126.8)
- added MH5: Hole, Mounting_Holes:MountingHole_3mm, F.Cu at (104.1, 142.2)
- added MH6: Hole, Mounting_Holes:MountingHole_3mm, F.Cu at (181.3, 142.2)
- added R4: R_Small, Resistors_SMD:R_0603_HandSoldering, B.Cu at (138.7, 134.2)
- added SH1: Hole, Mounting_Holes:MountingHole_4mm, F.Cu at (164.7, 138.3)
- added SH2: Hole, Mounting_Holes:MountingHole_4mm, F.Cu at (120.7, 138.3)
- added SH3: Hole, Mounting_Holes:MountingHole_4mm, F.Cu at (278.7, 97.1)
- added SH4: Hole, Mounting_Holes:MountingHole_4mm, F.Cu at (278.7, 76.5)
- added SH5: Hole, Mounting_Holes:MountingHole_4mm, F.Cu at (276.1, 66.2)
- added SH6: Hole, Mounting_Holes:MountingHole_4mm, F.Cu at (255.2, 66.2)
- added SH7: Hole, Mounting_Holes:MountingHole_4mm, F.Cu at (21.5, 120.2)
- added SH8: Hole, Mounting_Holes:MountingHole_4mm, F.Cu at (50.0, 120.2)
- added SW78: ML, mntcomp-keyboard:cherry-ml, F.Cu at (92.2, 126.9)
- added SW79: ML, mntcomp-keyboard:cherry-ml, F.Cu at (181.2, 126.9)
- J2: moved to F.Cu
- J3: value Conn_01x04 -> Conn_01x05; footprint Pin_Headers:Pin_Header_Straight_1x04_Pitch2.00mm -> Pin_Headers:Pin_Header_Straight_1x05_Pitch2.00mm
- moved C5 17.0 mm to (115.4, 135.0), turned to 0 degrees
- moved J1 15.1 mm to (108.0, 138.6)
- moved D62 6.60 mm to (141.2, 119.9)
- moved J2 5.27 mm to (108.0, 136.2), turned to 180 degrees
- moved R1 4.40 mm to (130.3, 137.3)
- moved C1 4.40 mm to (114.2, 123.8)
- moved C2 4.40 mm to (114.2, 132.3)
- moved C3 4.40 mm to (126.7, 136.6)
- moved C4 4.40 mm to (125.0, 136.6)
- moved Y1 4.40 mm to (114.0, 128.1)
- moved R2 4.40 mm to (130.3, 135.6)
- moved U1 4.40 mm to (126.5, 127.5)
- moved SW77 1.90 mm to (263.3, 126.9)
- moved SW69 1.76 mm to (263.3, 108.9)
- moved SW68 1.64 mm to (240.3, 108.9)
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Connections:
- J3 pad 4: Net-(J3-Pad4) -> GND
- U1 pad 1: Net-(J3-Pad4) -> Net-(D80-Pad1)
Routing:
- net COL9: track 171.2 -> 298.5 mm, vias 1 -> 2
- net COL10: track 189.2 -> 259.0 mm, vias 1 -> 2
- net Net-(D80-Pad1): track 0.00 -> 29.1 mm
- net RAWVCC: track 47.8 -> 74.5 mm
- net ROW6: track 444.8 -> 420.4 mm, vias 2 -> 4
- net Net-(J3-Pad4): track 16.5 -> 0.00 mm, vias 1 -> 0
- net ROW2: track 496.2 -> 512.5 mm
- net Net-(D80-Pad2): track 0.00 -> 14.3 mm, vias 0 -> 1
- net UVCC: track 28.8 -> 37.4 mm
- net D+: track 24.2 -> 32.4 mm
- net COL6: track 218.7 -> 210.7 mm, vias 1 -> 0
- net COL4: track 143.9 -> 151.9 mm, vias 1 -> 3
- net COL3: track 156.1 -> 162.8 mm
- net COL1: track 206.1 -> 212.1 mm
- net PWRON: track 26.3 -> 32.2 mm
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Other:
- board size 275.2 x 114.1 mm -> 276.9 x 114.8 mm

Commit message: Reform keyboard 0.4 snapshot for manufacturing
Parts:
- removed the G*** at (170.7, 128.9)
- added G***: LOGO, mnt:reform04, B.Cu at (170.7, 128.7)
- added R: V, mnt:VIA-0.4mm, F.Cu at (227.9, 122.3)
- added R: V, mnt:VIA-0.4mm, F.Cu at (213.7, 140.9)
- added R: V, mnt:VIA-0.4mm, F.Cu at (252.7, 140.9)
- added R: V, mnt:VIA-0.4mm, F.Cu at (234.2, 140.9)
- added R: V, mnt:VIA-0.4mm, F.Cu at (193.2, 143.4)
- added R: V, mnt:VIA-0.4mm, F.Cu at (216.2, 143.4)
- added R: V, mnt:VIA-0.4mm, F.Cu at (219.2, 137.4)
- added R: V, mnt:VIA-0.4mm, F.Cu at (199.2, 137.4)
- added R: V, mnt:VIA-0.4mm, F.Cu at (199.2, 131.4)
- added R: V, mnt:VIA-0.4mm, F.Cu at (169.2, 131.4)
- added R: V, mnt:VIA-0.4mm, F.Cu at (174.2, 137.4)
- added R: V, mnt:VIA-0.4mm, F.Cu at (214.5, 122.6)
- added R: V, mnt:VIA-0.4mm, F.Cu at (156.2, 137.4)
- added R: V, mnt:VIA-0.4mm, F.Cu at (257.2, 114.4)
- added R: V, mnt:VIA-0.4mm, F.Cu at (258.2, 132.4)
- added R: V, mnt:VIA-0.4mm, F.Cu at (279.2, 140.4)
- added R: V, mnt:VIA-0.4mm, F.Cu at (272.2, 106.4)
- added R: V, mnt:VIA-0.4mm, F.Cu at (262.2, 76.4)
- added R: V, mnt:VIA-0.4mm, F.Cu at (243.2, 88.4)
- added R: V, mnt:VIA-0.4mm, F.Cu at (226.2, 88.4)
- added R: V, mnt:VIA-0.4mm, F.Cu at (15.2, 69.4)
- added R: V, mnt:VIA-0.4mm, F.Cu at (17.2, 110.4)
- added R: V, mnt:VIA-0.4mm, F.Cu at (219.9, 122.6)
- added R: V, mnt:VIA-0.4mm, F.Cu at (20.2, 100.4)
- added R: V, mnt:VIA-0.4mm, F.Cu at (17.2, 88.4)
- added R: V, mnt:VIA-0.4mm, F.Cu at (42.2, 88.4)
- added R: V, mnt:VIA-0.4mm, F.Cu at (62.2, 88.4)
- added R: V, mnt:VIA-0.4mm, F.Cu at (77.2, 88.4)
- added R: V, mnt:VIA-0.4mm, F.Cu at (99.2, 88.4)
- added R: V, mnt:VIA-0.4mm, F.Cu at (118.2, 88.4)
- added R: V, mnt:VIA-0.4mm, F.Cu at (135.2, 88.4)
- added R: V, mnt:VIA-0.4mm, F.Cu at (153.2, 88.4)
- added R: V, mnt:VIA-0.4mm, F.Cu at (173.2, 88.4)
- added R: V, mnt:VIA-0.4mm, F.Cu at (200.8, 122.1)
- added R: V, mnt:VIA-0.4mm, F.Cu at (190.2, 88.4)
- added R: V, mnt:VIA-0.4mm, F.Cu at (111.2, 133.4)
- added R: V, mnt:VIA-0.4mm, F.Cu at (137.2, 138.4)
- added R: V, mnt:VIA-0.4mm, F.Cu at (201.2, 88.4)
- added R: V, mnt:VIA-0.4mm, F.Cu at (232.2, 117.4)
- added R: V, mnt:VIA-0.4mm, F.Cu at (214.7, 117.4)
- added R: V, mnt:VIA-0.4mm, F.Cu at (218.7, 111.9)
- added R: V, mnt:VIA-0.4mm, F.Cu at (221.2, 106.4)
- added R: V, mnt:VIA-0.4mm, F.Cu at (208.2, 94.9)
- added R: V, mnt:VIA-0.4mm, F.Cu at (208.2, 98.9)
- added R: V, mnt:VIA-0.4mm, F.Cu at (68.2, 142.9)
- added R: V, mnt:VIA-0.4mm, F.Cu at (212.2, 105.4)
- added R: V, mnt:VIA-0.4mm, F.Cu at (89.7, 140.9)
- added R: V, mnt:VIA-0.4mm, F.Cu at (113.7, 142.9)
- added R: V, mnt:VIA-0.4mm, F.Cu at (160.7, 143.4)
- added R: V, mnt:VIA-0.4mm, F.Cu at (197.0, 140.2)
Routing:
- net RAWVCC: track 74.5 -> 73.7 mm
- net RESET: track 21.1 -> 20.4 mm
- net ROW1: track 511.8 -> 512.4 mm
