File: electronics/reform-audio.sch (KiCad schematic (older format))
At the start: 16 parts, among them J16 Conn_LineIn, J17 Conn_LineOut, J18 SJ-43516-SMT, U10 SGTL5000XNAA3

Commit message: KiCad 4 to KiCad 5 conversion
Parts:
- C55, C56, C57, C58, C59, C60, C61, C62, C63, C64, C65: symbol C_Small -> reform-motherboard-rescue:C_Small
- J16, J17: symbol Conn_01x03 -> reform-motherboard-rescue:Conn_01x03
- J18: symbol SJ-43516-SMT -> reform-motherboard-rescue:SJ-43516-SMT
- R31: symbol R_Small -> reform-motherboard-rescue:R_Small
- U10: symbol SGTL5000XNAA3 -> reform-motherboard-rescue:SGTL5000XNAA3
Changed lines of the file:
@@
-EESchema Schematic File Version 2
-LIBS:power
-LIBS:device
-LIBS:switches
-LIBS:relays
-LIBS:motors
-LIBS:transistors
-LIBS:conn
-LIBS:linear
-LIBS:regul
-LIBS:74xx
-LIBS:cmos4000
-LIBS:adc-dac
-LIBS:memory
-LIBS:xilinx
-LIBS:microcontrollers
-LIBS:dsp
-LIBS:microchip
-LIBS:analog_switches
-LIBS:motorola
-LIBS:texas
-LIBS:intel
-LIBS:audio
-LIBS:interface
-LIBS:digital-audio
-LIBS:philips
-LIBS:display
-LIBS:cypress
-LIBS:siliconi
-LIBS:opto
-LIBS:atmel
-LIBS:contrib
-LIBS:valves
-LIBS:J0G-0003NL
-LIBS:TUSB4041IPAPR
-LIBS:TPS61235RWLR
-LIBS:AP1501A-33K5G-13
-LIBS:TPS74801DRCR
-LIBS:MCP73123T-22SI_MF
-LIBS:SGTL5000XNAA3
-LIBS:CM2020-00TR
-LIBS:INA260AIPW
-LIBS:SN74LVC1G14DBVR
-LIBS:SN74LVC1G08DCKR
-LIBS:693072010801
-LIBS:48099-5701
-LIBS:67910-5700
-LIBS:DF40C-100DS-0.4V_51_
-LIBS:5622-4100-ML
-LIBS:TUSB2046BVFR
-LIBS:TPS2044BDR
-LIBS:LP3962EMP-2.5
-LIBS:BQ24650RVAT
-LIBS:SJ-43516-SMT
+EESchema Schematic File Version 4
 LIBS:reform-motherboard-cache
-EELAYER 25 0
+EELAYER 26 0
 EELAYER END
 $Descr A4 11693 8268
@@
 $EndDescr
 $Comp
-L SGTL5000XNAA3 U10
+L reform-motherboard-rescue:SGTL5000XNAA3 U10
 U 1 1 5A11FBBE
 P 5400 3550
@@
 	7950 1950 7950 5800
 $Comp
-L GND #PWR0224
+L reform-motherboard-rescue:GND #PWR0224
 U 1 1 5A120C9E
 P 6300 5400
@@
 I2C3_SCL
 $Comp
-L GND #PWR0225
+L reform-motherboard-rescue:GND #PWR0225
 U 1 1 5A122337
 P 4050 4850
@@
 	4500 5800 7950 5800
 $Comp
-L C_Small C64
+L reform-motherboard-rescue:C_Small C64
 U 1 1 5A122A76
 P 6500 2950
@@
 $EndComp
 $Comp
-L C_Small C65
+L reform-motherboard-rescue:C_Small C65
 U 1 1 5A122B49
 P 6750 3050
@@
 	6950 3050 6850 3050
 $Comp
-L C_Small C62
+L reform-motherboard-rescue:C_Small C62
 U 1 1 5A122C86
 P 4300 2950
@@
 $EndComp
 $Comp
-L C_Small C60
+L reform-motherboard-rescue:C_Small C60
 U 1 1 5A122CF9
 P 3950 3050
@@
 	3300 3450 4500 3450
 $Comp
-L GND #PWR0226
+L reform-motherboard-rescue:GND #PWR0226
 U 1 1 5A1234F8
 P 3300 3650
@@
 Connection ~ 6300 5250
 $Comp
-L C_Small C55
+L reform-motherboard-rescue:C_Small C55
 U 1 1 5A124351
 P 2550 3550
@@
 $EndComp
 $Comp
-L GND #PWR0227
+L reform-motherboard-rescue:GND #PWR0227
 U 1 1 5A124399
 P 2550 3650
@@
 	2550 2650 2550 3450
 $Comp
-L R_Small R31
+L reform-motherboard-rescue:R_Small R31
 U 1 1 5A124AE8
 P 2950 3250
@@
 $EndComp
 $Comp
-L C_Small C57
+L reform-motherboard-rescue:C_Small C57
 U 1 1 5A124B94
 P 3200 2950
@@
 Connection ~ 3200 2550
 $Comp
-L C_Small C56
+L reform-motherboard-rescue:C_Small C56
 U 1 1 5A1269AF
 P 2950 3550
@@
 	2950 3450 2950 3350
 $Comp
-L GND #PWR0228
+L reform-motherboard-rescue:GND #PWR0228
 U 1 1 5A126A30
 P 2950 3650
@@
 $EndComp
 $Comp
-L C_Small C63
+L reform-motherboard-rescue:C_Small C63
 U 1 1 5A127261
 P 6400 2150
@@
 	6400 1950 6400 2050
 $Comp
-L C_Small C59
+L reform-motherboard-rescue:C_Small C59
 U 1 1 5A127330
 P 3750 2000
@@
 $EndComp
 $Comp
-L C_Small C61
+L reform-motherboard-rescue:C_Small C61
 U 1 1 5A1273F1
 P 4050 2250
@@
 	4350 2550 4500 2550
 $Comp
-L GND #PWR0229
+L reform-motherboard-rescue:GND #PWR0229
 U 1 1 5A1274D7
 P 4050 2350
@@
 $EndComp
 $Comp
-L GND #PWR0230
+L reform-motherboard-rescue:GND #PWR0230
 U 1 1 5A127512
 P 3750 2100
@@
 Connection ~ 4200 1900
 $Comp
-L +3V3 #PWR0231
+L reform-motherboard-rescue:+3V3 #PWR0231
 U 1 1 5A1282F7
 P 6400 1950
@@
 $EndComp
 $Comp
-L GND #PWR0232
+L reform-motherboard-rescue:GND #PWR0232
 U 1 1 5A1289F2
 P 6400 2250
@@
 $EndComp
 $Comp
-L Conn_01x03 J16
+L reform-motherboard-rescue:Conn_01x03 J16
 U 1 1 5A180365
 P 3550 2950
@@
 	4500 2650 4500 2750
 $Comp
-L Conn_01x03 J17
+L reform-motherboard-rescue:Conn_01x03 J17
 U 1 1 5A18063F
 P 7250 2950
@@
 	6950 2850 7050 2850
 $Comp
-L GND #PWR0233
+L reform-motherboard-rescue:GND #PWR0233
 U 1 1 5A1809B9
 P 7000 3450
@@
 	7000 3050 7050 3050
 $Comp
-L GND #PWR0234
+L reform-motherboard-rescue:GND #PWR0234
 U 1 1 5A180B77
 P 3800 3650
@@
 	3800 2850 3750 2850
 $Comp
-L +1V5 #PWR0235
+L reform-motherboard-rescue:+1V5 #PWR0235
 U 1 1 5A1DA4BE
 P 4200 1900
@@
 $EndComp
 $Comp
-L +3V3 #PWR0236
+L reform-motherboard-rescue:+3V3 #PWR0236
 U 1 1 5A4E2A64
 P 4200 2150
@@
 $EndComp
 $Comp
-L C_Small C58
+L reform-motherboard-rescue:C_Small C58
 U 1 1 5A123466
 P 3300 3550
@@
 I2C Addr: 0001010
 $Comp
-L SJ-43516-SMT J18
+L reform-motherboard-rescue:SJ-43516-SMT J18
 U 1 1 5B151703
 P 7350 2050
