File: electronics/reform-eth-usb.sch (KiCad schematic (older format))
At the start: 53 parts, among them J12 USB_INT_3, J5 USB_A, J7 USB_A, J9 USB_INT_1, P2 J0G-0003NL, U15 TPS2044BDR, U9 TUSB4041IPAPR, Y1 24MHz

Commit message: KiCad 4 to KiCad 5 conversion
Parts:
- C13, C14, C15, C16, C17, C40, C41, C45, C46, C47, C48, C49, C50, C51, C52, C53, C54, C75, C83, C84, C85, C86, C87: symbol C_Small -> reform-motherboard-rescue:C_Small
- J12, J9: symbol Conn_01x04 -> reform-motherboard-rescue:Conn_01x04
- J5, J7: symbol USB_A -> reform-motherboard-rescue:USB_A
- L4, L5: symbol Ferrite_Bead_Small -> reform-motherboard-rescue:Ferrite_Bead_Small
- P2: symbol J0G-0003NL -> reform-motherboard-rescue:J0G-0003NL
- R18, R19, R20, R21, R22, R23, R24, R25, R26, R27, R28, R30, R33, R34, R35, R43, R44, R45, R46, R49: symbol R_Small -> reform-motherboard-rescue:R_Small
- U15: symbol TPS2044BDR -> reform-motherboard-rescue:TPS2044BDR
- U9: symbol TUSB4041IPAPR -> reform-motherboard-rescue:TUSB4041IPAPR
- Y1: symbol Crystal_Small -> reform-motherboard-rescue:Crystal_Small
