File: electronics/reform-motherboard.sch (KiCad schematic (older format))
At the start: 19 parts, among them J1 TinyRex-J1-DF40C, J10 TEST_PMIC_ON, J11 TEST_ON, J2 TinyRex-J2-DF40C, J20 Conn_GPIO1, J21 Conn_SPI2, J3 TinyRex-J3-DF40C, J35 Conn_SPI1, J8 TEST_BM0

Commit message: KiCad 4 to KiCad 5 conversion
Parts:
- C11, C12: symbol C_Small -> reform-motherboard-rescue:C_Small
- J1: symbol TinyRex-J1-DF40C -> reform-motherboard-rescue:TinyRex-J1-DF40C
- J10, J11, J8: symbol TEST_1P -> reform-motherboard-rescue:TEST_1P
- J2: symbol TinyRex-J2-DF40C -> reform-motherboard-rescue:TinyRex-J2-DF40C
- J20: symbol Conn_01x04 -> reform-motherboard-rescue:Conn_01x04
- J21, J35: symbol Conn_01x06 -> reform-motherboard-rescue:Conn_01x06
- J3: symbol TinyRex-J3-DF40C -> reform-motherboard-rescue:TinyRex-J3-DF40C
- MH1, MH2, MH3, MH4, MH5, MH6, TP13: symbol TEST -> reform-motherboard-rescue:TEST
- R6: symbol R_Small -> reform-motherboard-rescue:R_Small
