File: electronics/reform-pcie.sch (KiCad schematic (older format))
At the start: 33 parts, among them J27 48099-5701, J31 48099-5701, J32 SIM_Card, J36 Conn_WWAN_AUX, U1 mPCIE 2.0, U8 WWAN USB2.0

Commit message: KiCad 4 to KiCad 5 conversion
Parts:
- C10, C30, C4, C5, C6, C7, C76, C77, C78, C79, C8, C80, C81, C82, C9: symbol C_Small -> reform-motherboard-rescue:C_Small
- C31, C32: symbol CP1_Small -> reform-motherboard-rescue:CP1_Small
- D10, D9: symbol LED_Small -> reform-motherboard-rescue:LED_Small
- J27, J31: symbol 48099-5701 -> reform-motherboard-rescue:48099-5701
- J32: symbol SIM_Card -> reform-motherboard-rescue:SIM_Card
- J36: symbol Conn_01x06 -> reform-motherboard-rescue:Conn_01x06
- R11, R13, R14, R15, R16, R17: symbol R_Small -> reform-motherboard-rescue:R_Small
- TP17, TP7: symbol TEST -> reform-motherboard-rescue:TEST
- U1, U8: symbol MPCIE-Socket -> reform-motherboard-rescue:MPCIE-Socket
