File: electronics/reform-power.sch (KiCad schematic (older format))
At the start: 78 parts, among them J15 Conn_FAN, J22 Conn_PWR, J33 BAT, J34 Conn_ATTINY, J6 Barrel_Jack, Q2 Si2333DDS, Q3 Si7288DP, Q5 Si2333DDS, U11 LP3962EMP-2.5, U13 TLV1117-15, U16 ATTINY841-SSU, U2 BQ24650RVAT, U3 TPS61235RWLR, U4 AP1501A-33K5G-13, U5 TLV74311PDBVR, U6 INA260AIPW

Commit message: KiCad 4 to KiCad 5 conversion
Parts:
- C18, C19, C2, C20, C24, C25, C26, C28, C29, C33, C34, C35, C36, C37, C38, C39, C42, C43, C44, C92, C94: symbol C_Small -> reform-motherboard-rescue:C_Small
- C21, C22, C23: symbol CP1_Small -> reform-motherboard-rescue:CP1_Small
- C27, C3: symbol C -> reform-motherboard-rescue:C
- D11, D3, D7: symbol LED_Small -> reform-motherboard-rescue:LED_Small
- D2, D4, D8: symbol D_Schottky -> reform-motherboard-rescue:D_Schottky
- D5: symbol D_Schottky_Small -> reform-motherboard-rescue:D_Schottky_Small
- J15: symbol Conn_01x03 -> reform-motherboard-rescue:Conn_01x03
- J22, J33: symbol Conn_01x04 -> reform-motherboard-rescue:Conn_01x04
- J34: symbol Conn_01x08 -> reform-motherboard-rescue:Conn_01x08
- J6: symbol Barrel_Jack -> reform-motherboard-rescue:Barrel_Jack
- L1, L2, L3: symbol L -> reform-motherboard-rescue:L
- Q2, Q5: symbol TP0610T -> reform-motherboard-rescue:TP0610T
- Q3: symbol FDS6898A -> reform-motherboard-rescue:FDS6898A
- R1, R10, R2, R29, R3, R4, R41, R42, R47, R48, R5, R50, R51, R52, R53, R54, R55, R7, R8, R9: symbol R_Small -> reform-motherboard-rescue:R_Small
- TP12, TP18, TP2, TP3, TP5, TP6: symbol TEST -> reform-motherboard-rescue:TEST
- U11: symbol LP3962EMP-2.5 -> reform-motherboard-rescue:LP3962EMP-2.5
- U13: symbol TLV1117-15 -> reform-motherboard-rescue:TLV1117-15
- U16: symbol ATTINY841-SSU -> reform-motherboard-rescue:ATTINY841-SSU
- U2: symbol BQ24650RVAT -> reform-motherboard-rescue:BQ24650RVAT
- U3: symbol TPS61235RWLR -> reform-motherboard-rescue:TPS61235RWLR
- U4: symbol AP1501A-33K5G-13 -> reform-motherboard-rescue:AP1501A-33K5G-13
- U5: symbol TLV70012_SOT23-5 -> reform-motherboard-rescue:TLV70012_SOT23-5
- U6: symbol INA260AIPW -> reform-motherboard-rescue:INA260AIPW
