File: electronics/reform-sata-sd.sch (KiCad schematic (older format))
At the start: 17 parts, among them J23 Conn_RESET, J24 Conn_01x04, J25 Conn_CONSOLE, J28 Conn_SDWP, J29 Conn_5V, J30 48099-5701, J38 Conn_SD1, J4 693072010801, Q1 2N7002, U12 SN74LVC1G08DCKR, U7 mSATA II

Commit message: KiCad 4 to KiCad 5 conversion
Parts:
- C1, C66, C74: symbol C_Small -> reform-motherboard-rescue:C_Small
- J23, J28, J29: symbol Conn_01x02 -> reform-motherboard-rescue:Conn_01x02
- J24: symbol Conn_01x04 -> reform-motherboard-rescue:Conn_01x04
- J25: symbol Conn_01x06 -> reform-motherboard-rescue:Conn_01x06
- J30: symbol 48099-5701 -> reform-motherboard-rescue:48099-5701
- J38: symbol Conn_02x04_Odd_Even -> reform-motherboard-rescue:Conn_02x04_Odd_Even
- J4: symbol 693072010801 -> reform-motherboard-rescue:693072010801
- Q1: symbol 2N7002 -> reform-motherboard-rescue:2N7002
- R12, R32: symbol R_Small -> reform-motherboard-rescue:R_Small
- TP1: symbol TEST -> reform-motherboard-rescue:TEST
- U12: symbol SN74LVC1G08DCKR -> reform-motherboard-rescue:SN74LVC1G08DCKR
- U7: symbol MPCIE-Socket -> reform-motherboard-rescue:MPCIE-Socket
Changed lines of the file:
@@
-EESchema Schematic File Version 2
-LIBS:power
-LIBS:device
-LIBS:switches
-LIBS:relays
-LIBS:motors
-LIBS:transistors
-LIBS:conn
-LIBS:linear
-LIBS:regul
-LIBS:74xx
-LIBS:cmos4000
-LIBS:adc-dac
-LIBS:memory
-LIBS:xilinx
-LIBS:microcontrollers
-LIBS:dsp
-LIBS:microchip
-LIBS:analog_switches
-LIBS:motorola
-LIBS:texas
-LIBS:intel
-LIBS:audio
-LIBS:interface
-LIBS:digital-audio
-LIBS:philips
-LIBS:display
-LIBS:cypress
-LIBS:siliconi
-LIBS:opto
-LIBS:atmel
-LIBS:contrib
-LIBS:valves
-LIBS:J0G-0003NL
-LIBS:TUSB4041IPAPR
-LIBS:TPS61235RWLR
-LIBS:AP1501A-33K5G-13
-LIBS:TPS74801DRCR
-LIBS:MCP73123T-22SI_MF
-LIBS:SGTL5000XNAA3
-LIBS:CM2020-00TR
-LIBS:INA260AIPW
-LIBS:SN74LVC1G14DBVR
-LIBS:SN74LVC1G08DCKR
-LIBS:693072010801
-LIBS:48099-5701
-LIBS:67910-5700
-LIBS:DF40C-100DS-0.4V_51_
-LIBS:5622-4100-ML
-LIBS:TUSB2046BVFR
-LIBS:TPS2044BDR
-LIBS:LP3962EMP-2.5
-LIBS:BQ24650RVAT
-LIBS:SJ-43516-SMT
+EESchema Schematic File Version 4
 LIBS:reform-motherboard-cache
-EELAYER 25 0
+EELAYER 26 0
 EELAYER END
 $Descr A4 11693 8268
@@
 SD3_CLK
 $Comp
-L GND #PWR0108
+L reform-motherboard-rescue:GND #PWR0108
 U 1 1 59F3C8F9
 P 1500 3600
@@
 $EndComp
 $Comp
-L GND #PWR0109
+L reform-motherboard-rescue:GND #PWR0109
 U 1 1 59F3CBCC
 P 3850 3050
@@
 $EndComp
 $Comp
-L +3V3 #PWR0110
+L reform-motherboard-rescue:+3V3 #PWR0110
 U 1 1 59F3CDDC
 P 1650 1750
@@
 $EndComp
 $Comp
-L C_Small C1
+L reform-motherboard-rescue:C_Small C1
 U 1 1 59F3CE15
 P 1650 1950
@@
 $EndComp
 $Comp
-L GND #PWR0111
+L reform-motherboard-rescue:GND #PWR0111
 U 1 1 59F3CE96
 P 1650 2300
@@
 	1650 1750 1650 1850
 $Comp
-L 2N7002 Q1
+L reform-motherboard-rescue:2N7002 Q1
 U 1 1 5A116186
 P 3100 3600
@@
 $EndComp
 $Comp
-L GND #PWR0112
+L reform-motherboard-rescue:GND #PWR0112
 U 1 1 5A116311
 P 3200 3800
@@
 	2900 2350 2900 3600
 $Comp
-L +3V3 #PWR0113
+L reform-motherboard-rescue:+3V3 #PWR0113
 U 1 1 5A1163C1
 P 2500 3300
@@
 $EndComp
 $Comp
-L R_Small R12
+L reform-motherboard-rescue:R_Small R12
 U 1 1 5A1163DF
 P 2500 3400
@@
 	2500 3600 2500 3500
 $Comp
-L Conn_01x06 J25
+L reform-motherboard-rescue:Conn_01x06 J25
 U 1 1 5A16C8DA
 P 2400 4900
@@
 UART1_CTS
 $Comp
-L GND #PWR0114
+L reform-motherboard-rescue:GND #PWR0114
 U 1 1 5A16C9D1
 P 2000 5200
@@
 I2C2_SDA
 $Comp
-L Conn_01x04 J24
+L reform-motherboard-rescue:Conn_01x04 J24
 U 1 1 5A16DC69
 P 3850 4900
@@
 $EndComp
 $Comp
-L GND #PWR0115
+L reform-motherboard-rescue:GND #PWR0115
 U 1 1 5A16DCEF
 P 3400 5100
@@
 	3400 4800 3650 4800
 $Comp
-L +3V3 #PWR0116
+L reform-motherboard-rescue:+3V3 #PWR0116
 U 1 1 5A16E57E
 P 3400 4800
@@
 $EndComp
 $Comp
-L +5V #PWR0117
+L reform-motherboard-rescue:+5V #PWR0117
 U 1 1 5A16EE82
 P 2000 4700
@@
 	2000 5100 2200 5100
 $Comp
-L SN74LVC1G08DCKR U12
+L reform-motherboard-rescue:SN74LVC1G08DCKR U12
 U 1 1 5A17082C
 P 2150 6700
@@
 $EndComp
 $Comp
-L +3V3 #PWR0118
+L reform-motherboard-rescue:+3V3 #PWR0118
 U 1 1 5A171278
 P 1500 6350
@@
 Connection ~ 1550 6700
 $Comp
-L GND #PWR0119
+L reform-motherboard-rescue:GND #PWR0119
 U 1 1 5A1713E3
 P 1500 6950
@@
 RESETn
 $Comp
-L Conn_01x02 J23
+L reform-motherboard-rescue:Conn_01x02 J23
 U 1 1 5A172819
 P 3500 6750
@@
 $EndComp
 $Comp
-L GND #PWR0120
+L reform-motherboard-rescue:GND #PWR0120
 U 1 1 5A1728B5
 P 3750 6950
@@
 RSTINn
 $Comp
-L +3V3 #PWR0121
+L reform-motherboard-rescue:+3V3 #PWR0121
 U 1 1 5A173249
 P 3950 6350
@@
 $EndComp
 $Comp
-L R_Small R32
+L reform-motherboard-rescue:R_Small R32
 U 1 1 5A173270
 P 3950 6500
@@
 Console
 $Comp
-L 693072010801 J4
+L reform-motherboard-rescue:693072010801 J4
 U 1 1 5A18AFBB
 P 3050 1450
@@
 Boot SD Card
 $Comp
-L Conn_01x02 J28
+L reform-motherboard-rescue:Conn_01x02 J28
 U 1 1 5A61FA0C
 P 1300 3600
@@
 SD Write Protect
 $Comp
-L Conn_01x02 J29
+L reform-motherboard-rescue:Conn_01x02 J29
 U 1 1 5A621B49
 P 5600 4850
@@
 $EndComp
 $Comp
-L +5V #PWR0122
+L reform-motherboard-rescue:+5V #PWR0122
 U 1 1 5A621CBC
 P 5200 4850
@@
 $EndComp
 $Comp
-L GND #PWR0123
+L reform-motherboard-rescue:GND #PWR0123
 U 1 1 5A621D48
 P 5200 4950
@@
 $EndComp
 $Comp
-L MPCIE-Socket U7
+L reform-motherboard-rescue:MPCIE-Socket U7
 U 1 1 5AD63344
 P 8550 2300
@@
 mSATA II
 $Comp
-L GND #PWR0124
+L reform-motherboard-rescue:GND #PWR0124
 U 1 1 5AD84AD7
 P 7250 3900
@@
 Connection ~ 7250 1950
 $Comp
-L GND #PWR0125
+L reform-motherboard-rescue:GND #PWR0125
 U 1 1 5AD84DC9
 P 9450 3900
@@
 Connection ~ 9450 1750
 $Comp
-L +3V3 #PWR0126
+L reform-motherboard-rescue:+3V3 #PWR0126
 U 1 1 5AD84FB0
 P 10300 1050
@@
 Connection ~ 10300 2550
 $Comp
-L +3V3 #PWR0127
+L reform-motherboard-rescue:+3V3 #PWR0127
 U 1 1 5AD8519E
 P 7100 1100
@@
 Connection ~ 7100 1650
 $Comp
-L C_Small C74
+L reform-motherboard-rescue:C_Small C74
 U 1 1 5AD89617
 P 10050 1300
@@
 $EndComp
 $Comp
-L GND #PWR0128
+L reform-motherboard-rescue:GND #PWR0128
 U 1 1 5AD8961E
 P 10050 1450
@@
 	10050 1450 10050 1400
 $Comp
-L C_Small C66
+L reform-motherboard-rescue:C_Small C66
 U 1 1 5AD89625
 P 9750 1300
@@
 $EndComp
 $Comp
-L GND #PWR0129
+L reform-motherboard-rescue:GND #PWR0129
 U 1 1 5AD8962C
 P 9750 1450
@@
 Connection ~ 9750 1150
 $Comp
-L 48099-5701 J30
+L reform-motherboard-rescue:48099-5701 J30
 U 1 1 5ADB383A
 P 8550 4950
@@
 mSATA Latch
 $Comp
-L GND #PWR0130
+L reform-motherboard-rescue:GND #PWR0130
 U 1 1 5ADB3842
 P 8250 5250
@@
 $EndComp
 $Comp
-L GND #PWR0131
+L reform-motherboard-rescue:GND #PWR0131
 U 1 1 5ADB3848
 P 8850 5250
@@
 NC
 $Comp
-L TEST TP1
+L reform-motherboard-rescue:TEST TP1
 U 1 1 5ADF82E0
 P 7550 1250
@@
 SD1_CMD
 $Comp
-L GND #PWR0132
+L reform-motherboard-rescue:GND #PWR0132
 U 1 1 5B15CE5E
 P 6400 2400
@@
 SD1_CLK
 $Comp
-L +3V3 #PWR0133
+L reform-motherboard-rescue:+3V3 #PWR0133
 U 1 1 5B15D0D0
 P 4850 2400
@@
 Additional SD Card
 $Comp
-L Conn_02x04_Odd_Even J38
+L reform-motherboard-rescue:Conn_02x04_Odd_Even J38
 U 1 1 5B16F224
 P 5550 2500
