File: reform-keyboard-pcb/mntcomp-keyboard.sch (KiCad schematic (older format))
At the start: 166 parts, among them SW1 ML, SW10 ML, SW11 ML, SW12 ML, SW13 ML, SW14 ML, SW15 ML, SW16 ML, SW17 ML, SW18 ML, SW19 ML, SW2 ML, SW20 ML, SW21 ML, SW22 ML, SW23 ML, SW24 ML, SW25 ML, SW26 ML, SW27 ML, SW28 ML, SW29 ML, SW3 ML, SW30 ML, SW31 ML, SW32 ML, SW33 ML, SW34 ML, SW35 ML, SW36 ML, SW37 ML, SW38 ML, SW39 ML, SW4 ML, SW40 ML, SW41 ML, SW42 ML, SW43 ML, SW44 ML, SW45 ML, SW46 ML, SW47 ML, SW48 ML, SW49 ML, SW5 ML, SW50 ML, SW51 ML, SW52 ML, SW53 ML, SW54 ML, SW55 ML, SW56 ML, SW57 ML, SW58 ML, SW59 ML, SW6 ML, SW60 ML, SW61 ML, SW62 ML, SW63 ML, SW64 ML, SW65 ML, SW66 ML, SW67 ML, SW68 ML, SW69 ML, SW7 ML, SW70 ML, SW71 ML, SW72 ML, SW73 ML, SW74 ML, SW75 ML, SW76 ML, SW77 ML, SW78 ML, SW79 ML, SW8 ML, SW9 ML

Commit message: more keyboard sources
Connections:
- wire segments 138 -> 275

Commit message: keyboard pcb: updated with small cleanups to KiCAD 5.x
Parts:
- D1, D10, D11, D12, D13, D14, D15, D16, D17, D18, D19, D2, D20, D21, D22, D23, D24, D25, D26, D27, D28, D29, D3, D30, D31, D32, D33, D34, D35, D36, D37, D38, D39, D4, D40, D41, D42, D43, D44, D45, D46, D47, D48, D49, D5, D50, D51, D52, D53, D54, D55, D56, D57, D58, D59, D6, D60, D61, D62, D63, D64, D65, D66, D67, D68, D69, D7, D70, D71, D72, D73, D74, D75, D76, D77, D78, D79, D8, D9: symbol D_Small -> Device:D_Small
- SH1, SH2, SH3, SH4, SH5, SH6, SH7, SH8: symbol TEST -> Mechanical:MountingHole
- SW1, SW10, SW11, SW12, SW13, SW14, SW15, SW16, SW17, SW18, SW19, SW2, SW20, SW21, SW22, SW23, SW24, SW25, SW26, SW27, SW28, SW29, SW3, SW30, SW31, SW32, SW33, SW34, SW35, SW36, SW37, SW38, SW39, SW4, SW40, SW41, SW42, SW43, SW44, SW45, SW46, SW47, SW48, SW49, SW5, SW50, SW51, SW52, SW53, SW54, SW55, SW56, SW57, SW58, SW59, SW6, SW60, SW61, SW62, SW63, SW64, SW65, SW66, SW67, SW68, SW69, SW7, SW70, SW71, SW72, SW73, SW74, SW75, SW76, SW77, SW78, SW79, SW8, SW9: symbol ML -> mntcomp-keyboard:ML
Connections:
- wire segments 275 -> 202
