File: reform-keyboard-pcb/reform-kbd-mcu.sch (KiCad schematic (older format))
At the start: 21 parts, among them J1 Conn_01x02, J2 Conn_01x06, J3 Conn_01x05, U1 ATMEGA32U4-AU, Y1 16MHz

Commit message: more keyboard sources
Parts:
- C1, C2: value 10pF -> 18pF
- R1, R2: value 22 -> 0
Changed lines of the file:
@@
-EESchema Schematic File Version 2
+EESchema Schematic File Version 4
 LIBS:power
 LIBS:device
@@
 LIBS:mntcomp-keyboard
 LIBS:mntcomp-keyboard-cache
-EELAYER 25 0
+EELAYER 26 0
 EELAYER END
 $Descr A4 11693 8268
 encoding utf-8
 Sheet 2 2
-Title ""
-Date ""
-Rev ""
-Comp ""
-Comment1 ""
-Comment2 ""
-Comment3 ""
+Title "Reform Keyboard"
+Date "2018-11-11"
+Rev "0.4"
+Comp "MNT Media and Technology UG"
+Comment1 "License: GPLv3+ https://www.gnu.org/licenses/gpl-3.0.en.html"
+Comment2 "Copyright 2017,2018 Lukas F. Hartmann / mntmn"
+Comment3 "https://mntmn.com/reform"
 Comment4 ""
 $EndDescr
@@
 P 2700 3600
 F 0 "C1" H 2710 3670 50  0000 L CNN
-F 1 "10pF" H 2710 3520 50  0000 L CNN
+F 1 "18pF" H 2710 3520 50  0000 L CNN
 F 2 "Capacitors_SMD:C_0603_HandSoldering" H 2700 3600 50  0001 C CNN
 F 3 "" H 2700 3600 50  0001 C CNN
@@
 P 3300 3600
 F 0 "C2" H 3310 3670 50  0000 L CNN
-F 1 "10pF" H 3310 3520 50  0000 L CNN
+F 1 "18pF" H 3310 3520 50  0000 L CNN
 F 2 "Capacitors_SMD:C_0603_HandSoldering" H 3300 3600 50  0001 C CNN
 F 3 "" H 3300 3600 50  0001 C CNN
@@
 P 3750 4150
 F 0 "R2" V 3850 4100 50  0000 L CNN
-F 1 "22" V 3850 4250 50  0000 L CNN
+F 1 "0" V 3850 4250 50  0000 L CNN
 F 2 "Resistors_SMD:R_0603_HandSoldering" H 3750 4150 50  0001 C CNN
 F 3 "" H 3750 4150 50  0001 C CNN
@@
 P 3750 4050
 F 0 "R1" V 3650 4000 50  0000 L CNN
-F 1 "22" V 3650 4150 50  0000 L CNN
+F 1 "0" V 3650 4150 50  0000 L CNN
 F 2 "Resistors_SMD:R_0603_HandSoldering" H 3750 4050 50  0001 C CNN
 F 3 "" H 3750 4050 50  0001 C CNN

Commit message: keyboard pcb: updated with small cleanups to KiCAD 5.x
Parts:
- C1, C2, C3, C4, C5: symbol C_Small -> Device:C_Small
- D80: symbol LED -> Device:LED
- J1: symbol Conn_01x02 -> Connector_Generic:Conn_01x02
- J2: symbol Conn_01x06 -> Connector_Generic:Conn_01x06
- J3: symbol Conn_01x05 -> Connector_Generic:Conn_01x05
- MH1, MH2, MH3, MH4, MH5, MH6: symbol TEST -> Mechanical:MountingHole
- R1, R2, R3, R4: symbol R_Small -> Device:R_Small
- U1: symbol ATMEGA32U4-AU -> MCU_Microchip_ATmega:ATmega32U4-AU
- Y1: symbol Crystal_GND24 -> Device:Crystal_GND24
Connections:
- wire segments 63 -> 71
