File: reform2-motherboard/reform2-motherboard/reform2-motherboard.kicad_pcb (KiCad board)
At the start: 6 copper layers, 276 x 93.5 mm, 423 parts, among them J1 Jack-DC, J10 1-2199230-6, J11 48099-5701, J12 BATCON1, J13 BATCON2, J14 USB_INT2, J17 USB3_A, J18 Conn_01x03_Male, J19 JTAG, J2 EDP_30, J20 Conn_01x03_Male, J21 Conn_01x04_Male, J3 SD_Card, J4 HDMI_A, J5 USB3_A, J6 USB3_A, J7 SJ-43516-SMT, J8 USB_B_Micro, J9 USB_INT1, P1 J0G-0003NL, Q1 Si4850BDY, Q10 PMV50EPEAR, Q11 PMV50EPEAR, Q12 PMV50EPEAR, Q13 PMV55ENEA, Q2 Si4850BDY, Q3 PMV55ENEA, Q4 PMV55ENEA, Q5 PMV50EPEAR, Q6 PMV50EPEAR, Q7 PMV50EPEAR, Q8 PMV50EPEAR, Q9 PMV50EPEAR, SW1 SW_Push, SW2 SW_Push, SW3 SW_DIP_x01, SW6 SW_Push, SW7 SW_Push, U1 CL-SOM-iMX8, U10 SN65DSI86ZQER, U11 679105700, U12 LM2677-3.3, U13 TLV71312PDBV, U14 TLV71311PDBV, U15 TPS2561, U16 TPS2561, U17 TLV1117-18, U18 LPC11U24FBD48-301, U19 TLV1117-15, U2 LTC4162-F, U20 WM8731, U21 MAX9715ETE+, U22 CM2020-00TR, U3 LTC4359-MS8, U4 LTC6803-4, U5 LTC4359-MS8, U6 INA260, U7 LM2596T-5, U8 LM2596T-ADJ, U9 TUSB8041, Y1 24MHz, Y2 12MHz

Commit message: WIP: reform2 motherboard: WIP power routing
Parts:
- moved TP4 76.1 mm to (183.2, 41.2)
- moved R134 13.8 mm to (93.2, 44.0), turned to 90 degrees
- moved TP6 2.75 mm to (179.5, 117.2)
- moved TP7 2.75 mm to (182.2, 117.2)
- moved TP5 1.06 mm to (71.2, 44.2)
- moved C112 0.56 mm to (80.5, 64.0)
- moved C101 0.50 mm to (82.0, 65.8)
- moved C102 0.35 mm to (83.6, 63.2)
Routing:
- net +3V3: track 95.3 -> 824.8 mm, vias 0 -> 24
- net USB_PWR: track 62.7 -> 398.3 mm, vias 0 -> 8
- net BAT5+: track 34.9 -> 163.4 mm
- net GND: track 68.3 -> 170.6 mm, vias 6 -> 47
- net +1V8: track 12.4 -> 73.5 mm, vias 0 -> 2
- net /Reform 2 Power/28V_GATE2: track 80.0 -> 130.8 mm, vias 0 -> 3
- net +1V1: track 0.00 -> 35.9 mm, vias 0 -> 2
- net Net-(C90-Pad1): track 39.1 -> 73.1 mm, vias 1 -> 5
- net Net-(R64-Pad2): track 0.00 -> 28.2 mm, vias 0 -> 2
- net /Reform 2 Display/EDP_BL_ENABLE: track 0.00 -> 19.4 mm
- net /Reform 2 Display/EDP_LCD_TEST: track 0.00 -> 17.6 mm, vias 0 -> 2
- net Net-(C74-Pad1): track 29.2 -> 37.7 mm
- net Net-(D19-Pad1): track 8.42 -> 15.1 mm
- net +1V2: track 31.5 -> 37.4 mm
- net Net-(C27-Pad2): track 0.00 -> 4.49 mm
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- added copper zone on GND.Cu, net GND

Commit message: WIP: reform2: migrate to Boundary Devices i.MX8M SOM
Parts:
- removed R112: 10k, Resistor_SMD:R_0603_1608Metric
- removed R114, R121, R150: 0, Resistor_SMD:R_0603_1608Metric
- removed TP6: T_USB1_ID, TestPoint:TestPoint_Pad_1.0x1.0mm
- removed TP7: T_PWM3, TestPoint:TestPoint_Pad_1.0x1.0mm
- removed TP9: T_SD2_RESET, TestPoint:TestPoint_Pad_1.0x1.0mm
- U1: value CL-SOM-iMX8 -> Nitrogen8M; footprint footprints:TE_2-2013289-1 -> footprints:TE_1473149-4
- moved H10 260.1 mm to (65.2, 85.8)
- moved R42 86.8 mm to (127.0, -17.5)
- moved C121 68.7 mm to (144.6, 3.20)
- moved C122 68.7 mm to (142.8, 3.20)
- moved TP4 39.5 mm to (193.0, 3.00)
- moved R111 10.6 mm to (170.8, 84.3), turned to 0 degrees
- moved R131 3.26 mm to (86.8, 82.8)
- moved R132 3.25 mm to (92.0, 82.8)
- moved U1 0.50 mm to (161.0, 77.0), turned to 90 degrees
Connections:
- net SD2_WP renamed Net-(U1-Pad67)
- U1 pad 1: GND -> +4V
- U1 pad 10: +4V -> Net-(U1-Pad10)
- U1 pad 100: Net-(U1-Pad100) -> USB1_DP
- U1 pad 101: Net-(U1-Pad101) -> DAC_SCL
- U1 pad 102: Net-(U1-Pad102) -> USB1_DN
- U1 pad 103: Net-(U1-Pad103) -> DAC_SDA
- U1 pad 104: Net-(U1-Pad104) -> GND
- U1 pad 105: GND -> BACKLIGHT_EN
- U1 pad 106: Net-(U1-Pad106) -> USB1_TX_N
- U1 pad 107: Net-(U1-Pad107) -> EDP_SCL
- U1 pad 108: Net-(U1-Pad108) -> USB1_TX_P
- U1 pad 109: Net-(U1-Pad109) -> EDP_SDA
- U1 pad 11: LPC_MOSI -> Net-(U1-Pad11)
- U1 pad 110: Net-(U1-Pad110) -> GND
- U1 pad 111: IMX_UART1_TX -> GND
- U1 pad 112: Net-(U1-Pad112) -> USB1_RX_N
- U1 pad 113: Net-(U1-Pad113) -> USB2_TX_P
- U1 pad 114: +4V -> USB1_RX_P
- U1 pad 115: Net-(U1-Pad115) -> USB2_TX_N
- U1 pad 116: Net-(U1-Pad116) -> GND
- U1 pad 117: IMX_UART1_RX -> GND
- U1 pad 118: Net-(U1-Pad118) -> Net-(R111-Pad2)
- U1 pad 119: PCIE1_CLK_P -> USB2_RX_P
- U1 pad 12: ETH0_B+ -> SD2_DATA0
- U1 pad 121: PCIE1_CLK_N -> USB2_RX_N
- U1 pad 122: Net-(U1-Pad122) -> IMX_UART2_RX
- U1 pad 124: Net-(U1-Pad124) -> IMX_UART2_TX
- U1 pad 125: PCIE1_TX_P -> USB2_DN
- U1 pad 126: Net-(U1-Pad126) -> IMX_UART1_RX
- U1 pad 127: PCIE1_TX_N -> USB2_DP
- U1 pad 128: Net-(U1-Pad128) -> IMX_UART1_TX
- U1 pad 129: Net-(U1-Pad129) -> GND
- U1 pad 13: LPC_SCK -> GND
- U1 pad 131: PCIE1_RX_P -> Net-(U1-Pad131)
- U1 pad 132: +4V -> Net-(U1-Pad132)
- U1 pad 133: PCIE1_RX_N -> Net-(U1-Pad133)
- U1 pad 139: Net-(U1-Pad139) -> Net-(SW3-Pad2)
- U1 pad 14: ETH0_B- -> SD2_DATA1
- U1 pad 141: GND -> Net-(U1-Pad141)
- U1 pad 15: LPC_MISO -> Net-(U1-Pad15)
- U1 pad 150: +4V -> Net-(U1-Pad150)
- U1 pad 156: Net-(R111-Pad2) -> Net-(U1-Pad156)
- U1 pad 158: USB2_RX_P -> Net-(U1-Pad158)
- U1 pad 159: GND -> Net-(U1-Pad159)
- U1 pad 16: ETH0_LED_LINK1 -> SD2_DATA2
- U1 pad 160: USB2_RX_N -> Net-(U1-Pad160)
- U1 pad 161: Net-(U1-Pad161) -> GND
- U1 pad 164: USB2_TX_P -> BACKLIGHT_PWM
- U1 pad 165: IMX_ONOFF -> Net-(U1-Pad165)
- U1 pad 166: USB2_TX_N -> DAC_DIN
- U1 pad 167: PCIE2_RX_N -> GND
- U1 pad 168: +4V -> DAC_RXFS
- U1 pad 169: PCIE2_RX_P -> HDMI_D0-
- U1 pad 170: USB2_DN -> DAC_BCLK
- U1 pad 171: IMX_RESETn -> HDMI_D0+
- U1 pad 172: USB2_DP -> DAC_TXFS
- U1 pad 173: PCIE2_TX_P -> GND
- U1 pad 175: PCIE2_TX_N -> HDMI_D1-
- U1 pad 176: USB1_DP -> DAC_MCLK
- U1 pad 177: GND -> HDMI_D1+
- U1 pad 178: USB1_DN -> DAC_DOUT
- U1 pad 179: PCIE2_CLK_N -> GND
- U1 pad 18: ETH0_C- -> SD2_DATA3
- U1 pad 181: PCIE2_CLK_P -> HDMI_D2-
- U1 pad 182: USB1_RX_P -> Net-(U1-Pad182)
- U1 pad 183: Net-(R150-Pad1) -> HDMI_D2+
- U1 pad 184: USB1_RX_N -> Net-(U1-Pad184)
- U1 pad 185: Net-(SW3-Pad2) -> GND
- U1 pad 186: +4V -> Net-(U1-Pad186)
- U1 pad 187: Net-(U1-Pad187) -> HDMI_D3+
- U1 pad 188: USB1_TX_P -> Net-(U1-Pad188)
- U1 pad 189: Net-(R112-Pad1) -> HDMI_D3-
- U1 pad 190: USB1_TX_N -> Net-(U1-Pad190)
- U1 pad 191: DAC_MCLK -> GND
- U1 pad 193: Net-(U1-Pad193) -> HDMI_SDA
- U1 pad 195: Net-(U1-Pad195) -> HDMI_SCL
- U1 pad 197: DAC_BCLK -> HDMI_CEC
- U1 pad 198: BACKLIGHT_EN -> Net-(U1-Pad198)
- U1 pad 199: DAC_TXFS -> HDMI_HPD
- U1 pad 2: Net-(U1-Pad2) -> +4V
- U1 pad 20: ETH0_C+ -> SD2_CMD
- U1 pad 200: BACKLIGHT_PWM -> Net-(U1-Pad200)
- U1 pad 22: ETH0_LED_LINK2 -> SD2_CLK
- U1 pad 24: ETH0_D- -> Net-(U1-Pad24)
- U1 pad 25: HDMI_SCL -> GND
- U1 pad 26: ETH0_D+ -> SD2_CD
- U1 pad 28: +4V -> Net-(U1-Pad28)
- U1 pad 3: PCIE2_CLKREQn -> +4V
- U1 pad 30: HDMI_D3+ -> Net-(U1-Pad30)
- U1 pad 31: HDMI_SDA -> GND
- U1 pad 32: HDMI_D3- -> Net-(U1-Pad32)
- U1 pad 33: DSI_D2_P -> Net-(U1-Pad33)
- U1 pad 34: HDMI_CEC -> Net-(U1-Pad34)
- U1 pad 35: DSI_D2_N -> Net-(U1-Pad35)
- U1 pad 36: HDMI_D0+ -> Net-(U1-Pad36)
- U1 pad 37: GND -> Net-(U1-Pad37)
- U1 pad 38: HDMI_D0- -> Net-(U1-Pad38)
- U1 pad 39: DSI_D0_P -> Net-(U1-Pad39)
- U1 pad 4: ETH0_LED_RX -> +4V
- U1 pad 40: HDMI_HPD -> Net-(U1-Pad40)
- U1 pad 41: DSI_D0_N -> GND
- U1 pad 42: HDMI_D1+ -> Net-(U1-Pad42)
- U1 pad 43: DAC_SCL -> Net-(U1-Pad43)
- U1 pad 44: HDMI_D1- -> GND
- U1 pad 45: DSI_D1_P -> Net-(U1-Pad45)
- U1 pad 46: +4V -> PCIE1_TX_P
- U1 pad 47: DSI_D1_N -> GND
- U1 pad 48: HDMI_D2+ -> PCIE1_TX_N
- U1 pad 49: DAC_SDA -> Net-(U1-Pad49)
- U1 pad 5: PCIE1_CLKREQn -> +4V
- U1 pad 50: HDMI_D2- -> GND
- U1 pad 51: DSI_D3_P -> Net-(U1-Pad51)
- U1 pad 52: Net-(U1-Pad52) -> PCIE1_RX_P
- U1 pad 53: DSI_D3_N -> GND
- U1 pad 54: Net-(TP4-Pad1) -> PCIE1_RX_N
- U1 pad 55: GND -> Net-(U1-Pad55)
- U1 pad 56: IMX_JTAG_RSTn -> GND
- U1 pad 57: DSI_CLK_N -> Net-(U1-Pad57)
- U1 pad 58: IMX_UART2_TX -> PCIE1_CLK_P
- U1 pad 59: DSI_CLK_P -> GND
- U1 pad 6: ETH0_A- -> +4V
- U1 pad 60: Net-(U1-Pad60) -> PCIE1_CLK_N
- U1 pad 61: SD2_CD -> Net-(U1-Pad61)
- U1 pad 62: Net-(U1-Pad62) -> GND
- U1 pad 63: IMX_UART2_RX -> Net-(U1-Pad63)
- U1 pad 64: +4V -> PCIE2_CLK_P
- U1 pad 65: Net-(U1-Pad65) -> GND
- U1 pad 66: IMX_JTAG_TCK -> PCIE2_CLK_N
- U1 pad 68: IMX_JTAG_TMS -> GND
- U1 pad 7: Net-(U1-Pad7) -> GND
- U1 pad 70: IMX_JTAG_TDI -> PCIE2_TX_N
- U1 pad 72: IMX_JTAG_TDO -> PCIE2_TX_P
- U1 pad 73: EDP_SCL -> IMX_JTAG_TCK
- U1 pad 74: Net-(U1-Pad74) -> GND
- U1 pad 75: EDP_SDA -> IMX_JTAG_TDI
- U1 pad 76: Net-(U1-Pad76) -> PCIE2_RX_P
- U1 pad 77: Net-(U1-Pad77) -> IMX_JTAG_TMS
- U1 pad 78: +4V -> PCIE2_RX_N
- U1 pad 79: Net-(U1-Pad79) -> Net-(TP4-Pad1)
- U1 pad 8: ETH0_A+ -> Net-(TP8-Pad1)
- U1 pad 80: SD2_CLK -> GND
- U1 pad 81: Net-(U1-Pad81) -> IMX_JTAG_RSTn
- U1 pad 82: SD2_CMD -> Net-(U1-Pad82)
- U1 pad 83: Net-(U1-Pad83) -> IMX_JTAG_TDO
- U1 pad 84: SD2_DATA0 -> Net-(U1-Pad84)
- U1 pad 86: SD2_DATA1 -> Net-(U1-Pad86)
- U1 pad 87: GND -> IMX_RESETn
- U1 pad 88: SD2_DATA2 -> Net-(U1-Pad88)
- U1 pad 90: SD2_DATA3 -> Net-(U1-Pad90)
- U1 pad 91: Net-(U1-Pad91) -> LPC_MOSI
- U1 pad 93: Net-(U1-Pad93) -> LPC_MISO
- U1 pad 94: Net-(U1-Pad94) -> GND
- U1 pad 95: Net-(U1-Pad95) -> GND
- U1 pad 96: +4V -> Net-(U1-Pad96)
- U1 pad 97: Net-(U1-Pad97) -> LPC_SCK
- U1 pad 98: Net-(U1-Pad98) -> GND
- U1 pad 99: Net-(U1-Pad99) -> GND
Routing:
- net ETH0_LED_LINK2: track 198.9 -> 0.00 mm, vias 1 -> 0
- net ETH0_A+: track 175.9 -> 0.00 mm, vias 1 -> 0
- net ETH0_LED_RX: track 173.4 -> 0.00 mm, vias 1 -> 0
- net ETH0_A-: track 173.1 -> 0.00 mm, vias 1 -> 0
- net ETH0_LED_LINK1: track 168.1 -> 0.00 mm, vias 1 -> 0
- net ETH0_B-: track 163.9 -> 0.00 mm, vias 1 -> 0
- net ETH0_B+: track 158.7 -> 0.00 mm, vias 1 -> 0
- net ETH0_D+: track 145.4 -> 0.00 mm, vias 1 -> 0
- net ETH0_D-: track 143.2 -> 0.00 mm, vias 1 -> 0
- net ETH0_C-: track 139.4 -> 0.00 mm, vias 1 -> 0
- net ETH0_C+: track 139.1 -> 0.00 mm, vias 1 -> 0
- net SD2_DATA1: track 132.3 -> 5.05 mm, vias 2 -> 1
- net HDMI_HPD: track 114.7 -> 10.2 mm, vias 2 -> 1
- net HDMI_SCL: track 102.1 -> 0.00 mm, vias 2 -> 0
- net HDMI_SDA: track 101.8 -> 0.00 mm, vias 2 -> 0
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
Commit message: WIP: reform2: more routing, 73 pads left
Parts:
- SW3: footprint Button_Switch_SMD:SW_DIP_SPSTx01_Slide_6.7x4.1mm_W8.61mm_P2.54mm_LowProfile -> Button_Switch_SMD:SW_DIP_SPSTx01_Slide_Omron_A6S-110x_W8.9mm_P2.54mm
- moved R42 83.9 mm to (168.0, 55.7), turned to 90 degrees
- moved TP4 79.7 mm to (154.0, 72.5)
- moved TP8 78.5 mm to (185.5, 41.5)
- moved SW3 74.0 mm to (220.0, 119.2), turned to 90 degrees
- moved R113 62.0 mm to (216.3, 119.2), turned to 270 degrees
- moved C121 55.8 mm to (144.9, 59.0)
- moved C122 55.8 mm to (143.2, 59.0)
- moved C124 6.73 mm to (150.5, 54.2), turned to 270 degrees
- moved C126 6.59 mm to (152.8, 54.2), turned to 90 degrees
- moved FB4 3.79 mm to (151.8, 57.0), turned to 0 degrees
- moved C45 2.00 mm to (153.2, 110.2)
- moved R111 1.51 mm to (169.3, 84.1), turned to 180 degrees
- moved C61 1.50 mm to (148.5, 54.2), turned to 270 degrees
- moved C44 1.50 mm to (153.2, 112.0)
- moved R100 0.60 mm to (165.0, 120.6)
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Connections:
- U1 pad 11: Net-(U1-Pad11) -> ETH0_D+
- U1 pad 15: Net-(U1-Pad15) -> ETH0_B-
- U1 pad 163: Net-(U1-Pad163) -> HDMI_D3+
- U1 pad 165: Net-(U1-Pad165) -> HDMI_D3-
- U1 pad 17: Net-(U1-Pad17) -> ETH0_B+
- U1 pad 187: HDMI_D3+ -> Net-(U1-Pad187)
- U1 pad 189: HDMI_D3- -> Net-(U1-Pad189)
- U1 pad 21: Net-(U1-Pad21) -> ETH0_C-
- U1 pad 23: Net-(U1-Pad23) -> ETH0_C+
- U1 pad 27: Net-(U1-Pad27) -> ETH0_A-
- U1 pad 29: Net-(U1-Pad29) -> ETH0_A+
- U1 pad 9: Net-(U1-Pad9) -> ETH0_D-
Routing:
- net GND: track 170.6 -> 368.3 mm, vias 41 -> 104
- net ETH0_B-: track 0.00 -> 152.2 mm, vias 0 -> 2
- net ETH0_B+: track 0.00 -> 151.0 mm, vias 0 -> 2
- net ETH0_D-: track 0.00 -> 149.0 mm, vias 0 -> 2
- net ETH0_C-: track 0.00 -> 146.7 mm, vias 0 -> 1
- net ETH0_C+: track 0.00 -> 146.7 mm, vias 0 -> 1
- net ETH0_D+: track 0.00 -> 146.2 mm, vias 0 -> 2
- net ETH0_A-: track 0.00 -> 144.9 mm, vias 0 -> 1
- net ETH0_A+: track 0.00 -> 144.9 mm, vias 0 -> 1
- net SD2_DATA1: track 5.05 -> 146.6 mm, vias 1 -> 3
- net HDMI_SCL: track 0.00 -> 134.3 mm, vias 0 -> 2
- net HDMI_SDA: track 0.00 -> 128.3 mm, vias 0 -> 2
- net HDMI_HPD: track 10.2 -> 134.5 mm, vias 1 -> 2
- net DAC_RXFS: track 14.3 -> 128.7 mm
- net BACKLIGHT_PWM: track 0.00 -> 106.5 mm, vias 0 -> 2
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Other:
- board text removed: "USB SW 1"

Commit message: WIP: reform2: more routing, 11 pads left
Parts:
- added J15: Conn_01x33, Connector_FFC-FPC:Hirose_FH12-33S-0.5SH_1x33-1MP_P0.50mm_Horizontal, F.Cu at (200.4, 63.7)
- moved C7 42.6 mm to (274.6, 102.2)
- moved C34 14.9 mm to (260.2, 115.8), turned to 270 degrees
- moved C33 7.70 mm to (246.0, 101.8), turned to 90 degrees
- moved C1 2.81 mm to (255.2, 97.7)
- moved Q2 0.50 mm to (264.4, 112.0)
Routing:
- net GND: track 368.3 -> 546.2 mm, vias 104 -> 129
- net DSI_D0_P: track 0.00 -> 156.9 mm, vias 0 -> 2
- net DSI_D0_N: track 0.00 -> 155.2 mm, vias 0 -> 2
- net DSI_D1_P: track 0.00 -> 147.5 mm, vias 0 -> 2
- net DSI_D1_N: track 0.00 -> 146.0 mm, vias 0 -> 2
- net DSI_CLK_P: track 0.00 -> 141.3 mm, vias 0 -> 2
- net DSI_CLK_N: track 0.00 -> 139.9 mm, vias 0 -> 2
- net DSI_D2_P: track 0.00 -> 134.5 mm, vias 0 -> 2
- net DSI_D2_N: track 0.00 -> 133.0 mm, vias 0 -> 2
- net DSI_D3_P: track 0.00 -> 129.1 mm, vias 0 -> 2
- net DSI_D3_N: track 0.00 -> 127.9 mm, vias 0 -> 2
- net +3V3: track 850.1 -> 973.2 mm, vias 26 -> 30
- net /Reform 2 Power/36V_IN: track 34.6 -> 124.4 mm, vias 2 -> 6
- net +1V2: track 42.0 -> 130.5 mm, vias 2 -> 8
- net +1V8: track 65.0 -> 135.8 mm, vias 2 -> 3
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Other:
- board text removed: "USB SW 2"

Commit message: WIP: reform2: silkscreen cleanups and more 3d models added
Parts:
- added G***: LOGO, footprints:36v, F.Cu at (289.0, 44.2)
- added G***: LOGO, footprints:cpu, F.Cu at (182.5, 69.2)
- H11: value LABEL_MPCIE1 -> LOGO; footprint footprints:label-mpcie -> footprints:mpcie
- H12: value LABEL_MPCIE2 -> LOGO; footprint footprints:label-mpcie -> footprints:nvme
- moved H12 34.6 mm to (142.5, 69.2)
- moved H11 1.77 mm to (111.2, 69.2)

Commit message: reform2: first motherboard fully routed, checks TBD
Parts:
- removed SW7: SW_Push, Button_Switch_SMD:SW_Push_1P1T_NO_CK_KMR2
- removed TP4: T_JTAG_MOD, TestPoint:TestPoint_Pad_1.0x1.0mm
- added J16: LINE_IN, Connector_PinHeader_2.54mm:PinHeader_1x03_P2.54mm_Vertical, F.Cu at (286.8, 130.5)
- added J22: LPC_IO, Connector_PinHeader_2.54mm:PinHeader_2x08_P2.54mm_Vertical, F.Cu at (227.8, 84.2)
- added R112: 220, Resistor_SMD:R_0603_1608Metric, F.Cu at (205.7, 80.8)
- added R114: 33, Resistor_SMD:R_0603_1608Metric, F.Cu at (279.2, 84.0)
- added R121: 33, Resistor_SMD:R_0603_1608Metric, F.Cu at (278.6, 85.9)
- added R150: 33, Resistor_SMD:R_0603_1608Metric, F.Cu at (279.6, 89.5)
- added R151: 33, Resistor_SMD:R_0603_1608Metric, F.Cu at (279.1, 87.7)
- added R152: 0, Resistor_SMD:R_0603_1608Metric, F.Cu at (295.5, 83.5)
- added R153: 0, Resistor_SMD:R_0603_1608Metric, F.Cu at (151.8, 60.0)
- added R154: 0, Resistor_SMD:R_0603_1608Metric, F.Cu at (176.4, 55.1)
- added R155: 0, Resistor_SMD:R_0603_1608Metric, F.Cu at (181.1, 55.1)
- added R156: 0, Resistor_SMD:R_0603_1608Metric, F.Cu at (151.8, 94.8)
- added R157: 0, Resistor_SMD:R_0603_1608Metric, F.Cu at (213.5, 84.8)
- added R65: 0, Resistor_SMD:R_0603_1608Metric, F.Cu at (215.5, 107.3)
- added R66: 220, Resistor_SMD:R_0603_1608Metric, F.Cu at (214.0, 80.8)
- added TP1: T_GAIN, TestPoint:TestPoint_Pad_1.0x1.0mm, F.Cu at (293.6, 81.5)
- added TP2: T_OTG, TestPoint:TestPoint_Pad_1.0x1.0mm, F.Cu at (188.4, 41.5)
- H11: value LOGO -> LABEL_MPCIE1
- H12: value LOGO -> LABEL_MPCIE2
- H13: renamed from G***; value LOGO -> LABEL_CPU
- H14: renamed from G***; value LOGO -> LABEL_36V
- J18, J20: footprint Connector_PinSocket_2.54mm:PinSocket_1x03_P2.54mm_Vertical -> Connector_PinHeader_2.54mm:PinHeader_1x03_P2.54mm_Vertical
- J21: footprint Connector_PinSocket_2.54mm:PinSocket_1x04_P2.54mm_Vertical -> Connector_PinHeader_2.54mm:PinHeader_1x04_P2.54mm_Vertical
- R123: value 2.4k 1% -> 3k 1%
- R138: value 0 -> 33
- R139: value 100 -> 33
- moved R139 4.81 mm to (278.7, 91.3), turned to 0 degrees
- moved R136 4.50 mm to (209.2, 80.8)
- moved C139 3.58 mm to (279.5, 97.5)
- moved C142 3.58 mm to (277.5, 97.5)
- moved C146 3.58 mm to (279.5, 94.2)
- moved C151 3.58 mm to (277.5, 94.2)
- moved R54 2.49 mm to (271.8, 89.2)
- moved R42 1.74 mm to (169.6, 56.4), turned to 180 degrees
Connections:
- net Net-(U18-Pad48) renamed /Reform 2 Power/LPC_PIO1_16
- net USB3_3_SSRXN renamed Net-(U9-Pad23)
- net USB3_3_SSRXP renamed Net-(U9-Pad22)
- net USB3_3_SSTXN renamed Net-(U9-Pad20)
- net USB3_3_SSTXP renamed Net-(U9-Pad19)
- net USB3_4_SSRXN renamed Net-(U9-Pad30)
- net USB3_4_SSRXP renamed Net-(U9-Pad29)
- net USB3_4_SSTXN renamed Net-(U9-Pad27)
- net USB3_4_SSTXP renamed Net-(U9-Pad26)
- J19 pad 13: IMX_JTAG_TDO -> ETH0_LED_LINK1
- J19 pad 15: IMX_JTAG_RSTn -> ETH0_LED_LINK2
- R119 pad 2: IMX_JTAG_RSTn -> ETH0_LED_LINK2
- R135 pad 2: DAC_SCL -> Net-(R135-Pad2)
- R136 pad 2: DAC_SDA -> Net-(R112-Pad2)
- R139 pad 1: Net-(R139-Pad1) -> DAC_RXFS
- R149 pad 2: IMX_JTAG_RSTn -> ETH0_LED_LINK2
- U1 pad 100: USB1_DP -> USB1_DN
- U1 pad 102: USB1_DN -> USB1_DP
- U1 pad 131: Net-(U1-Pad131) -> USB_RESETn
- U1 pad 164: BACKLIGHT_PWM -> Net-(R156-Pad2)
- U1 pad 70: PCIE2_TX_N -> PCIE2_TX_P
- U1 pad 72: PCIE2_TX_P -> PCIE2_TX_N
- U1 pad 79: Net-(TP4-Pad1) -> ETH0_LED_RX
- U1 pad 81: IMX_JTAG_RSTn -> ETH0_LED_LINK2
- U1 pad 83: IMX_JTAG_TDO -> ETH0_LED_LINK1
- U1 pad 89: Net-(U1-Pad89) -> LPC_SS0
- U18 pad 1: Net-(U18-Pad1) -> /Reform 2 Power/LPC_PIO1_25
- U18 pad 25: Net-(U18-Pad25) -> /Reform 2 Power/LPC_PIO1_31
- U18 pad 36: /Reform 2 Power/LPC_TXDb -> LPC_UART2_TX
- U18 pad 37: /Reform 2 Power/LPC_RXDb -> LPC_UART2_RX
- U20 pad 2: Net-(R139-Pad1) -> Net-(U20-Pad2)
- U20 pad 23: DAC_SDA -> Net-(R112-Pad2)
- U20 pad 24: DAC_SCL -> Net-(R135-Pad2)
- U20 pad 3: DAC_BCLK -> Net-(R114-Pad2)
- U20 pad 4: DAC_DOUT -> Net-(R121-Pad2)
- U20 pad 5: DAC_TXFS -> Net-(R151-Pad2)
- U20 pad 6: DAC_DIN -> Net-(R150-Pad2)
- U20 pad 7: DAC_RXFS -> Net-(R139-Pad2)
Routing:
- net ETH0_LED_LINK2: track 0.00 -> 252.2 mm, vias 0 -> 4
- net ETH0_LED_LINK1: track 0.00 -> 234.9 mm, vias 0 -> 4
- net ETH0_LED_RX: track 0.00 -> 169.8 mm, vias 0 -> 3
- net SD2_CD: track 4.01 -> 152.4 mm, vias 0 -> 3
- net IMX_JTAG_RSTn: track 98.2 -> 0.00 mm, vias 2 -> 0
- net Net-(R112-Pad2): track 0.00 -> 95.2 mm, vias 0 -> 2
- net Net-(R135-Pad2): track 0.00 -> 91.6 mm, vias 0 -> 2
- net DAC_SDA: track 142.2 -> 52.5 mm, vias 4 -> 2
- net DAC_SCL: track 142.5 -> 61.6 mm, vias 4 -> 2
- net IMX_JTAG_TDO: track 77.7 -> 0.00 mm, vias 2 -> 0
- net LPC_SS0: track 0.00 -> 77.5 mm, vias 0 -> 2
- net USB_RESETn: track 0.00 -> 69.6 mm, vias 0 -> 2
- net Net-(R65-Pad2): track 0.00 -> 66.8 mm, vias 0 -> 2
- net LPC_UART2_RX: track 0.00 -> 64.9 mm, vias 0 -> 2
- net LPC_UART2_TX: track 0.00 -> 64.6 mm, vias 0 -> 2
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Other:
- board text added: "JTAG"
- board text added: "LPC I/O"
- board text removed: "DAC"
