File: reform2-motherboard/reform2-motherboard/reform2-power.sch (KiCad schematic (older format))
At the start: 158 parts, among them J1 Jack-DC, J2 BATCON, J22 LPC_IO, J23 POWERS, J8 USB_B_Micro, Q1 Si4850BDY, Q10 PMV50EPEAR, Q11 PMV50EPEAR, Q12 PMV50EPEAR, Q13 PMV55ENEA, Q14 PMV50EPEAR, Q15 PMV50EPEAR, Q2 Si4850BDY, Q3 PMV55ENEA, Q4 PMV55ENEA, Q5 PMV50EPEAR, Q6 PMV50EPEAR, Q7 PMV50EPEAR, Q8 PMV50EPEAR, Q9 PMV50EPEAR, SW1 SW_DIP_x01, SW2 SW_Push, U12 LM2677SX-3.3, U13 TLV71312PDBV, U14 TLV71311PDBV, U17 TLV1117-18, U18 LPC11U24FBD48-301, U19 TLV1117-15, U2 LTC4162-F, U3 LTC4359-MS8, U4 LTC6803-4, U5 LTC4359-MS8, U6 INA260, U7 LM2677SX-5, Y2 12MHz

Commit message: reform2 motherboard: finalize BOM
Parts:
- removed Q14: PMV50EPEAR, Package_TO_SOT_SMD:SOT-23, symbol Transistor_FET:DMG2301L
- added R149, R166: 0, Resistor_SMD:R_0603_1608Metric, symbol Device:R_Small
- added SW4: SW_3V3OFF, Button_Switch_SMD:SW_DIP_SPSTx01_Slide_Omron_A6S-110x_W8.9mm_P2.54mm, symbol Switch:SW_DIP_x01
- C125, C34: value 1uF -> 10uF; Manufacturer Taiyo Yuden -> Murata; Manufacturer_No UMK107BJ105KA-T -> GRM188R6YA106MA73D
- C16, C17, C18, C19, C3: Manufacturer KEMET -> UCC; Manufacturer_No EDH226M050S9GAA -> EMZR500ARA221MHA0G
- C2: Manufacturer (none) -> Yageo; Manufacturer_No (none) -> CC0603JPX7R9BB104
- C37, C38, C46, C47: Manufacturer TDK -> Murata; Manufacturer_No CGA3E2X8R1E104K080AE -> GRM188R6YA106MA73D
- D10, D3, D4, D5, D6, D7, D8, D9: Manufacturer_No PDZ7.5B -> PDZ7.5BGWJ
- D2: value BAT46W -> BAT46WJ,115; Manufacturer_No BAT46W -> BAT46WJ,115
- J2: Manufacturer (none) -> Molex; Manufacturer_No (none) -> 105405-1110
- Q1: value Si4850BDY -> SI4850BDY; Manufacturer_No Si4850BDY -> SI4850BDY-T1-GE3
- Q13, Q3, Q4: value PMV55ENEA -> PMV55ENEAR; Manufacturer_No PMV55ENEA -> PMV55ENEAR
- Q2: Manufacturer_No Si4850BDY -> SI4850BDY-T1-GE3
- R128: Manufacturer_No CRCW06030000Z0EAC -> CRCW060310K0JNEAC
- SW1: value SW_DIP_x01 -> SW_LPCPROG
- SW2: value SW_Push -> SW_LPCRST; Manufacturer_No KMR2 -> KMR223NGULCLFG
- U12: Manufacturer_No LM2677-3.3 -> LM2677SX-3.3
- U13: Manufacturer_No TLV71312PDBV -> TLV71312PDBVR
- U14: Manufacturer_No TLV71311PDBV -> TLV71311PDBVR
- U17: Manufacturer_No TLV1117-18 -> TLV1117-18CDCYR
- U19: Manufacturer_No TLV1117-15 -> TLV1117-15CDCYR
- U2: Manufacturer_No LTC4162-F -> LTC4162EUFD-FAD#PBF
- U3, U5: value LTC4359-MS8 -> LTC4359IMS8; Manufacturer_No LTC4359-MS8 -> LTC4359IMS8#PBF
- U4: Manufacturer_No LTC6803-4 -> LTC6803IG-4#PBF
- U6: Manufacturer_No INA260 -> INA260AIPWR
- U7: Manufacturer_No LM2677-3.3 -> LM2677SX-5
- Y2: Manufacturer_No ABM8AIG-12.000MHZ -> ABM8AIG-12.000MHz-2-T
Connections:
- net 28V_GATE2: no longer U12.7 (ON/~OFF~)
- net GND: now also SW4.2
- net LPC_UART2_RX: now also R166.1; no longer U18.37 (PIO1_14)
- net LPC_UART2_TX: now also R149.1; no longer U18.36 (PIO1_13)
- net at R163.2: now also U7.7 (ON/~OFF~)
- new net: SW4.1, U12.7 (ON/~OFF~)
- new net LPC_RXDb: R166.2, U18.37 (PIO1_14)
- new net LPC_TXDb: R149.2, U18.36 (PIO1_13)
Other:
- note added: ""decreases gate\nramp time""
- note removed: "NOTE: C34 and C125\nhave lower than recmd\ncapacitance (10uF)"
- note removed: "Replace with general 3v3 switch"
- note removed: "TODO:\n1. physical switch for 3v3\n2. 8x LED moved to LPC control? how to identify problematic cells?\n3. 5v switch is controlled by LPC, can be bypassed by DIP switch\n4. LPC checks cell health when powered, alerts of problems\n"
- moved on the sheet: C17, R128, R163
