File: reform2-oled/reform2-oled.kicad_pcb (KiCad board)
At the start: 2 copper layers, 80 x 12 mm, 14 parts, among them J1 AUX, U1 SSD1306

Commit message: Reform2.0D-3 snapshot of PCBs and input device firmware
Parts:
- removed REF**: WEEE-Logo_4.2x6mm_SilkScreen, Symbol:WEEE-Logo_4.2x6mm_SilkScreen
- removed TP1: TP_RES, TestPoint:TestPoint_Pad_D1.0mm
- added C7: 1uF, Capacitor_SMD:C_0603_1608Metric_Pad1.05x0.95mm_HandSolder, B.Cu at (181.2, 99.5)
- added R2: 4.7k, Resistor_SMD:R_0603_1608Metric_Pad1.05x0.95mm_HandSolder, B.Cu at (177.4, 99.5)
- J1: footprint Connector_PinHeader_2.00mm:PinHeader_1x04_P2.00mm_Horizontal -> Connector_FFC-FPC:Molex_200528-0040_1x04-1MP_P1.00mm_Horizontal
- moved C5 12.9 mm to (162.4, 99.5)
- moved J1 6.58 mm to (170.7, 94.9), turned to 270 degrees
Connections:
- J1 pad 1: +3V3 -> GND
- J1 pad 2: DISP_SDA -> DISP_SCL
- J1 pad 3: DISP_SCL -> DISP_SDA
- J1 pad 4: GND -> +3V3
Routing:
- net +3V3: track 33.5 -> 22.3 mm
- net DISP_SDA: track 6.15 -> 13.2 mm, vias 0 -> 1
- net Net-(C5-Pad2): track 4.44 -> 10.4 mm
- net Net-(C7-Pad1): track 10.3 -> 12.7 mm
- net Net-(C5-Pad1): track 9.26 -> 6.99 mm
- net GND: track 11.3 -> 12.9 mm, vias 1 -> 6
- net DISP_SCL: track 6.27 -> 7.09 mm, vias 0 -> 1
Other:
- board text added: "REFORM OLED 2.0D-3 2020-03-05 MNTRE.COM"
- board text removed: "3V3 SDA SCL GND"
- board text removed: "Status OLED Rev D-1 (SSD3306 to I2C) 2019-11-07 MNT Research GmbH"
