File: reform2-oled/reform2-oled.sch (KiCad schematic (older format))
At the start: 13 parts, among them J1 AUX, U1 SSD1306

Commit message: Reform2.0D-3 snapshot of PCBs and input device firmware
Parts:
- removed TP1: TP_RES, TestPoint:TestPoint_Pad_D1.0mm, symbol Connector:TestPoint
- added C7: 1uF, Capacitor_SMD:C_0603_1608Metric_Pad1.05x0.95mm_HandSolder, symbol Device:C_Small
- added R2: 4.7k, Resistor_SMD:R_0603_1608Metric_Pad1.05x0.95mm_HandSolder, symbol Device:R_Small
- C3, C4: Manufacturer_No UMK107BJ105KA-T -> LMK107BBJ106KALT
- J1: footprint Connector_PinHeader_2.00mm:PinHeader_1x04_P2.00mm_Horizontal -> Connector_FFC-FPC:Molex_200528-0040_1x04-1MP_P1.00mm_Horizontal; Manufacturer Wurth -> Molex; Manufacturer_No 61300411121 -> 200528-0040
- R1: Manufacturer_No AF0603JR-0710KL -> AF0603FR-07330KL
Connections:
- net +3V3: now also J1.4 (Pin_4), R2.2; no longer J1.1 (Pin_1)
- net DISP_SCL: now also J1.2 (Pin_2); no longer J1.3 (Pin_3)
- net DISP_SDA: now also J1.3 (Pin_3); no longer J1.2 (Pin_2)
- net GND: now also J1.1 (Pin_1), C7.2; no longer J1.4 (Pin_4)
- net at U1.9 (~RES): now also C7.1, R2.1
Other:
- note added: "Reset RC circuit"
- note added: "Same side FFC mirrors the pins!"
- note removed: "TODO: reset RC circuit\nTODO: I2C resistor option"
Changed lines of the file:
@@
 L Connector_Generic:Conn_01x04 J1
 U 1 1 5D0C1E6C
-P 5850 3400
-F 0 "J1" H 5850 3700 50  0000 C CNN
-F 1 "AUX" H 5850 3000 50  0000 C CNN
-F 2 "Connector_PinHeader_2.00mm:PinHeader_1x04_P2.00mm_Horizontal" H 5850 3400 50  0001 C CNN
-F 3 "" H 5850 3400 50  0001 C CNN
-F 4 "Wurth" H 5850 3400 50  0001 C CNN "Manufacturer"
-F 5 "61300411121" H 5850 3400 50  0001 C CNN "Manufacturer_No"
-	1    5850 3400
-	1    0    0    -1
+P 5850 3500
+F 0 "J1" H 5850 3800 50  0000 C CNN
+F 1 "AUX" H 5850 3100 50  0000 C CNN
+F 2 "Connector_FFC-FPC:Molex_200528-0040_1x04-1MP_P1.00mm_Horizontal" H 5850 3500 50  0001 C CNN
+F 3 "" H 5850 3500 50  0001 C CNN
+F 4 "Molex" H 5850 3500 50  0001 C CNN "Manufacturer"
+F 5 "200528-0040" H 5850 3500 50  0001 C CNN "Manufacturer_No"
+	1    5850 3500
+	1    0    0    1
 $EndComp
 $Comp
@@
 Wire Wire Line
 	5200 3600 5650 3600
-$Comp
-L SSD1306_OLED-0.91-128x32:SSD1306 U1
-U 1 1 5EAB622B
-P 3350 3350
-F 0 "U1" V 3297 4028 60  0000 L CNN
-F 1 "SSD1306" V 3403 4028 60  0000 L CNN
-F 2 "KiCad-SSD1306_OLED-0:SSD1306_OLED-0.91-128x32" H 3350 3350 60  0001 C CNN
-F 3 "" H 3350 3350 60  0001 C CNN
-	1    3350 3350
-	0    1    1    0
-$EndComp
 $Comp
 L Device:C_Small C5
@@
 $EndComp
 Wire Wire Line
-	3350 2850 2700 2850
+	3350 2850 2900 2850
 Wire Wire Line
 	2700 2850 2700 2750
@@
 F 3 "" H 3050 4250 50  0001 C CNN
 F 4 "Yageo" H 3050 4250 50  0001 C CNN "Manufacturer"
-F 5 "AF0603JR-0710KL" H 3050 4250 50  0001 C CNN "Manufacturer_No"
+F 5 "AF0603FR-07330KL" H 3050 4250 50  0001 C CNN "Manufacturer_No"
 	1    3050 4250
 	0    1    1    0
@@
 F 3 "" H 2750 4450 50  0001 C CNN
 F 4 "Taiyo Yuden" H 2750 4450 50  0001 C CNN "Manufacturer"
-F 5 "UMK107BJ105KA-T" H 2750 4450 50  0001 C CNN "Manufacturer_No"
+F 5 "LMK107BBJ106KALT" H 2750 4450 50  0001 C CNN "Manufacturer_No"
 	1    2750 4450
 	0    1    -1   0
@@
 F 3 "" H 3000 4650 50  0001 C CNN
 F 4 "Taiyo Yuden" H 3000 4650 50  0001 C CNN "Manufacturer"
-F 5 "UMK107BJ105KA-T" H 3000 4650 50  0001 C CNN "Manufacturer_No"
+F 5 "LMK107BBJ106KALT" H 3000 4650 50  0001 C CNN "Manufacturer_No"
 	1    3000 4650
 	0    1    -1   0
@@
 	2350 3450 2200 3450
 Connection ~ 2200 3450
-Wire Wire Line
-	2200 3450 2200 4250
 Text Notes 2600 1750 0    60   ~ 0
 Based on Adafruit 931
-$Comp
-L Connector:TestPoint TP1
-U 1 1 5DC4FB56
-P 3350 3650
-F 0 "TP1" V 3400 3950 50  0000 C CNN
-F 1 "TP_RES" V 3300 3950 50  0000 C CNN
-F 2 "TestPoint:TestPoint_Pad_D1.0mm" H 3550 3650 50  0001 C CNN
-F 3 "~" H 3550 3650 50  0001 C CNN
-	1    3350 3650
-	0    -1   -1   0
-$EndComp
 $Comp
 L power:PWR_FLAG #FLG0101
@@
 Wire Wire Line
 	5450 3300 5650 3300
-Text Notes 4450 2700 0    50   ~ 0
-TODO: reset RC circuit\nTODO: I2C resistor option
+Text Notes 1500 3700 0    50   ~ 0
+Reset RC circuit
+$Comp
+L SSD1306_OLED-0.91-128x32:SSD1306 U1
+U 1 1 5EAB622B
+P 3350 3350
+F 0 "U1" V 3297 4028 60  0000 L CNN
+F 1 "SSD1306" V 3403 4028 60  0000 L CNN
+F 2 "KiCad-SSD1306_OLED-0:SSD1306_OLED-0.91-128x32" H 3350 3350 60  0001 C CNN
+F 3 "" H 3350 3350 60  0001 C CNN
+	1    3350 3350
+	0    1    1    0
+$EndComp
+$Comp
+L Device:C_Small C7
+U 1 1 5E7CCF56
+P 2450 3650
+F 0 "C7" H 2460 3720 50  0000 L CNN
+F 1 "1uF" H 2460 3570 50  0000 L CNN
+F 2 "Capacitor_SMD:C_0603_1608Metric_Pad1.05x0.95mm_HandSolder" H 2450 3650 50  0001 C CNN
+F 3 "" H 2450 3650 50  0001 C CNN
+F 4 "Taiyo Yuden" H 2450 3650 50  0001 C CNN "Manufacturer"
+F 5 "UMK107BJ105KA-T" H 2450 3650 50  0001 C CNN "Manufacturer_No"
+	1    2450 3650
+	0    1    -1   0
+$EndComp
+$Comp
+L Device:R_Small R2
+U 1 1 5E7D0D47
+P 2900 3050
+F 0 "R2" V 2800 3000 50  0000 L CNN
+F 1 "4.7k" V 3000 2950 50  0000 L CNN
+F 2 "Resistor_SMD:R_0603_1608Metric_Pad1.05x0.95mm_HandSolder" H 2900 3050 50  0001 C CNN
+F 3 "" H 2900 3050 50  0001 C CNN
+F 4 "Yageo" H 2900 3050 50  0001 C CNN "Manufacturer"
+F 5 "RC0603FR-074K7L" H 2900 3050 50  0001 C CNN "Manufacturer_No"
+	1    2900 3050
+	-1   0    0    1
+$EndComp
+Text Notes 4750 3000 0    60   ~ 0
+Same side FFC mirrors the pins!
+Wire Wire Line
+	2200 3450 2200 3650
+Wire Wire Line
+	2900 2950 2900 2850
+Connection ~ 2900 2850
+Wire Wire Line
+	2900 2850 2700 2850
+Wire Wire Line
+	2900 3150 2900 3650
+Connection ~ 2900 3650
+Wire Wire Line
+	2900 3650 3350 3650
+Wire Wire Line
+	2550 3650 2900 3650
+Wire Wire Line
+	2350 3650 2200 3650
+Connection ~ 2200 3650
+Wire Wire Line
+	2200 3650 2200 4250
 $EndSCHEMATC
