File: reform2-batterypack/reform2-batterypack.kicad_pcb (KiCad board)
At the start: 2 copper layers, 91 x 65.5 mm, 10 parts, among them J1 Conn_01x05_Female, U1 KEYSTONE_54, U2 KEYSTONE_54, U3 KEYSTONE_54, U4 KEYSTONE_54

Commit message: Reform2.0D-3 snapshot of PCBs and input device firmware
Parts:
- removed REF**: WEEE-Logo_4.2x6mm_SilkScreen, Symbol:WEEE-Logo_4.2x6mm_SilkScreen
- added H5: MountingHole, MountingHole:MountingHole_2.2mm_M2, F.Cu at (113.0, 106.5)
- added H6: MountingHole, MountingHole:MountingHole_2.2mm_M2, F.Cu at (159.0, 106.5)
- added H7: MountingHole, MountingHole:MountingHole_2.2mm_M2, F.Cu at (113.0, 140.5)
- added H8: MountingHole, MountingHole:MountingHole_2.2mm_M2, F.Cu at (159.0, 140.5)
- added H9: LOGO, footprints:mnt-minilogo, F.Cu at (113.2, 120.0)
- J1: footprint Connector_Molex:Molex_Nano-Fit_105309-xx05_1x05_P2.50mm_Vertical -> Connector_Molex:Molex_Pico-Lock_504050-0591_1x05-1MP_P1.50mm_Horizontal
- moved J1 5.93 mm to (179.2, 120.0), turned to 270 degrees
- moved H1 3.50 mm to (113.0, 100.5)
- moved H2 3.50 mm to (159.0, 100.5)
- moved H3 3.50 mm to (113.0, 134.5)
- moved H4 3.50 mm to (159.0, 134.5)
Connections:
- U1 pad 1: Net-(J1-Pad4) -> Net-(J1-Pad2)
- U1 pad 2: Net-(J1-Pad4) -> Net-(J1-Pad2)
- U1 pad 3: Net-(J1-Pad4) -> Net-(J1-Pad2)
- U1 pad 4: Net-(J1-Pad5) -> Net-(J1-Pad1)
- U1 pad 5: Net-(J1-Pad5) -> Net-(J1-Pad1)
- U1 pad 6: Net-(J1-Pad5) -> Net-(J1-Pad1)
- U2 pad 4: Net-(J1-Pad4) -> Net-(J1-Pad2)
- U2 pad 5: Net-(J1-Pad4) -> Net-(J1-Pad2)
- U2 pad 6: Net-(J1-Pad4) -> Net-(J1-Pad2)
- U3 pad 1: Net-(J1-Pad2) -> Net-(J1-Pad4)
- U3 pad 2: Net-(J1-Pad2) -> Net-(J1-Pad4)
- U3 pad 3: Net-(J1-Pad2) -> Net-(J1-Pad4)
- U4 pad 1: Net-(J1-Pad1) -> Net-(J1-Pad5)
- U4 pad 2: Net-(J1-Pad1) -> Net-(J1-Pad5)
- U4 pad 3: Net-(J1-Pad1) -> Net-(J1-Pad5)
- U4 pad 4: Net-(J1-Pad2) -> Net-(J1-Pad4)
- U4 pad 5: Net-(J1-Pad2) -> Net-(J1-Pad4)
- U4 pad 6: Net-(J1-Pad2) -> Net-(J1-Pad4)
Routing:
- net Net-(J1-Pad2): track 70.7 -> 131.2 mm
- net Net-(J1-Pad1): track 45.4 -> 102.7 mm
- net Net-(J1-Pad5): track 102.4 -> 52.8 mm
- net Net-(J1-Pad4): track 122.8 -> 82.5 mm
- net Net-(J1-Pad3): track 95.3 -> 97.2 mm
Other:
- board size 91 x 65.5 mm -> 91 x 66 mm
- board text added: "MNT REFORM 2.0D-3 BATTERIES 2020-02-26 MNTRE.COM"
- board text removed: "MNT Reform Battery Board D-2 2019-11-09 MNT Research GmbH"

Commit message: WIP battery pack now CERN-OHL-S 2.0
Other:
- board text added: "MNT REFORM 2.0D-3 BATTERIES 2020-02-26 MNTRE.COM MNT RESEARCH GMBH LICENSE: CERN-OHL-S 2.0"
- board text removed: "MNT REFORM 2.0D-3 BATTERIES 2020-02-26 MNTRE.COM"
Changed lines of the file:
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@@
-(kicad_pcb (version 20171130) (host pcbnew 5.1.2+dfsg1-1)
+(kicad_pcb (version 20171130) (host pcbnew 5.1.5+dfsg1-2+b1)
   (general
     (thickness 1.6)
@@
   (gr_line (start 113.75 97) (end 113.75 87.5) (layer Edge.Cuts) (width 0.05))
   (gr_line (start 112.25 87.5) (end 112.25 97) (layer Edge.Cuts) (width 0.05))
-  (gr_text "MNT REFORM 2.0D-3 BATTERIES\n2020-02-26 MNTRE.COM" (at 136 133 90) (layer F.SilkS)
+  (gr_text "MNT REFORM 2.0D-3 BATTERIES\n2020-02-26 MNTRE.COM\nMNT RESEARCH GMBH\nLICENSE: CERN-OHL-S 2.0" (at 136 133 90) (layer F.SilkS)
     (effects (font (size 1 1) (thickness 0.15) italic) (justify left))
   )
@@
   (gr_line (start 95.5 153.5) (end 95.5 87.5) (layer Edge.Cuts) (width 0.05))
   (gr_line (start 95.5 87.5) (end 112.25 87.5) (layer Edge.Cuts) (width 0.05))
-  (segment (start 104 92.95) (end 101.46 90.41) (width 1) (layer F.Cu) (net 5))
-  (segment (start 104 98.03) (end 104 92.95) (width 1) (layer F.Cu) (net 5))
-  (segment (start 104 98.03) (end 98.92 98.03) (width 1) (layer F.Cu) (net 5))
+  (segment (start 168 98) (end 173.08 98) (width 1) (layer F.Cu) (net 1))
+  (segment (start 173.08 92.92) (end 170.54 90.38) (width 1) (layer F.Cu) (net 1))
+  (segment (start 173.08 98) (end 173.08 92.92) (width 1) (layer F.Cu) (net 1))
+  (segment (start 173.08 103.33) (end 173.08 97.5) (width 1) (layer F.Cu) (net 1))
+  (segment (start 180.125 110.375) (end 173.08 103.33) (width 1) (layer F.Cu) (net 1))
+  (segment (start 182.625 110.375) (end 180.125 110.375) (width 1) (layer F.Cu) (net 1))
+  (segment (start 184.75 112.5) (end 182.625 110.375) (width 1) (layer F.Cu) (net 1))
+  (segment (start 184.75 121.25) (end 184.75 112.5) (width 1) (layer F.Cu) (net 1))
+  (segment (start 176.455 123) (end 183 123) (width 1) (layer F.Cu) (net 1))
+  (segment (start 183 123) (end 184.75 121.25) (width 1) (layer F.Cu) (net 1))
+  (segment (start 168 147.8) (end 170.54 150.34) (width 1) (layer F.Cu) (net 2))
+  (segment (start 168 142.72) (end 168 147.8) (width 1) (layer F.Cu) (net 2))
+  (segment (start 168 142.72) (end 173.08 142.72) (width 1) (layer F.Cu) (net 2))
+  (segment (start 168 132) (end 168 142.72) (width 1) (layer F.Cu) (net 2))
+  (segment (start 166 130) (end 168 132) (width 1) (layer F.Cu) (net 2))
+  (segment (start 157 130) (end 166 130) (width 1) (layer F.Cu) (net 2))
+  (segment (start 153.625 133.375) (end 157 130) (width 1) (layer F.Cu) (net 2))
+  (segment (start 144.92 147.83) (end 144.92 142.75) (width 1) (layer F.Cu) (net 2))
+  (segment (start 144.92 142.75) (end 150 142.75) (width 1) (layer F.Cu) (net 2))
+  (segment (start 150 142.75) (end 153.625 139.125) (width 1) (layer F.Cu) (net 2))
+  (segment (start 147.46 150.37) (end 144.92 147.83) (width 1) (layer F.Cu) (net 2))
+  (segment (start 153.625 139.125) (end 153.625 133.375) (width 1) (layer F.Cu) (net 2))
+  (segment (start 168 125.25) (end 168 132) (width 1) (layer F.Cu) (net 2))
+  (segment (start 176.455 121.5) (end 171.75 121.5) (width 1) (layer F.Cu) (net 2))
+  (segment (start 171.75 121.5) (end 168 125.25) (width 1) (layer F.Cu) (net 2))
+  (segment (start 150 92.95) (end 147.46 90.41) (width 1) (layer F.Cu) (net 3))
+  (segment (start 150 98.03) (end 150 92.95) (width 1) (layer F.Cu) (net 3))
+  (segment (start 127.08 92.92) (end 124.54 90.38) (width 1) (layer F.Cu) (net 3))
+  (segment (start 127.08 98) (end 127.08 92.92) (width 1) (layer F.Cu) (net 3))
+  (segment (start 127.08 98) (end 122 98) (width 1) (layer F.Cu) (net 3))
+  (segment (start 141.45 101.5) (end 144.92 98.03) (width 1) (layer F.Cu) (net 3))
+  (segment (start 144.92 98.03) (end 150 98.03) (width 1) (layer F.Cu) (net 3))
+  (segment (start 127.08 98) (end 130.58 101.5) (width 1) (layer F.Cu) (net 3))
+  (segment (start 130.58 101.5) (end 141.45 101.5) (width 1) (layer F.Cu) (net 3))
+  (segment (start 177.75 120) (end 178.75 119) (width 1) (layer F.Cu) (net 3))
+  (segment (start 176.455 120) (end 177.75 120) (width 1) (layer F.Cu) (net 3))
+  (segment (start 178.75 119) (end 178.75 115.75) (width 1) (layer F.Cu) (net 3))
+  (segment (start 178.75 115.75) (end 175.75 112.75) (width 1) (layer F.Cu) (net 3))
+  (segment (start 150 109) (end 150 97.53) (width 1) (layer F.Cu) (net 3))
+  (segment (start 175.75 112.75) (end 153.75 112.75) (width 1) (layer F.Cu) (net 3))
+  (segment (start 153.75 112.75) (end 150 109) (width 1) (layer F.Cu) (net 3))
   (segment (start 122 147.8) (end 124.54 150.34) (width 1) (layer F.Cu) (net 4))
   (segment (start 122 142.72) (end 122 147.8) (width 1) (layer F.Cu) (net 4))
@@
   (segment (start 119.5 130) (end 110 130) (width 1) (layer F.Cu) (net 4))
   (segment (start 110 130) (end 106.5 133.5) (width 1) (layer F.Cu) (net 4))
-  (segment (start 150 92.95) (end 147.46 90.41) (width 1) (layer F.Cu) (net 3))
-  (segment (start 150 98.03) (end 150 92.95) (width 1) (layer F.Cu) (net 3))
-  (segment (start 127.08 92.92) (end 124.54 90.38) (width 1) (layer F.Cu) (net 3))
-  (segment (start 127.08 98) (end 127.08 92.92) (width 1) (layer F.Cu) (net 3))
-  (segment (start 127.08 98) (end 122 98) (width 1) (layer F.Cu) (net 3))
-  (segment (start 141.45 101.5) (end 144.92 98.03) (width 1) (layer F.Cu) (net 3))
-  (segment (start 144.92 98.03) (end 150 98.03) (width 1) (layer F.Cu) (net 3))
-  (segment (start 127.08 98) (end 130.58 101.5) (width 1) (layer F.Cu) (net 3))
-  (segment (start 130.58 101.5) (end 141.45 101.5) (width 1) (layer F.Cu) (net 3))
-  (segment (start 168 147.8) (end 170.54 150.34) (width 1) (layer F.Cu) (net 2))
-  (segment (start 168 142.72) (end 168 147.8) (width 1) (layer F.Cu) (net 2))
-  (segment (start 168 142.72) (end 173.08 142.72) (width 1) (layer F.Cu) (net 2))
-  (segment (start 168 132) (end 168 142.72) (width 1) (layer F.Cu) (net 2))
-  (segment (start 166 130) (end 168 132) (width 1) (layer F.Cu) (net 2))
-  (segment (start 157 130) (end 166 130) (width 1) (layer F.Cu) (net 2))
-  (segment (start 153.625 133.375) (end 157 130) (width 1) (layer F.Cu) (net 2))
-  (segment (start 144.92 147.83) (end 144.92 142.75) (width 1) (layer F.Cu) (net 2))
-  (segment (start 144.92 142.75) (end 150 142.75) (width 1) (layer F.Cu) (net 2))
-  (segment (start 150 142.75) (end 153.625 139.125) (width 1) (layer F.Cu) (net 2))
-  (segment (start 147.46 150.37) (end 144.92 147.83) (width 1) (layer F.Cu) (net 2))
-  (segment (start 153.625 139.125) (end 153.625 133.375) (width 1) (layer F.Cu) (net 2))
-  (segment (start 168 98) (end 173.08 98) (width 1) (layer F.Cu) (net 1))
-  (segment (start 173.08 92.92) (end 170.54 90.38) (width 1) (layer F.Cu) (net 1))
-  (segment (start 173.08 98) (end 173.08 92.92) (width 1) (layer F.Cu) (net 1))
-  (segment (start 173.08 103.33) (end 173.08 97.5) (width 1) (layer F.Cu) (net 1))
-  (segment (start 180.125 110.375) (end 173.08 103.33) (width 1) (layer F.Cu) (net 1))
-  (segment (start 182.625 110.375) (end 180.125 110.375) (width 1) (layer F.Cu) (net 1))
-  (segment (start 184.75 112.5) (end 182.625 110.375) (width 1) (layer F.Cu) (net 1))
-  (segment (start 184.75 121.25) (end 184.75 112.5) (width 1) (layer F.Cu) (net 1))
-  (segment (start 176.455 123) (end 183 123) (width 1) (layer F.Cu) (net 1))
-  (segment (start 183 123) (end 184.75 121.25) (width 1) (layer F.Cu) (net 1))
-  (segment (start 168 125.25) (end 168 132) (width 1) (layer F.Cu) (net 2))
-  (segment (start 176.455 121.5) (end 171.75 121.5) (width 1) (layer F.Cu) (net 2))
-  (segment (start 171.75 121.5) (end 168 125.25) (width 1) (layer F.Cu) (net 2))
-  (segment (start 177.75 120) (end 178.75 119) (width 1) (layer F.Cu) (net 3))
-  (segment (start 176.455 120) (end 177.75 120) (width 1) (layer F.Cu) (net 3))
-  (segment (start 178.75 119) (end 178.75 115.75) (width 1) (layer F.Cu) (net 3))
-  (segment (start 178.75 115.75) (end 175.75 112.75) (width 1) (layer F.Cu) (net 3))
-  (segment (start 150 109) (end 150 97.53) (width 1) (layer F.Cu) (net 3))
-  (segment (start 175.75 112.75) (end 153.75 112.75) (width 1) (layer F.Cu) (net 3))
-  (segment (start 153.75 112.75) (end 150 109) (width 1) (layer F.Cu) (net 3))
   (segment (start 122 126) (end 122 132.5) (width 1) (layer F.Cu) (net 4))
   (segment (start 176.455 118.5) (end 129.5 118.5) (width 1) (layer F.Cu) (net 4))
   (segment (start 129.5 118.5) (end 122 126) (width 1) (layer F.Cu) (net 4))
+  (segment (start 104 92.95) (end 101.46 90.41) (width 1) (layer F.Cu) (net 5))
+  (segment (start 104 98.03) (end 104 92.95) (width 1) (layer F.Cu) (net 5))
+  (segment (start 104 98.03) (end 98.92 98.03) (width 1) (layer F.Cu) (net 5))
   (segment (start 176.455 117) (end 174.955 115.5) (width 1) (layer F.Cu) (net 5))
   (segment (start 104 112) (end 104 97.53) (width 1) (layer F.Cu) (net 5))
