File: reform2-batterypack/reform2-batterypack.sch (KiCad schematic (older format))
At the start: 9 parts, among them J1 Conn_01x05_Female, U1 KEYSTONE_54, U2 KEYSTONE_54, U3 KEYSTONE_54, U4 KEYSTONE_54

Commit message: Reform2.0D-3 snapshot of PCBs and input device firmware
Parts:
- added H5, H6, H7, H8: MountingHole, MountingHole:MountingHole_2.2mm_M2, symbol Mechanical:MountingHole
- added H9: LOGO, footprints:mnt-minilogo, symbol Mechanical:MountingHole
- J1: footprint Connector_Molex:Molex_Nano-Fit_105309-xx05_1x05_P2.50mm_Vertical -> Connector_Molex:Molex_Pico-Lock_504050-0591_1x05-1MP_P1.50mm_Horizontal; Manufacturer (none) -> Molex; Manufacturer_No (none) -> 504050-0591
- U1, U2, U3, U4: Manufacturer (none) -> Keystone; Manufacturer_No (none) -> 54
Connections:
- net at U4.1 (+), U4.2 (+), U4.3 (+): now also J1.5 (Pin_5); no longer J1.1 (Pin_1)
- net at U3.1 (+), U3.2 (+), U3.3 (+)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: now also J1.4 (Pin_4); no longer J1.2 (Pin_2)
- net at U1.1 (+), U1.2 (+), U1.3 (+)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: now also J1.2 (Pin_2); no longer J1.4 (Pin_4)
- net at U1.4 (-), U1.5 (-), U1.6 (-): now also J1.1 (Pin_1); no longer J1.5 (Pin_5)
Other:
- note added: "Connector pinout is\nflipped in respect to\nmotherboard pinout!"
Changed lines of the file:
@@
 F 2 "reform2-batterypack:Keystone54" H 3450 2850 50  0001 C CNN
 F 3 "" H 3450 2850 50  0001 C CNN
+F 4 "Keystone" H 3450 2850 50  0001 C CNN "Manufacturer"
+F 5 "54" H 3450 2850 50  0001 C CNN "Manufacturer_No"
 	1    3450 2850
 	1    0    0    -1
@@
 F 2 "reform2-batterypack:Keystone54" H 3900 2850 50  0001 C CNN
 F 3 "" H 3900 2850 50  0001 C CNN
+F 4 "Keystone" H 3900 2850 50  0001 C CNN "Manufacturer"
+F 5 "54" H 3900 2850 50  0001 C CNN "Manufacturer_No"
 	1    3900 2850
 	1    0    0    -1
@@
 F 2 "reform2-batterypack:Keystone54" H 4350 2850 50  0001 C CNN
 F 3 "" H 4350 2850 50  0001 C CNN
+F 4 "Keystone" H 4350 2850 50  0001 C CNN "Manufacturer"
+F 5 "54" H 4350 2850 50  0001 C CNN "Manufacturer_No"
 	1    4350 2850
 	1    0    0    -1
@@
 F 2 "reform2-batterypack:Keystone54" H 3000 2850 50  0001 C CNN
 F 3 "" H 3000 2850 50  0001 C CNN
+F 4 "Keystone" H 3000 2850 50  0001 C CNN "Manufacturer"
+F 5 "54" H 3000 2850 50  0001 C CNN "Manufacturer_No"
 	1    3000 2850
 	1    0    0    -1
@@
 F 0 "J1" V 3638 1162 50  0000 R CNN
 F 1 "Conn_01x05_Female" V 3547 1162 50  0000 R CNN
-F 2 "Connector_Molex:Molex_Nano-Fit_105309-xx05_1x05_P2.50mm_Vertical" H 3700 1550 50  0001 C CNN
+F 2 "Connector_Molex:Molex_Pico-Lock_504050-0591_1x05-1MP_P1.50mm_Horizontal" H 3700 1550 50  0001 C CNN
 F 3 "~" H 3700 1550 50  0001 C CNN
+F 4 "Molex" H 3700 1550 50  0001 C CNN "Manufacturer"
+F 5 "504050-0591" H 3700 1550 50  0001 C CNN "Manufacturer_No"
 	1    3700 1550
-	0    1    -1   0
+	0    -1   -1   0
 $EndComp
 Wire Wire Line
@@
 Wire Wire Line
 	3900 1750 3900 2000
+$Comp
+L Mechanical:MountingHole H5
+U 1 1 5E649298
+P 1750 3000
+F 0 "H5" H 1850 3046 50  0000 L CNN
+F 1 "MountingHole" H 1850 2955 50  0000 L CNN
+F 2 "MountingHole:MountingHole_2.2mm_M2" H 1750 3000 50  0001 C CNN
+F 3 "~" H 1750 3000 50  0001 C CNN
+	1    1750 3000
+	1    0    0    -1
+$EndComp
+$Comp
+L Mechanical:MountingHole H6
+U 1 1 5E6492A2
+P 1750 3200
+F 0 "H6" H 1850 3246 50  0000 L CNN
+F 1 "MountingHole" H 1850 3155 50  0000 L CNN
+F 2 "MountingHole:MountingHole_2.2mm_M2" H 1750 3200 50  0001 C CNN
+F 3 "~" H 1750 3200 50  0001 C CNN
+	1    1750 3200
+	1    0    0    -1
+$EndComp
+$Comp
+L Mechanical:MountingHole H7
+U 1 1 5E6492AC
+P 1750 3400
+F 0 "H7" H 1850 3446 50  0000 L CNN
+F 1 "MountingHole" H 1850 3355 50  0000 L CNN
+F 2 "MountingHole:MountingHole_2.2mm_M2" H 1750 3400 50  0001 C CNN
+F 3 "~" H 1750 3400 50  0001 C CNN
+	1    1750 3400
+	1    0    0    -1
+$EndComp
+$Comp
+L Mechanical:MountingHole H8
+U 1 1 5E6492B6
+P 1750 3600
+F 0 "H8" H 1850 3646 50  0000 L CNN
+F 1 "MountingHole" H 1850 3555 50  0000 L CNN
+F 2 "MountingHole:MountingHole_2.2mm_M2" H 1750 3600 50  0001 C CNN
+F 3 "~" H 1750 3600 50  0001 C CNN
+	1    1750 3600
+	1    0    0    -1
+$EndComp
+Text Notes 3350 1400 0    50   ~ 0
+Connector pinout is\nflipped in respect to\nmotherboard pinout!
+$Comp
+L Mechanical:MountingHole H9
+U 1 1 5E56D901
+P 1750 1300
+F 0 "H9" H 1850 1346 50  0000 L CNN
+F 1 "LOGO" H 1850 1255 50  0000 L CNN
+F 2 "footprints:mnt-minilogo" H 1750 1300 50  0001 C CNN
+F 3 "~" H 1750 1300 50  0001 C CNN
+	1    1750 1300
+	1    0    0    -1
+$EndComp
 $EndSCHEMATC
