File: reform2-trackball-sensor-pcb/reform2-trackball-sensor.sch (KiCad schematic (older format))
At the start: 8 parts, among them J1 Conn_01x05_Male, U1 PAT9125EL

Commit message: Reform2.0D-3 snapshot of PCBs and input device firmware
Parts:
- added H3, H4, H5, H6: MountingHole, MountingHole:MountingHole_2.2mm_M2, symbol Mechanical:MountingHole
- added H7, H8: LOGO, footprints:mnt-minilogo, symbol Mechanical:MountingHole
- C1: MFR Generic -> TDK; MFR_NO Generic 1uF 0603 5V -> C1608X8L1C105K080AC
- C2: MFR Generic -> Yageo; MFR_NO Generic 0.1uF 0603 5V -> CC0603JPX7R9BB104
- C3: MFR Generic -> Taiyo Yuden; MFR_NO Generic 10uF 0603 5V -> LMK107BBJ106KALT
- J1: value Conn_01x05_Male -> Conn_01x06_Male; footprint Connector_PinHeader_2.54mm:PinHeader_1x05_P2.54mm_Horizontal -> Connector_FFC-FPC:Hirose_FH12-6S-0.5SH_1x06-1MP_P0.50mm_Horizontal; symbol Connector:Conn_01x05_Male -> Connector:Conn_01x06_Male; MFR NOSTUFF -> Hirose; MFR_NO NOSTUFF -> FH12-6S-0.5SH(55)
Connections:
- net +3V3: now also J1.1 (Pin_1); no longer J1.5 (Pin_5)
- net GND: now also J1.6 (Pin_6); no longer J1.1 (Pin_1)
- net MOTION: now also J1.5 (Pin_5); no longer J1.2 (Pin_2)
- net SCL: now also J1.3 (Pin_3); no longer J1.4 (Pin_4)
- net SDA: now also J1.4 (Pin_4); no longer J1.3 (Pin_3)
- no-connect marks 1 -> 2
Other:
- moved on the sheet: R1
Changed lines of the file:
@@
 	4950 3700 5100 3700
-$Comp
-L Connector:Conn_01x05_Male J1
-U 1 1 5D1E2C79
-P 7000 3600
-F 0 "J1" H 6972 3624 50  0000 R CNN
-F 1 "Conn_01x05_Male" H 6972 3533 50  0000 R CNN
-F 2 "Connector_PinHeader_2.54mm:PinHeader_1x05_P2.54mm_Horizontal" H 7000 3600 50  0001 C CNN
-F 3 "~" H 7000 3600 50  0001 C CNN
-F 4 "NOSTUFF" H 7000 3600 50  0001 C CNN "MFR"
-F 5 "NOSTUFF" H 7000 3600 50  0001 C CNN "MFR_NO"
-	1    7000 3600
-	-1   0    0    -1
-$EndComp
 $Comp
 L power:+3V3 #PWR0102
 U 1 1 5D1E3F38
-P 3850 3350
-F 0 "#PWR0102" H 3850 3200 50  0001 C CNN
-F 1 "+3V3" H 3865 3523 50  0000 C CNN
-F 2 "" H 3850 3350 50  0001 C CNN
-F 3 "" H 3850 3350 50  0001 C CNN
-	1    3850 3350
+P 3850 3200
+F 0 "#PWR0102" H 3850 3050 50  0001 C CNN
+F 1 "+3V3" H 3865 3373 50  0000 C CNN
+F 2 "" H 3850 3200 50  0001 C CNN
+F 3 "" H 3850 3200 50  0001 C CNN
+	1    3850 3200
 	1    0    0    -1
 $EndComp
@@
 	5100 3400 3850 3400
 Wire Wire Line
-	3850 3400 3850 3350
-Wire Wire Line
 	5100 3600 4200 3600
-Wire Wire Line
-	3850 3600 3850 3400
-Connection ~ 3850 3400
 $Comp
 L Device:C_Small C1
@@
 F 2 "Capacitor_SMD:C_0603_1608Metric" H 3850 3700 50  0001 C CNN
 F 3 "~" H 3850 3700 50  0001 C CNN
-F 4 "Generic" H 3850 3700 50  0001 C CNN "MFR"
-F 5 "Generic 1uF 0603 5V" H 3850 3700 50  0001 C CNN "MFR_NO"
+F 4 "TDK" H 3850 3700 50  0001 C CNN "MFR"
+F 5 "C1608X8L1C105K080AC" H 3850 3700 50  0001 C CNN "MFR_NO"
 	1    3850 3700
 	1    0    0    -1
@@
 F 2 "Capacitor_SMD:C_0603_1608Metric" H 4200 3700 50  0001 C CNN
 F 3 "~" H 4200 3700 50  0001 C CNN
-F 4 "Generic" H 4200 3700 50  0001 C CNN "MFR"
-F 5 "Generic 0.1uF 0603 5V" H 4200 3700 50  0001 C CNN "MFR_NO"
+F 4 "Yageo" H 4200 3700 50  0001 C CNN "MFR"
+F 5 "CC0603JPX7R9BB104" H 4200 3700 50  0001 C CNN "MFR_NO"
 	1    4200 3700
 	1    0    0    -1
@@
 F 2 "Capacitor_SMD:C_0603_1608Metric" H 4600 3600 50  0001 C CNN
 F 3 "~" H 4600 3600 50  0001 C CNN
-F 4 "Generic" H 4600 3600 50  0001 C CNN "MFR"
-F 5 "Generic 10uF 0603 5V" H 4600 3600 50  0001 C CNN "MFR_NO"
+F 4 "Taiyo Yuden" H 4600 3600 50  0001 C CNN "MFR"
+F 5 "LMK107BBJ106KALT" H 4600 3600 50  0001 C CNN "MFR_NO"
 	1    4600 3600
 	1    0    0    -1
@@
 L Device:R_Small R1
 U 1 1 5D1E6137
-P 6200 3400
-F 0 "R1" V 6004 3400 50  0000 C CNN
-F 1 "0" V 6095 3400 50  0000 C CNN
-F 2 "Resistor_SMD:R_0603_1608Metric" H 6200 3400 50  0001 C CNN
-F 3 "~" H 6200 3400 50  0001 C CNN
-F 4 "NOSTUFF" H 6200 3400 50  0001 C CNN "MFR"
-F 5 "NOSTUFF" H 6200 3400 50  0001 C CNN "MFR_NO"
-	1    6200 3400
+P 6250 3000
+F 0 "R1" V 6054 3000 50  0000 C CNN
+F 1 "0" V 6145 3000 50  0000 C CNN
+F 2 "Resistor_SMD:R_0603_1608Metric" H 6250 3000 50  0001 C CNN
+F 3 "~" H 6250 3000 50  0001 C CNN
+F 4 "NOSTUFF" H 6250 3000 50  0001 C CNN "MFR"
+F 5 "NOSTUFF" H 6250 3000 50  0001 C CNN "MFR_NO"
+	1    6250 3000
 	0    1    1    0
 $EndComp
-Text Label 6450 3500 0    50   ~ 0
-MOTION
-Text Label 6450 3600 0    50   ~ 0
+Text Label 6500 3600 0    50   ~ 0
 SDA
-Text Label 6450 3700 0    50   ~ 0
+Text Label 6500 3700 0    50   ~ 0
 SCL
-Wire Wire Line
-	6800 3600 6100 3600
-Wire Wire Line
-	6100 3700 6800 3700
-Wire Wire Line
-	6800 3500 6100 3500
 $Comp
 L power:GND #PWR0103
 U 1 1 5D1E79D9
-P 6350 3850
-F 0 "#PWR0103" H 6350 3600 50  0001 C CNN
-F 1 "GND" H 6355 3677 50  0000 C CNN
-F 2 "" H 6350 3850 50  0001 C CNN
-F 3 "" H 6350 3850 50  0001 C CNN
-	1    6350 3850
-	1    0    0    -1
-$EndComp
-$Comp
-L power:+3V3 #PWR0104
-U 1 1 5D1E8452
-P 6800 3800
-F 0 "#PWR0104" H 6800 3650 50  0001 C CNN
-F 1 "+3V3" V 6815 3928 50  0000 L CNN
-F 2 "" H 6800 3800 50  0001 C CNN
-F 3 "" H 6800 3800 50  0001 C CNN
-	1    6800 3800
-	0    -1   -1   0
-$EndComp
-Wire Wire Line
-	6300 3400 6350 3400
-Wire Wire Line
-	6350 3400 6350 3850
+P 6400 3050
+F 0 "#PWR0103" H 6400 2800 50  0001 C CNN
+F 1 "GND" H 6405 2877 50  0000 C CNN
+F 2 "" H 6400 3050 50  0001 C CNN
+F 3 "" H 6400 3050 50  0001 C CNN
+	1    6400 3050
+	1    0    0    -1
+$EndComp
 $Comp
 L power:GND #PWR0105
 U 1 1 5D1F19B7
-P 6750 3300
-F 0 "#PWR0105" H 6750 3050 50  0001 C CNN
-F 1 "GND" V 6755 3172 50  0000 R CNN
-F 2 "" H 6750 3300 50  0001 C CNN
-F 3 "" H 6750 3300 50  0001 C CNN
-	1    6750 3300
+P 6450 3400
+F 0 "#PWR0105" H 6450 3150 50  0001 C CNN
+F 1 "GND" V 6455 3272 50  0000 R CNN
+F 2 "" H 6450 3400 50  0001 C CNN
+F 3 "" H 6450 3400 50  0001 C CNN
+	1    6450 3400
 	0    1    1    0
 $EndComp
-Wire Wire Line
-	6750 3300 6750 3400
-Wire Wire Line
-	6750 3400 6800 3400
 $Comp
 L Mechanical:MountingHole H1
@@
 	1    0    0    -1
 $EndComp
+$Comp
+L Connector:Conn_01x06_Male J1
+U 1 1 5D1E2C79
+P 7000 3700
+F 0 "J1" H 6972 3724 50  0000 R CNN
+F 1 "Conn_01x06_Male" H 6972 3633 50  0000 R CNN
+F 2 "Connector_FFC-FPC:Hirose_FH12-6S-0.5SH_1x06-1MP_P0.50mm_Horizontal" H 7000 3700 50  0001 C CNN
+F 3 "~" H 7000 3700 50  0001 C CNN
+F 4 "Hirose" H 7000 3700 50  0001 C CNN "MFR"
+F 5 "FH12-6S-0.5SH(55)" H 7000 3700 50  0001 C CNN "MFR_NO"
+	1    7000 3700
+	-1   0    0    1
+$EndComp
+$Comp
+L power:+3V3 #PWR0104
+U 1 1 5D1E8452
+P 6450 3900
+F 0 "#PWR0104" H 6450 3750 50  0001 C CNN
+F 1 "+3V3" V 6465 4028 50  0000 L CNN
+F 2 "" H 6450 3900 50  0001 C CNN
+F 3 "" H 6450 3900 50  0001 C CNN
+	1    6450 3900
+	0    -1   -1   0
+$EndComp
+NoConn ~ 6800 3800
+Text Label 6500 3500 0    50   ~ 0
+MOTION
+Wire Wire Line
+	6400 3050 6400 3000
+Wire Wire Line
+	6400 3000 6350 3000
+Wire Wire Line
+	6100 3400 6100 3000
+Wire Wire Line
+	6100 3000 6150 3000
+Wire Wire Line
+	6100 3700 6800 3700
+Wire Wire Line
+	6100 3600 6800 3600
+Wire Wire Line
+	6100 3500 6800 3500
+Wire Wire Line
+	6450 3400 6750 3400
+Wire Wire Line
+	6450 3900 6750 3900
+$Comp
+L power:PWR_FLAG #FLG0101
+U 1 1 5E567A57
+P 6750 3900
+F 0 "#FLG0101" H 6750 3975 50  0001 C CNN
+F 1 "PWR_FLAG" V 6750 4027 50  0000 L CNN
+F 2 "" H 6750 3900 50  0001 C CNN
+F 3 "~" H 6750 3900 50  0001 C CNN
+	1    6750 3900
+	-1   0    0    1
+$EndComp
+Connection ~ 6750 3900
+Wire Wire Line
+	6750 3900 6800 3900
+Wire Wire Line
+	3850 3200 3850 3400
+Connection ~ 3850 3400
+Wire Wire Line
+	3850 3400 3850 3600
+$Comp
+L power:PWR_FLAG #FLG0102
+U 1 1 5E568ABF
+P 6750 3400
+F 0 "#FLG0102" H 6750 3475 50  0001 C CNN
+F 1 "PWR_FLAG" H 6750 3573 50  0000 C CNN
+F 2 "" H 6750 3400 50  0001 C CNN
+F 3 "~" H 6750 3400 50  0001 C CNN
+	1    6750 3400
+	1    0    0    -1
+$EndComp
+Connection ~ 6750 3400
+Wire Wire Line
+	6750 3400 6800 3400
+$Comp
+L Mechanical:MountingHole H3
+U 1 1 5E56B94C
+P 4100 5350
+F 0 "H3" H 4200 5396 50  0000 L CNN
+F 1 "MountingHole" H 4200 5305 50  0000 L CNN
+F 2 "MountingHole:MountingHole_2.2mm_M2" H 4100 5350 50  0001 C CNN
+F 3 "~" H 4100 5350 50  0001 C CNN
+F 4 "NOSTUFF" H 4100 5350 50  0001 C CNN "MFR"
+F 5 "NOSTUFF" H 4100 5350 50  0001 C CNN "MFR_NO"
+	1    4100 5350
+	1    0    0    -1
+$EndComp
+$Comp
+L Mechanical:MountingHole H4
+U 1 1 5E56B958
+P 4100 5650
+F 0 "H4" H 4200 5696 50  0000 L CNN
+F 1 "MountingHole" H 4200 5605 50  0000 L CNN
+F 2 "MountingHole:MountingHole_2.2mm_M2" H 4100 5650 50  0001 C CNN
+F 3 "~" H 4100 5650 50  0001 C CNN
+F 4 "NOSTUFF" H 4100 5650 50  0001 C CNN "MFR"
+F 5 "NOSTUFF" H 4100 5650 50  0001 C CNN "MFR_NO"
+	1    4100 5650
+	1    0    0    -1
+$EndComp
+$Comp
+L Mechanical:MountingHole H5
+U 1 1 5E56C467
+P 5000 4700
+F 0 "H5" H 5100 4746 50  0000 L CNN
+F 1 "MountingHole" H 5100 4655 50  0000 L CNN
+F 2 "MountingHole:MountingHole_2.2mm_M2" H 5000 4700 50  0001 C CNN
+F 3 "~" H 5000 4700 50  0001 C CNN
+F 4 "NOSTUFF" H 5000 4700 50  0001 C CNN "MFR"
+F 5 "NOSTUFF" H 5000 4700 50  0001 C CNN "MFR_NO"
+	1    5000 4700
+	1    0    0    -1
+$EndComp
+$Comp
+L Mechanical:MountingHole H6
+U 1 1 5E56C473
+P 5000 5000
+F 0 "H6" H 5100 5046 50  0000 L CNN
+F 1 "MountingHole" H 5100 4955 50  0000 L CNN
+F 2 "MountingHole:MountingHole_2.2mm_M2" H 5000 5000 50  0001 C CNN
+F 3 "~" H 5000 5000 50  0001 C CNN
+F 4 "NOSTUFF" H 5000 5000 50  0001 C CNN "MFR"
+F 5 "NOSTUFF" H 5000 5000 50  0001 C CNN "MFR_NO"
+	1    5000 5000
+	1    0    0    -1
+$EndComp
+$Comp
+L Mechanical:MountingHole H7
+U 1 1 5E56C47F
+P 4100 6300
+F 0 "H7" H 4200 6346 50  0000 L CNN
+F 1 "LOGO" H 4200 6255 50  0000 L CNN
+F 2 "footprints:mnt-minilogo" H 4100 6300 50  0001 C CNN
+F 3 "~" H 4100 6300 50  0001 C CNN
+F 4 "NOSTUFF" H 4100 6300 50  0001 C CNN "MFR"
+F 5 "NOSTUFF" H 4100 6300 50  0001 C CNN "MFR_NO"
+	1    4100 6300
+	1    0    0    -1
+$EndComp
+$Comp
+L Mechanical:MountingHole H8
+U 1 1 5E56C48B
+P 4100 6600
+F 0 "H8" H 4200 6646 50  0000 L CNN
+F 1 "LOGO" H 4200 6555 50  0000 L CNN
+F 2 "footprints:mnt-minilogo" H 4100 6600 50  0001 C CNN
+F 3 "~" H 4100 6600 50  0001 C CNN
+F 4 "NOSTUFF" H 4100 6600 50  0001 C CNN "MFR"
+F 5 "NOSTUFF" H 4100 6600 50  0001 C CNN "MFR_NO"
+	1    4100 6600
+	1    0    0    -1
+$EndComp
