File: reform2-motherboard-pcb/reform2-power.sch (KiCad schematic (older format))
At the start: 200 parts, among them J1 Jack-DC, J13 BATCON1, J2 BATCON2, J22 LPC_IO, J23 KDBSYSCTL, J8 USB_B_Micro, Q1 Si7850DP, Q10 PMV50EPEAR, Q11 PMV50EPEAR, Q12 PMV50EPEAR, Q13 PMV50ENEA, Q14 PMV50ENEA, Q15 Si7850DP, Q17 Si7850DP, Q18 Si7461DP, Q2 Si7850DP, Q3 Si7461DP, Q4 PMV50ENEA, Q5 PMV50EPEAR, Q6 PMV50EPEAR, Q7 PMV50EPEAR, Q8 PMV50EPEAR, Q9 PMV50EPEAR, SW1 SW_DIP_x01, SW2 SW_Push, U12 LM2677SX-3.3, U13 TLV62568DBV, U14 LMR16006YQ3, U17 TLV1117-18, U18 LPC11U24FBD48-301, U19 TLV62568DBV, U2 LTC4020EUHFPBF, U4 LTC6803-4, U5 PCF8523T, U6 INA260, U7 LM2677SX-5, Y2 12MHz, Y4 32.768 kHz

Commit message: motherboard: r-1 release snapshot
Parts:
- added R100, R98: 0, Resistor_SMD:R_0603_1608Metric, symbol Device:R_Small
- C1, C129, C130, C145, C146, C32, C4, C5: Manufacturer_No UMK107AB7105KA-T -> UMK107BJ105KA-T
- D13: Distributor (none) -> Mouser; Manufacturer (none) -> Vishay; Manufacturer_No (none) -> SMAJ36CA-E3/5A
- D3, D4, D6: Manufacturer_No SBR0560S1 -> SBR0560S1-7
- D5: Manufacturer_No RBR3MM60ATF -> RBR3MM60ATFTR
- J8: footprint Connector_USB:USB_Micro-B_Molex-105017-0001 -> footprints:WE_629105136821; Manufacturer Molex -> Wuerth; Manufacturer_No 105017-0001 -> 629105136821
- Q13, Q14, Q4: value PMV50ENEA -> PMV50ENEAR; Distributor (none) -> Mouser; Manufacturer (none) -> Nexperia; Manufacturer_No (none) -> PMV50ENEAR
- R34: Manufacturer_No CRCW0603100KJNEAC -> CRCW0603150KFKEAC
- R95: Manufacturer Vishay Dale -> Yageo; Manufacturer_No CRCW0603100KJNEAC -> RC0603FR-0710KL
Connections:
- net +3V3: now also R100.2; no longer C129.1, U17.3 (VI)
- new net: C129.1, R100.1, R98.1, U17.3 (VI)
- new net 3V3_PWR_AUX: R98.2
Changed lines of the file:
@@
 Sheet 9 9
 Title "MNT Reform 2 Power System"
-Date "2020-05-19"
-Rev "2.0D-4"
+Date "2020-09-24"
+Rev "2.0R-1"
 Comp "MNT Research GmbH"
 Comment1 "https://mntre.com"
@@
 F 0 "J8" H 15070 8039 50  0000 R CNN
 F 1 "USB_B_Micro" H 15070 7948 50  0000 R CNN
-F 2 "Connector_USB:USB_Micro-B_Molex-105017-0001" H 15450 8000 50  0001 C CNN
+F 2 "footprints:WE_629105136821" H 15450 8000 50  0001 C CNN
 F 3 "~" H 15450 8000 50  0001 C CNN
-F 4 "Molex" H 15300 8050 50  0001 C CNN "Manufacturer"
-F 5 "105017-0001" H 15300 8050 50  0001 C CNN "Manufacturer_No"
+F 4 "Wuerth" H 15300 8050 50  0001 C CNN "Manufacturer"
+F 5 "629105136821" H 15300 8050 50  0001 C CNN "Manufacturer_No"
 F 6 "y" H 15300 8050 50  0001 C CNN "Checked"
 F 7 "Mouser" H 15300 8050 50  0001 C CNN "Distributor"
@@
 L power:+3V3 #PWR068
 U 1 1 5EB4EB3E
-P 10300 3100
-F 0 "#PWR068" H 10300 2950 50  0001 C CNN
-F 1 "+3V3" H 10315 3273 50  0000 C CNN
-F 2 "" H 10300 3100 50  0001 C CNN
-F 3 "" H 10300 3100 50  0001 C CNN
-	1    10300 3100
+P 10300 2850
+F 0 "#PWR068" H 10300 2700 50  0001 C CNN
+F 1 "+3V3" H 10315 3023 50  0000 C CNN
+F 2 "" H 10300 2850 50  0001 C CNN
+F 3 "" H 10300 2850 50  0001 C CNN
+	1    10300 2850
 	1    0    0    -1
 $EndComp
@@
 F 2 "Capacitor_SMD:C_0603_1608Metric" H 10300 3300 50  0001 C CNN
 F 3 "~" H 10300 3300 50  0001 C CNN
-F 4 "UMK107AB7105KA-T" H 10300 3300 50  0001 C CNN "Manufacturer_No"
+F 4 "UMK107BJ105KA-T" H 10300 3300 50  0001 C CNN "Manufacturer_No"
 F 5 "Taiyo Yuden" H 10300 3300 50  0001 C CNN "Manufacturer"
 F 6 "y" H 10300 3300 50  0001 C CNN "Checked"
@@
 $EndComp
 Wire Wire Line
-	10300 3200 10700 3200
+	10300 3200 10550 3200
 Wire Wire Line
 	10300 3100 10300 3200
@@
 F 2 "Capacitor_SMD:C_0603_1608Metric" H 11500 3300 50  0001 C CNN
 F 3 "~" H 11500 3300 50  0001 C CNN
-F 4 "UMK107AB7105KA-T" H 11500 3300 50  0001 C CNN "Manufacturer_No"
+F 4 "UMK107BJ105KA-T" H 11500 3300 50  0001 C CNN "Manufacturer_No"
 F 5 "Taiyo Yuden" H 11500 3300 50  0001 C CNN "Manufacturer"
 F 6 "y" H 11500 3300 50  0001 C CNN "Checked"
@@
 F 3 "" H 11600 1950 50  0001 C CNN
 F 4 "Diodes, Inc." H 11600 1950 50  0001 C CNN "Manufacturer"
-F 5 "SBR0560S1" H 11600 1950 50  0001 C CNN "Manufacturer_No"
+F 5 "SBR0560S1-7" H 11600 1950 50  0001 C CNN "Manufacturer_No"
 F 6 "y" H 11600 1950 50  0001 C CNN "Checked"
 F 7 "Mouser" H 11600 1950 50  0001 C CNN "Distributor"
@@
 F 2 "Capacitor_SMD:C_0603_1608Metric" H 5350 7450 50  0001 C CNN
 F 3 "~" H 5350 7450 50  0001 C CNN
-F 4 "UMK107AB7105KA-T" H 5350 7450 50  0001 C CNN "Manufacturer_No"
+F 4 "UMK107BJ105KA-T" H 5350 7450 50  0001 C CNN "Manufacturer_No"
 F 5 "Taiyo Yuden" H 5350 7450 50  0001 C CNN "Manufacturer"
 F 6 "y" H 5350 7450 50  0001 C CNN "Checked"
@@
 F 2 "Capacitor_SMD:C_0603_1608Metric" H 5650 7450 50  0001 C CNN
 F 3 "~" H 5650 7450 50  0001 C CNN
-F 4 "UMK107AB7105KA-T" H 5650 7450 50  0001 C CNN "Manufacturer_No"
+F 4 "UMK107BJ105KA-T" H 5650 7450 50  0001 C CNN "Manufacturer_No"
 F 5 "Taiyo Yuden" H 5650 7450 50  0001 C CNN "Manufacturer"
 F 6 "y" H 5650 7450 50  0001 C CNN "Checked"
@@
 F 3 "~" H 4050 4800 50  0001 C CNN
 F 4 "Taiyo Yuden" H 4050 4800 50  0001 C CNN "Manufacturer"
-F 5 "UMK107AB7105KA-T" H 4050 4800 50  0001 C CNN "Manufacturer_No"
+F 5 "UMK107BJ105KA-T" H 4050 4800 50  0001 C CNN "Manufacturer_No"
 F 6 "y" H 4050 4800 50  0001 C CNN "Checked"
 F 7 "Mouser" H 4050 4800 50  0001 C CNN "Distributor"
@@
 F 4 "y" H 3450 4800 50  0001 C CNN "Checked"
 F 5 "Diodes, Inc." H 3450 4800 50  0001 C CNN "Manufacturer"
-F 6 "SBR0560S1" H 3450 4800 50  0001 C CNN "Manufacturer_No"
+F 6 "SBR0560S1-7" H 3450 4800 50  0001 C CNN "Manufacturer_No"
 F 7 "Mouser" H 3450 4800 50  0001 C CNN "Distributor"
 	1    3450 4800
@@
 F 4 "y" H 2200 4900 50  0001 C CNN "Checked"
 F 5 "Diodes, Inc." H 2200 4900 50  0001 C CNN "Manufacturer"
-F 6 "SBR0560S1" H 2200 4900 50  0001 C CNN "Manufacturer_No"
+F 6 "SBR0560S1-7" H 2200 4900 50  0001 C CNN "Manufacturer_No"
 F 7 "Mouser" H 2200 4900 50  0001 C CNN "Distributor"
 	1    2200 4900
@@
 F 3 "~" H 1850 5050 50  0001 C CNN
 F 4 "Taiyo Yuden" H 1850 5050 50  0001 C CNN "Manufacturer"
-F 5 "UMK107AB7105KA-T" H 1850 5050 50  0001 C CNN "Manufacturer_No"
+F 5 "UMK107BJ105KA-T" H 1850 5050 50  0001 C CNN "Manufacturer_No"
 F 6 "y" H 1850 5050 50  0001 C CNN "Checked"
 F 7 "Mouser" H 1850 5050 50  0001 C CNN "Distributor"
@@
 F 4 "ROHM" H 3000 2600 50  0001 C CNN "Manufacturer"
 F 5 "y" H 3000 2600 50  0001 C CNN "Checked"
-F 6 "RBR3MM60ATF" H 3000 2600 50  0001 C CNN "Manufacturer_No"
+F 6 "RBR3MM60ATFTR" H 3000 2600 50  0001 C CNN "Manufacturer_No"
 F 7 "Mouser" H 3000 2600 50  0001 C CNN "Distributor"
 	1    3000 2600
@@
 F 3 "~" H 6300 1500 50  0001 C CNN
 F 4 "Taiyo Yuden" H 6300 1500 50  0001 C CNN "Manufacturer"
-F 5 "UMK107AB7105KA-T" H 6300 1500 50  0001 C CNN "Manufacturer_No"
+F 5 "UMK107BJ105KA-T" H 6300 1500 50  0001 C CNN "Manufacturer_No"
 F 6 "y" H 6300 1500 50  0001 C CNN "Checked"
 F 7 "Mouser" H 6300 1500 50  0001 C CNN "Distributor"
@@
 F 3 "~" H 6150 2950 50  0001 C CNN
 F 4 "Taiyo Yuden" H 6150 2950 50  0001 C CNN "Manufacturer"
-F 5 "UMK107AB7105KA-T" H 6150 2950 50  0001 C CNN "Manufacturer_No"
+F 5 "UMK107BJ105KA-T" H 6150 2950 50  0001 C CNN "Manufacturer_No"
 F 6 "y" H 6150 2950 50  0001 C CNN "Checked"
 F 7 "Mouser" H 6150 2950 50  0001 C CNN "Distributor"
@@
 U 1 1 5FD6C758
 P 1150 5750
-F 0 "R34" H 1300 5700 50  0000 R CNN
+F 0 "R34" H 1350 5700 50  0000 R CNN
 F 1 "150k" H 1400 5800 50  0000 R CNN
 F 2 "Resistor_SMD:R_0603_1608Metric" H 1150 5750 50  0001 C CNN
@@
 F 5 "Mouser" H 1150 5750 50  0001 C CNN "Distributor"
 F 6 "Vishay Dale" H 1150 5750 50  0001 C CNN "Manufacturer"
-F 7 "CRCW0603100KJNEAC" H 1150 5750 50  0001 C CNN "Manufacturer_No"
+F 7 "CRCW0603150KFKEAC" H 1150 5750 50  0001 C CNN "Manufacturer_No"
 	1    1150 5750
 	-1   0    0    1
@@
 P 6800 2050
 F 0 "Q13" H 7000 2000 50  0000 L CNN
-F 1 "PMV50ENEA" H 7000 1900 50  0000 L CNN
+F 1 "PMV50ENEAR" H 7000 1900 50  0000 L CNN
 F 2 "Package_TO_SOT_SMD:SOT-23" H 7000 1975 50  0001 L CIN
 F 3 "http://www.diodes.com/assets/Datasheets/ds30376.pdf" H 6800 2050 50  0001 L CNN
+F 4 "Mouser" H 6800 2050 50  0001 C CNN "Distributor"
+F 5 "Nexperia" H 6800 2050 50  0001 C CNN "Manufacturer"
+F 6 "PMV50ENEAR" H 6800 2050 50  0001 C CNN "Manufacturer_No"
 	1    6800 2050
 	1    0    0    -1
@@
 P 6800 3450
 F 0 "Q14" H 7000 3400 50  0000 L CNN
-F 1 "PMV50ENEA" H 7000 3300 50  0000 L CNN
+F 1 "PMV50ENEAR" H 7000 3300 50  0000 L CNN
 F 2 "Package_TO_SOT_SMD:SOT-23" H 7000 3375 50  0001 L CIN
 F 3 "http://www.diodes.com/assets/Datasheets/ds30376.pdf" H 6800 3450 50  0001 L CNN
+F 4 "Mouser" H 6800 3450 50  0001 C CNN "Distributor"
+F 5 "Nexperia" H 6800 3450 50  0001 C CNN "Manufacturer"
+F 6 "PMV50ENEAR" H 6800 3450 50  0001 C CNN "Manufacturer_No"
 	1    6800 3450
 	1    0    0    -1
@@
 P 1950 7700
 F 0 "Q4" H 2150 7650 50  0000 L CNN
-F 1 "PMV50ENEA" H 2150 7550 50  0000 L CNN
+F 1 "PMV50ENEAR" H 2150 7550 50  0000 L CNN
 F 2 "Package_TO_SOT_SMD:SOT-23" H 2150 7625 50  0001 L CIN
 F 3 "http://www.diodes.com/assets/Datasheets/ds30376.pdf" H 1950 7700 50  0001 L CNN
+F 4 "Mouser" H 1950 7700 50  0001 C CNN "Distributor"
+F 5 "Nexperia" H 1950 7700 50  0001 C CNN "Manufacturer"
+F 6 "PMV50ENEAR" H 1950 7700 50  0001 C CNN "Manufacturer_No"
 	1    1950 7700
 	1    0    0    -1
@@
 F 2 "Resistor_SMD:R_0603_1608Metric" H 1700 7900 50  0001 C CNN
 F 3 "~" H 1700 7900 50  0001 C CNN
-F 4 "Vishay Dale" H 1700 7900 50  0001 C CNN "Manufacturer"
-F 5 "CRCW0603100KJNEAC" H 1700 7900 50  0001 C CNN "Manufacturer_No"
+F 4 "Yageo" H 1700 7900 50  0001 C CNN "Manufacturer"
+F 5 "RC0603FR-0710KL" H 1700 7900 50  0001 C CNN "Manufacturer_No"
 F 6 "y" H 1700 7900 50  0001 C CNN "Checked"
 F 7 "Mouser" H 1700 7900 50  0001 C CNN "Distributor"
@@
 F 2 "Diode_SMD:D_SMA" H 2250 1000 50  0001 C CNN
 F 3 "~" H 2250 1000 50  0001 C CNN
+F 4 "Mouser" H 2250 1000 50  0001 C CNN "Distributor"
+F 5 "Vishay" H 2250 1000 50  0001 C CNN "Manufacturer"
+F 6 "SMAJ36CA-E3/5A" H 2250 1000 50  0001 C CNN "Manufacturer_No"
 	1    2250 1000
 	0    1    1    0
@@
 Text Label 11500 8350 0    50   ~ 0
 LPC_~USBCON
+Text GLabel 10050 2850 1    50   Input ~ 0
+3V3_PWR_AUX
+$Comp
+L Device:R_Small R100
+U 1 1 5FC3EA3F
+P 10300 3000
+F 0 "R100" V 10400 2950 50  0000 C CNN
+F 1 "0" V 10300 3000 50  0000 C CNN
+F 2 "Resistor_SMD:R_0603_1608Metric" H 10300 3000 50  0001 C CNN
+F 3 "~" H 10300 3000 50  0001 C CNN
+F 4 "Vishay Dale" H 10300 3000 50  0001 C CNN "Manufacturer"
+F 5 "CRCW06030000Z0EAC" H 10300 3000 50  0001 C CNN "Manufacturer_No"
+F 6 "Mouser" H 10300 3000 50  0001 C CNN "Distributor"
+F 7 "y" H 10300 3000 50  0001 C CNN "Checked"
+F 8 "y" H 10300 3000 50  0001 C CNN "DNP"
+	1    10300 3000
+	-1   0    0    1
+$EndComp
+Wire Wire Line
+	10300 2850 10300 2900
+$Comp
+L Device:R_Small R98
+U 1 1 5FD8D200
+P 10050 3000
+F 0 "R98" V 10150 2950 50  0000 C CNN
+F 1 "0" V 10050 3000 50  0000 C CNN
+F 2 "Resistor_SMD:R_0603_1608Metric" H 10050 3000 50  0001 C CNN
+F 3 "~" H 10050 3000 50  0001 C CNN
+F 4 "Vishay Dale" H 10050 3000 50  0001 C CNN "Manufacturer"
+F 5 "CRCW06030000Z0EAC" H 10050 3000 50  0001 C CNN "Manufacturer_No"
+F 6 "Mouser" H 10050 3000 50  0001 C CNN "Distributor"
+F 7 "y" H 10050 3000 50  0001 C CNN "Checked"
+	1    10050 3000
+	-1   0    0    1
+$EndComp
+Wire Wire Line
+	10050 2850 10050 2900
+Wire Wire Line
+	10050 3100 10050 3200
+Wire Wire Line
+	10050 3200 10300 3200
+$Comp
+L power:PWR_FLAG #FLG02
+U 1 1 5FEDE4E5
+P 10550 3200
+F 0 "#FLG02" H 10550 3275 50  0001 C CNN
+F 1 "PWR_FLAG" H 10550 3373 50  0000 C CNN
+F 2 "" H 10550 3200 50  0001 C CNN
+F 3 "~" H 10550 3200 50  0001 C CNN
+	1    10550 3200
+	1    0    0    -1
+$EndComp
+Connection ~ 10550 3200
+Wire Wire Line
+	10550 3200 10700 3200
+Text Notes 10200 3100 0    50   ~ 0
+NOSTUFF
 $EndSCHEMATC

Commit message: reform2-motherboard: schematics,PCB,BOM,models for R-2C (probably final)
Parts:
- C16, C17: value 220uF -> 100uF
- D13, Q13, Q14, Q4: Checked (none) -> y
- J8: Manufacturer Wuerth -> Wurth
- SW2: footprint Button_Switch_SMD:SW_Push_1P1T_NO_CK_KMR2 -> footprints:UK-B0206-G3.8-250-JZ; Manufacturer C&K -> USAKRO; Manufacturer_No KMR221GLFS -> UK-B0206-G3.8-250-JZ
Connections:
- net LPC_AD5: now also J22.7 (Pin_7); no longer J22.2 (Pin_2)
- net LPC_AD7: now also J22.10 (Pin_10); no longer J22.13 (Pin_13)
- net LPC_MISO1a: now also J22.2 (Pin_2); no longer J22.8 (Pin_8)
- net LPC_MOSI1a: now also J22.14 (Pin_14); no longer J22.11 (Pin_11)
- net LPC_RXDa: now also J22.12 (Pin_12); no longer J22.6 (Pin_6)
- net LPC_SCK0b: now also J22.1 (Pin_1); no longer J22.10 (Pin_10)
- net LPC_SCLKa: now also J22.9 (Pin_9); no longer J22.14 (Pin_14)
- net LPC_SWDIO: now also J22.8 (Pin_8); no longer J22.1 (Pin_1)
- net LPC_TDI: now also J22.4 (Pin_4); no longer J22.9 (Pin_9)
- net LPC_TDO: now also J22.6 (Pin_6); no longer J22.5 (Pin_5)
- net LPC_TMS: now also J22.3 (Pin_3); no longer J22.7 (Pin_7)
- net LPC_TXDa: now also J22.11 (Pin_11); no longer J22.4 (Pin_4)
- net LPC_~TRST: now also J22.5 (Pin_5); no longer J22.3 (Pin_3)
- net LPC_~USBCON: now also J22.13 (Pin_13); no longer J22.12 (Pin_12)
Other:
- note added: "These values are\ncopied from the\ndatasheet and should\nbe verified with a VNA"
- note removed: "These values are\ncargoculted from the\nmanual and should\nbe verified with a VNA"
Changed lines of the file:
@@
 Sheet 9 9
 Title "MNT Reform 2 Power System"
-Date "2020-09-24"
-Rev "2.0R-1"
+Date "2020-10-29"
+Rev "2.0R-2C"
 Comp "MNT Research GmbH"
 Comment1 "https://mntre.com"
@@
 P 5950 1550
 F 0 "C16" H 6042 1596 50  0000 L CNN
-F 1 "220uF" H 6042 1505 50  0000 L CNN
+F 1 "100uF" H 6042 1505 50  0000 L CNN
 F 2 "Capacitor_SMD:CP_Elec_8x10" H 5950 1550 50  0001 C CNN
 F 3 "~" H 5950 1550 50  0001 C CNN
@@
 P 5700 2950
 F 0 "C17" H 5792 2996 50  0000 L CNN
-F 1 "220uF" H 5792 2905 50  0000 L CNN
+F 1 "100uF" H 5792 2905 50  0000 L CNN
 F 2 "Capacitor_SMD:CP_Elec_8x10" H 5700 2950 50  0001 C CNN
 F 3 "~" H 5700 2950 50  0001 C CNN
@@
 F 0 "SW2" H 11450 6535 50  0000 C CNN
 F 1 "SW_Push" H 11450 6444 50  0000 C CNN
-F 2 "Button_Switch_SMD:SW_Push_1P1T_NO_CK_KMR2" H 11450 6450 50  0001 C CNN
+F 2 "footprints:UK-B0206-G3.8-250-JZ" H 11450 6450 50  0001 C CNN
 F 3 "~" H 11450 6450 50  0001 C CNN
-F 4 "C&K" H 11450 6250 50  0001 C CNN "Manufacturer"
-F 5 "KMR221GLFS" H 11450 6250 50  0001 C CNN "Manufacturer_No"
+F 4 "USAKRO" H 11450 6250 50  0001 C CNN "Manufacturer"
+F 5 "UK-B0206-G3.8-250-JZ" H 11450 6250 50  0001 C CNN "Manufacturer_No"
 F 6 "y" H 11450 6250 50  0001 C CNN "Checked"
 F 7 "Mouser" H 11450 6250 50  0001 C CNN "Distributor"
@@
 F 2 "footprints:WE_629105136821" H 15450 8000 50  0001 C CNN
 F 3 "~" H 15450 8000 50  0001 C CNN
-F 4 "Wuerth" H 15300 8050 50  0001 C CNN "Manufacturer"
+F 4 "Wurth" H 15300 8050 50  0001 C CNN "Manufacturer"
 F 5 "629105136821" H 15300 8050 50  0001 C CNN "Manufacturer_No"
 F 6 "y" H 15300 8050 50  0001 C CNN "Checked"
@@
 Text Label 12050 7250 0    50   ~ 0
 LPC_SCK0a
-Text Label 12050 8450 0    50   ~ 0
+Text Label 11500 7850 0    50   ~ 0
 LPC_MISO1a
 Text Label 12050 8550 0    50   ~ 0
@@
 LPC_UART2_TX
 Wire Wire Line
-	11500 7850 12550 7850
-Wire Wire Line
-	10950 7750 10950 7850
-Wire Wire Line
-	10950 7850 11000 7850
-Wire Wire Line
-	10900 7650 10900 7950
-Wire Wire Line
-	10900 7950 11000 7950
-Wire Wire Line
-	10900 7650 12550 7650
-Wire Wire Line
-	10850 7550 10850 8050
-Wire Wire Line
-	10850 8050 11000 8050
-Wire Wire Line
-	10850 7550 12550 7550
-Wire Wire Line
-	10800 7450 10800 8150
-Wire Wire Line
-	10800 8150 11000 8150
-Wire Wire Line
-	10800 7450 12550 7450
-Wire Wire Line
-	10750 7350 10750 8250
-Wire Wire Line
-	10750 8250 11000 8250
-Wire Wire Line
-	10750 7350 12550 7350
-Wire Wire Line
-	10950 8350 11000 8350
-Wire Wire Line
 	14050 6550 13950 6550
 Text Label 14050 7250 0    50   ~ 0
@@
 Text Label 11350 4300 0    50   ~ 0
 LPC_TXDc
-Text Label 11500 8250 0    50   ~ 0
+Text Label 11000 7850 2    50   ~ 0
 LPC_SCK0b
 Wire Wire Line
-	12000 8450 12000 8150
-Wire Wire Line
-	12000 8150 11500 8150
-Wire Wire Line
 	12050 8550 12550 8550
-Text Label 10950 8450 2    50   ~ 0
+Text Label 11500 8250 0    50   ~ 0
 LPC_AD7
 Wire Wire Line
-	10950 8450 11000 8450
-Wire Wire Line
-	12000 8450 12550 8450
-Wire Wire Line
 	12050 8350 12550 8350
 Wire Wire Line
-	10950 8550 11000 8550
-Wire Wire Line
 	11500 8550 11600 8550
 Wire Wire Line
@@
 Text Label 11350 4200 0    50   ~ 0
 LPC_VCC
-Text Label 10950 8550 2    50   ~ 0
+Text Label 11000 8550 2    50   ~ 0
 LPC_VCC
 Wire Wire Line
@@
 $EndComp
 Text Notes 4700 4850 0    50   ~ 0
-These values are\ncargoculted from the\nmanual and should\nbe verified with a VNA
+These values are\ncopied from the\ndatasheet and should\nbe verified with a VNA
 Wire Wire Line
 	3350 7900 3250 7900
@@
 Wire Wire Line
 	9850 4150 9850 4250
-Wire Wire Line
-	10950 7750 12550 7750
 $Comp
 L Connector_Generic:Conn_02x08_Odd_Even J22
 U 1 1 61E919B8
 P 11200 8150
-F 0 "J22" H 11250 7300 50  0000 C CNN
-F 1 "LPC_IO" H 11250 7450 50  0000 C CNN
+F 0 "J22" H 11250 7500 50  0000 C CNN
+F 1 "LPC_IO" H 11250 7600 50  0000 C CNN
 F 2 "Connector_PinHeader_2.54mm:PinHeader_2x08_P2.54mm_Vertical" H 11200 8150 50  0001 C CNN
 F 3 "~" H 11200 8150 50  0001 C CNN
@@
 	1    0    0    -1
 $EndComp
-Text Label 11500 8050 0    50   ~ 0
+Text Label 11500 8350 0    50   ~ 0
 LPC_RXDa
-Text Label 11500 7950 0    50   ~ 0
+Text Label 11000 8350 2    50   ~ 0
 LPC_TXDa
 Wire Wire Line
@@
 Text Notes 14550 6650 0    50   ~ 0
 EN_1V2!
-Text Label 10950 8350 2    50   ~ 0
+Text Label 11500 8450 0    50   ~ 0
 LPC_MOSI1a
 Text Label 15200 9500 0    50   ~ 0
@@
 Wire Wire Line
 	1300 2150 1300 4300
-Text Label 11500 8450 0    50   ~ 0
+Text Label 11000 8250 2    50   ~ 0
 LPC_SCLKa
 $Comp
@@
 F 5 "Nexperia" H 6800 2050 50  0001 C CNN "Manufacturer"
 F 6 "PMV50ENEAR" H 6800 2050 50  0001 C CNN "Manufacturer_No"
+F 7 "y" H 6800 2050 50  0001 C CNN "Checked"
 	1    6800 2050
 	1    0    0    -1
@@
 F 5 "Nexperia" H 6800 3450 50  0001 C CNN "Manufacturer"
 F 6 "PMV50ENEAR" H 6800 3450 50  0001 C CNN "Manufacturer_No"
+F 7 "y" H 6800 3450 50  0001 C CNN "Checked"
 	1    6800 3450
 	1    0    0    -1
@@
 F 5 "Nexperia" H 1950 7700 50  0001 C CNN "Manufacturer"
 F 6 "PMV50ENEAR" H 1950 7700 50  0001 C CNN "Manufacturer_No"
+F 7 "y" H 1950 7700 50  0001 C CNN "Checked"
 	1    1950 7700
 	1    0    0    -1
@@
 F 5 "Vishay" H 2250 1000 50  0001 C CNN "Manufacturer"
 F 6 "SMAJ36CA-E3/5A" H 2250 1000 50  0001 C CNN "Manufacturer_No"
+F 7 "y" H 2250 1000 50  0001 C CNN "Checked"
 	1    2250 1000
 	0    1    1    0
@@
 Text Label 12050 6850 0    50   ~ 0
 LPC_~USBCON
-Text Label 11500 8350 0    50   ~ 0
+Text Label 11000 8450 2    50   ~ 0
 LPC_~USBCON
 Text GLabel 10050 2850 1    50   Input ~ 0
@@
 Text Notes 10200 3100 0    50   ~ 0
 NOSTUFF
+Wire Wire Line
+	12550 7750 12050 7750
+Wire Wire Line
+	12050 7650 12550 7650
+Wire Wire Line
+	12550 7550 12050 7550
+Wire Wire Line
+	12050 7450 12550 7450
+Wire Wire Line
+	12550 7350 12050 7350
+Wire Wire Line
+	12050 7850 12550 7850
+Wire Wire Line
+	12550 8450 12050 8450
+Text Label 11000 7950 2    50   ~ 0
+LPC_TMS
+Text Label 11500 7950 0    50   ~ 0
+LPC_TDI
+Text Label 11000 8050 2    50   ~ 0
+LPC_~TRST
+Text Label 11500 8050 0    50   ~ 0
+LPC_TDO
+Text Label 11000 8150 2    50   ~ 0
+LPC_AD5
+Text Label 11500 8150 0    50   ~ 0
+LPC_SWDIO
+Text Label 12050 8450 0    50   ~ 0
+LPC_MISO1a
 $EndSCHEMATC
