File: reform2-keyboard-pcb/reform-kbd-mcu.sch (KiCad schematic (older format))
At the start: 13 parts, among them J1 RST, J2 USB, J3 AUX, U1 ATMEGA32U4-AU, Y1 16MHz

Commit message: WIP reform2 kbd: restructure switches, led, finer placement, some routing
Parts:
- removed J1: RST, Pin_Headers:Pin_Header_Straight_1x02_Pitch2.00mm, symbol Connector_Generic:Conn_01x02
- removed J3: AUX, Pin_Headers:Pin_Header_Straight_1x05_Pitch2.00mm, symbol Connector_Generic:Conn_01x05
- added D83: LED_Small, LED_SMD:LED_0603_1608Metric_Pad1.05x0.95mm_HandSolder, symbol Device:LED_Small
- added GFX1, GFX2: MNT, reform2-keyboard:mntreform, symbol Mechanical:MountingHole
- added H1: MH1, MountingHole:MountingHole_2.2mm_M2_Pad, symbol Mechanical:MountingHole_Pad
- added H2: MH2, MountingHole:MountingHole_2.2mm_M2_Pad, symbol Mechanical:MountingHole_Pad
- added H3: MH3, MountingHole:MountingHole_2.2mm_M2_Pad, symbol Mechanical:MountingHole_Pad
- added H4: MH4, MountingHole:MountingHole_2.2mm_M2_Pad, symbol Mechanical:MountingHole_Pad
- added J1: UART, Connector_PinHeader_2.00mm:PinHeader_1x04_P2.00mm_Horizontal, symbol Connector_Generic:Conn_01x04
- added J3: POWERCONN, Connector_PinHeader_2.54mm:PinHeader_1x03_P2.54mm_Horizontal, symbol Connector:Conn_01x03_Male
- added R4: 0, Resistor_SMD:R_0603_1608Metric_Pad1.05x0.95mm_HandSolder, symbol Device:R_Small
- added R5: 330, Resistor_SMD:R_0603_1608Metric_Pad1.05x0.95mm_HandSolder, symbol Device:R_Small
- added SW90: POWER, Button_Switch_THT:SW_E-Switch_EG1271_DPDT, symbol Switch:SW_DPDT_x2
- added SW91: RESET, Button_Switch_SMD:SW_Push_1P1T_NO_CK_KMR2, symbol Switch:SW_SPST
- added SW92: SW_DIP_x02, Button_Switch_SMD:SW_DIP_SPSTx02_Slide_Omron_A6S-210x_W8.9mm_P2.54mm, symbol Switch:SW_DIP_x02
- added U2: SM351LT, Package_TO_SOT_SMD:SOT-23, symbol Sensor_Magnetic:SM351LT
- C1, C2, C3, C4: footprint Capacitors_SMD:C_0603_HandSoldering -> Capacitor_SMD:C_0603_1608Metric_Pad1.05x0.95mm_HandSolder
- C5: value 1uF -> 0.1uF; footprint Capacitors_SMD:C_0603_HandSoldering -> Capacitor_SMD:C_0603_1608Metric_Pad1.05x0.95mm_HandSolder
- R1, R2, R3: footprint Resistors_SMD:R_0603_HandSoldering -> Resistor_SMD:R_0603_1608Metric_Pad1.05x0.95mm_HandSolder
Connections:
- net labels added: AUX, LED, LID_SENSE, PROG, PWRIN, PWROUT, UART_RX, UART_TX, UD+, UD-
- net labels removed: UVCC
- wire segments 59 -> 68
Other:
- moved on the sheet: C1, C2, C3, C4, C5, J2, R1, R2, R3, Y1

Commit message: WIP reform2 kbd: MCU section routed, removed LED, introduced AUX port
Parts:
- removed D83: LED_Small, LED_SMD:LED_0603_1608Metric_Pad1.05x0.95mm_HandSolder, symbol Device:LED_Small
- removed R5: 330, Resistor_SMD:R_0603_1608Metric_Pad1.05x0.95mm_HandSolder, symbol Device:R_Small
- added J?: AUX, Connector_PinHeader_2.00mm:PinHeader_1x04_P2.00mm_Horizontal, symbol Connector_Generic:Conn_01x04
- added R6, R7: 0, Resistor_SMD:R_0603_1608Metric_Pad1.05x0.95mm_HandSolder, symbol Device:R_Small
- SW92: value SW_DIP_x02 -> SW_DIP_x01; footprint Button_Switch_SMD:SW_DIP_SPSTx02_Slide_Omron_A6S-210x_W8.9mm_P2.54mm -> Button_Switch_SMD:SW_DIP_SPSTx01_Slide_Omron_A6S-110x_W8.9mm_P2.54mm; symbol Switch:SW_DIP_x02 -> Switch:SW_DIP_x01
Connections:
- net labels added: AUX1, AUX2
- net labels removed: AUX, LED
- wire segments 68 -> 67
Other:
- moved on the sheet: SW91
Changed lines of the file:
@@
 	0    1    1    0
 $EndComp
-Wire Wire Line
-	7800 4400 7550 4400
 Text GLabel 6000 4300 0    60   Input ~ 0
 PROG
@@
 L Switch:SW_SPST SW91
 U 1 1 5CF3DA9E
-P 6250 3600
-F 0 "SW91" H 6250 3835 50  0000 C CNN
-F 1 "RESET" H 6250 3744 50  0000 C CNN
-F 2 "Button_Switch_SMD:SW_Push_1P1T_NO_CK_KMR2" H 6250 3600 50  0001 C CNN
-F 3 "~" H 6250 3600 50  0001 C CNN
-	1    6250 3600
-	1    0    0    -1
-$EndComp
-Text GLabel 6000 3600 0    60   Input ~ 0
+P 6350 3700
+F 0 "SW91" H 6350 3935 50  0000 C CNN
+F 1 "RESET" H 6350 3844 50  0000 C CNN
+F 2 "Button_Switch_SMD:SW_Push_1P1T_NO_CK_KMR2" H 6350 3700 50  0001 C CNN
+F 3 "~" H 6350 3700 50  0001 C CNN
+	1    6350 3700
+	1    0    0    -1
+$EndComp
+Text GLabel 6100 3700 0    60   Input ~ 0
 RESET
 Wire Wire Line
-	6000 3600 6050 3600
+	6100 3700 6150 3700
 $Comp
 L power:GND #PWR0103
 U 1 1 5CF3FA6D
-P 6550 3600
-F 0 "#PWR0103" H 6550 3350 50  0001 C CNN
-F 1 "GND" H 6550 3450 50  0000 C CNN
-F 2 "" H 6550 3600 50  0001 C CNN
-F 3 "" H 6550 3600 50  0001 C CNN
-	1    6550 3600
-	1    0    0    -1
-$EndComp
-Wire Wire Line
-	6550 3600 6450 3600
+P 6650 3700
+F 0 "#PWR0103" H 6650 3450 50  0001 C CNN
+F 1 "GND" H 6650 3550 50  0000 C CNN
+F 2 "" H 6650 3700 50  0001 C CNN
+F 3 "" H 6650 3700 50  0001 C CNN
+	1    6650 3700
+	1    0    0    -1
+$EndComp
+Wire Wire Line
+	6650 3700 6550 3700
 Text GLabel 6650 2100 2    60   Input ~ 0
 LID_SENSE
@@
 LID_SENSE
 Text GLabel 4800 3850 2    60   Input ~ 0
-LED
-$Comp
-L Switch:SW_DIP_x02 SW92
+AUX2
+$Comp
+L Switch:SW_DIP_x01 SW92
 U 1 1 5CF54073
 P 6350 4300
-F 0 "SW92" H 6350 4667 50  0000 C CNN
-F 1 "SW_DIP_x02" H 6350 4576 50  0000 C CNN
-F 2 "Button_Switch_SMD:SW_DIP_SPSTx02_Slide_Omron_A6S-210x_W8.9mm_P2.54mm" H 6350 4300 50  0001 C CNN
+F 0 "SW92" H 6350 4600 50  0000 C CNN
+F 1 "SW_DIP_x01" H 6350 4500 50  0000 C CNN
+F 2 "Button_Switch_SMD:SW_DIP_SPSTx01_Slide_Omron_A6S-110x_W8.9mm_P2.54mm" H 6350 4300 50  0001 C CNN
 F 3 "~" H 6350 4300 50  0001 C CNN
 	1    6350 4300
@@
 	6750 4300 6650 4300
 Wire Wire Line
-	6650 4200 6750 4200
-Wire Wire Line
-	6750 4200 6750 4300
-Connection ~ 6750 4300
-Wire Wire Line
-	6000 4200 6050 4200
-Text GLabel 6000 4200 0    60   Input ~ 0
-AUX
-Wire Wire Line
 	6000 4300 6050 4300
 $Comp
@@
 	3350 3950 3600 3950
 Text GLabel 4800 4150 2    60   Input ~ 0
-AUX
+AUX1
 $Comp
 L Connector_Generic:Conn_01x04 J1
@@
 Text Label 3400 4250 0    60   ~ 0
 UD-
-$Comp
-L Device:LED_Small D83
-U 1 1 5CFE699E
-P 6600 5200
-F 0 "D83" H 6600 4995 50  0000 C CNN
-F 1 "LED_Small" H 6600 5086 50  0000 C CNN
-F 2 "LED_SMD:LED_0603_1608Metric_Pad1.05x0.95mm_HandSolder" V 6600 5200 50  0001 C CNN
-F 3 "~" V 6600 5200 50  0001 C CNN
-	1    6600 5200
-	-1   0    0    1
-$EndComp
-Text GLabel 6100 5200 0    60   Input ~ 0
-LED
-$Comp
-L Device:R_Small R5
-U 1 1 5CFE99A4
-P 6250 5200
-F 0 "R5" V 6054 5200 50  0000 C CNN
-F 1 "330" V 6145 5200 50  0000 C CNN
-F 2 "Resistor_SMD:R_0603_1608Metric_Pad1.05x0.95mm_HandSolder" H 6250 5200 50  0001 C CNN
-F 3 "~" H 6250 5200 50  0001 C CNN
-	1    6250 5200
-	0    1    1    0
-$EndComp
-Wire Wire Line
-	6150 5200 6100 5200
-Wire Wire Line
-	6350 5200 6500 5200
-$Comp
-L power:GND #PWR0106
-U 1 1 5CFECA83
-P 6700 5200
-F 0 "#PWR0106" H 6700 4950 50  0001 C CNN
-F 1 "GND" H 6700 5050 50  0000 C CNN
-F 2 "" H 6700 5200 50  0001 C CNN
-F 3 "" H 6700 5200 50  0001 C CNN
-	1    6700 5200
-	0    -1   -1   0
-$EndComp
 Text GLabel 8100 2450 0    60   Input ~ 0
 PWRIN
@@
 Text GLabel 8100 1850 0    60   Input ~ 0
 PWRIN
+$Comp
+L Device:R_Small R6
+U 1 1 5D094D68
+P 7700 4400
+F 0 "R6" H 7730 4420 50  0000 L CNN
+F 1 "0" H 7730 4360 50  0000 L CNN
+F 2 "Resistor_SMD:R_0603_1608Metric_Pad1.05x0.95mm_HandSolder" H 7700 4400 50  0001 C CNN
+F 3 "" H 7700 4400 50  0001 C CNN
+	1    7700 4400
+	0    1    1    0
+$EndComp
+Wire Wire Line
+	7600 4400 7550 4400
+$Comp
+L Device:R_Small R7
+U 1 1 5D0965CF
+P 9750 3150
+F 0 "R7" H 9780 3170 50  0000 L CNN
+F 1 "0" H 9780 3110 50  0000 L CNN
+F 2 "Resistor_SMD:R_0603_1608Metric_Pad1.05x0.95mm_HandSolder" H 9750 3150 50  0001 C CNN
+F 3 "" H 9750 3150 50  0001 C CNN
+	1    9750 3150
+	0    1    1    0
+$EndComp
+Text GLabel 9500 3150 0    60   Input ~ 0
+PWRIN
+Wire Wire Line
+	9500 3150 9650 3150
+$Comp
+L power:+5V #PWR010
+U 1 1 5D097D89
+P 9950 3150
+F 0 "#PWR010" H 9950 3000 50  0001 C CNN
+F 1 "+5V" H 9950 3290 50  0000 C CNN
+F 2 "" H 9950 3150 50  0001 C CNN
+F 3 "" H 9950 3150 50  0001 C CNN
+	1    9950 3150
+	0    1    1    0
+$EndComp
+Wire Wire Line
+	9950 3150 9850 3150
+$Comp
+L Connector_Generic:Conn_01x04 J?
+U 1 1 5D0C1E6C
+P 9600 4300
+F 0 "J?" H 9600 4600 50  0000 C CNN
+F 1 "AUX" H 9600 3900 50  0000 C CNN
+F 2 "Connector_PinHeader_2.00mm:PinHeader_1x04_P2.00mm_Horizontal" H 9600 4300 50  0001 C CNN
+F 3 "" H 9600 4300 50  0001 C CNN
+	1    9600 4300
+	-1   0    0    1
+$EndComp
+$Comp
+L power:+5V #PWR?
+U 1 1 5D0C1E76
+P 10250 4400
+F 0 "#PWR?" H 10250 4250 50  0001 C CNN
+F 1 "+5V" H 10250 4540 50  0000 C CNN
+F 2 "" H 10250 4400 50  0001 C CNN
+F 3 "" H 10250 4400 50  0001 C CNN
+	1    10250 4400
+	0    1    1    0
+$EndComp
+Wire Wire Line
+	10250 4400 9800 4400
+$Comp
+L power:GND #PWR?
+U 1 1 5D0C1E81
+P 10250 4100
+F 0 "#PWR?" H 10250 3850 50  0001 C CNN
+F 1 "GND" H 10250 3950 50  0000 C CNN
+F 2 "" H 10250 4100 50  0001 C CNN
+F 3 "" H 10250 4100 50  0001 C CNN
+	1    10250 4100
+	0    -1   -1   0
+$EndComp
+Wire Wire Line
+	10250 4100 9800 4100
+Text GLabel 9800 4200 2    60   Input ~ 0
+AUX1
+Text GLabel 9800 4300 2    60   Input ~ 0
+AUX2
 $EndSCHEMATC

Commit message: Reform2 Keyboard final prep and snapshot for first prototype manufacturing
Parts:
- gave numbers to parts that had none: 1
Connections:
- wire segments 67 -> 71
- no-connect marks 0 -> 2
Changed lines of the file:
@@
 L power:+5V #PWR08
 U 1 1 5A635C68
-P 4300 2450
-F 0 "#PWR08" H 4300 2300 50  0001 C CNN
-F 1 "+5V" H 4300 2590 50  0000 C CNN
-F 2 "" H 4300 2450 50  0001 C CNN
-F 3 "" H 4300 2450 50  0001 C CNN
-	1    4300 2450
+P 4200 2350
+F 0 "#PWR08" H 4200 2200 50  0001 C CNN
+F 1 "+5V" H 4200 2490 50  0000 C CNN
+F 2 "" H 4200 2350 50  0001 C CNN
+F 3 "" H 4200 2350 50  0001 C CNN
+	1    4200 2350
 	1    0    0    -1
 $EndComp
@@
 	4300 2700 4300 2850
 Wire Wire Line
-	3850 2450 4100 2450
-Connection ~ 4100 2450
-Wire Wire Line
-	4200 2450 4300 2450
-Wire Wire Line
 	3050 4250 3000 4250
 Wire Wire Line
@@
 	3300 3150 3400 3150
 Connection ~ 3400 3150
-Connection ~ 4300 2450
 Wire Wire Line
 	4550 2700 4550 2650
@@
 	4200 2700 4300 2700
 Wire Wire Line
-	4100 2450 4100 2850
-Wire Wire Line
 	4200 2450 4200 2700
 Wire Wire Line
 	3400 3150 3600 3150
-Wire Wire Line
-	4300 2450 4550 2450
 Wire Wire Line
 	2050 3550 2050 3750
@@
 Wire Wire Line
 	3400 2500 3400 2700
-Wire Wire Line
-	4200 2450 4100 2450
 Connection ~ 4200 2450
 $Comp
@@
 $EndComp
 Wire Wire Line
-	7750 3150 8250 3150
+	7750 3150 7800 3150
 $Comp
 L Connector:Conn_01x03_Male J3
@@
 PWRIN
 Wire Wire Line
-	9500 3150 9650 3150
+	9500 3150 9550 3150
 $Comp
 L power:+5V #PWR010
@@
 	0    1    1    0
 $EndComp
-Wire Wire Line
-	9950 3150 9850 3150
-$Comp
-L Connector_Generic:Conn_01x04 J?
+$Comp
+L Connector_Generic:Conn_01x04 J4
 U 1 1 5D0C1E6C
 P 9600 4300
-F 0 "J?" H 9600 4600 50  0000 C CNN
+F 0 "J4" H 9600 4600 50  0000 C CNN
 F 1 "AUX" H 9600 3900 50  0000 C CNN
 F 2 "Connector_PinHeader_2.00mm:PinHeader_1x04_P2.00mm_Horizontal" H 9600 4300 50  0001 C CNN
@@
 $EndComp
 $Comp
-L power:+5V #PWR?
+L power:+5V #PWR0106
 U 1 1 5D0C1E76
 P 10250 4400
-F 0 "#PWR?" H 10250 4250 50  0001 C CNN
+F 0 "#PWR0106" H 10250 4250 50  0001 C CNN
 F 1 "+5V" H 10250 4540 50  0000 C CNN
 F 2 "" H 10250 4400 50  0001 C CNN
@@
 	10250 4400 9800 4400
 $Comp
-L power:GND #PWR?
+L power:GND #PWR0107
 U 1 1 5D0C1E81
 P 10250 4100
-F 0 "#PWR?" H 10250 3850 50  0001 C CNN
+F 0 "#PWR0107" H 10250 3850 50  0001 C CNN
 F 1 "GND" H 10250 3950 50  0000 C CNN
 F 2 "" H 10250 4100 50  0001 C CNN
@@
 Text GLabel 9800 4300 2    60   Input ~ 0
 AUX2
+NoConn ~ 8500 1750
+NoConn ~ 8500 2350
+$Comp
+L power:PWR_FLAG #FLG0101
+U 1 1 5D14B686
+P 9550 3050
+F 0 "#FLG0101" H 9550 3125 50  0001 C CNN
+F 1 "PWR_FLAG" H 9550 3223 50  0000 C CNN
+F 2 "" H 9550 3050 50  0001 C CNN
+F 3 "~" H 9550 3050 50  0001 C CNN
+	1    9550 3050
+	1    0    0    -1
+$EndComp
+$Comp
+L power:PWR_FLAG #FLG0102
+U 1 1 5D14D536
+P 7800 3100
+F 0 "#FLG0102" H 7800 3175 50  0001 C CNN
+F 1 "PWR_FLAG" H 7800 3273 50  0000 C CNN
+F 2 "" H 7800 3100 50  0001 C CNN
+F 3 "~" H 7800 3100 50  0001 C CNN
+	1    7800 3100
+	1    0    0    -1
+$EndComp
+Wire Wire Line
+	7800 3100 7800 3150
+Connection ~ 7800 3150
+Wire Wire Line
+	7800 3150 8250 3150
+Wire Wire Line
+	9850 3150 9950 3150
+Wire Wire Line
+	9550 3050 9550 3150
+Connection ~ 9550 3150
+Wire Wire Line
+	9550 3150 9650 3150
+Wire Wire Line
+	4200 2350 4200 2450
+Wire Wire Line
+	4200 2450 4550 2450
+Wire Wire Line
+	3850 2450 4200 2450
+Wire Wire Line
+	4100 2850 4100 2700
+Wire Wire Line
+	4100 2700 4200 2700
 $EndSCHEMATC

Commit message: reform2.0 d-2 keyboard snapshot
Parts:
- removed J3: POWERCONN, Connector_PinHeader_2.54mm:PinHeader_1x03_P2.54mm_Horizontal, symbol Connector:Conn_01x03_Male
- removed R7: 0, Resistor_SMD:R_0603_1608Metric_Pad1.05x0.95mm_HandSolder, symbol Device:R_Small
- removed SW90: POWER, Button_Switch_THT:SW_E-Switch_EG1271_DPDT, symbol Switch:SW_DPDT_x2
- removed U2: SM351LT, Package_TO_SOT_SMD:SOT-23, symbol Sensor_Magnetic:SM351LT
- added C6: 0.1uF, Capacitor_SMD:C_0603_1608Metric_Pad1.05x0.95mm_HandSolder, symbol Device:C_Small
- added H5: MH5, MountingHole:MountingHole_2.2mm_M2_Pad, symbol Mechanical:MountingHole_Pad
- added H6: MH6, MountingHole:MountingHole_2.2mm_M2_Pad, symbol Mechanical:MountingHole_Pad
- added R5: 4.7k, Resistor_SMD:R_0603_1608Metric, symbol Device:R_Small
- added TP1: TestPoint, TestPoint:TestPoint_Pad_D1.0mm, symbol Connector:TestPoint
- C1, C2: Manufacturer (none) -> Yageo; Manufacturer_No (none) -> CC0603JRNPO9BN180
- C3, C4: Manufacturer (none) -> Taiyo Yuden; Manufacturer_No (none) -> UMK107BJ105KA-T
- C5: Manufacturer (none) -> Yageo; Manufacturer_No (none) -> CC0603JPX7R9BB104
- J1, J2, J4: Manufacturer (none) -> Wurth; Manufacturer_No (none) -> 61300411121
- R1, R2: value 0 -> 22; Manufacturer (none) -> Vishay Dale; Manufacturer_No (none) -> CRCW06030000Z0EAC
- R3: Manufacturer (none) -> Yageo; Manufacturer_No (none) -> AF0603JR-0710KL
- R4: Manufacturer (none) -> Vishay Dale; Manufacturer_No (none) -> CRCW06030000Z0EAC
- R6: value 0 -> 4.7k; footprint Resistor_SMD:R_0603_1608Metric_Pad1.05x0.95mm_HandSolder -> Resistor_SMD:R_0603_1608Metric
- SW91: Manufacturer (none) -> CK; Manufacturer_No (none) -> KMR223NGULCLFG
- SW92: Manufacturer (none) -> Omron; Manufacturer_No (none) -> A6S-1101-H
- U1: Manufacturer (none) -> Microchip; Manufacturer_No (none) -> ATMEGA32U4-AU
- Y1: Manufacturer (none) -> Abracon; Manufacturer_No (none) -> ABM8AIG-16.000MHz-4-T
Connections:
- net labels added: +3V3, AUX, DISP_SCL, DISP_SDA
- net labels removed: AUX1, AUX2, LID_SENSE, PWRIN, PWROUT
- wire segments 71 -> 83
- no-connect marks 2 -> 0
Other:
- note added: "To SSD1306"
- note added: "lid sensor was SM351LT"
- moved on the sheet: C4, C5, GFX1, GFX2, H1, H2, H3, H4, J1, J2, J4, SW91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

Commit message: Reform2.0D-3 snapshot of PCBs and input device firmware
Parts:
- removed TP1: TestPoint, TestPoint:TestPoint_Pad_D1.0mm, symbol Connector:TestPoint
- added J4: USB_C_Receptacle_USB2.0, Connector_USB:USB_C_Receptacle_Amphenol_12401610E4-2A, symbol Connector:USB_C_Receptacle_USB2.0
- added R13, R14: 5.1k, Resistor_SMD:R_0603_1608Metric, symbol Device:R_Small
- C1, C2, C6: footprint Capacitor_SMD:C_0603_1608Metric_Pad1.05x0.95mm_HandSolder -> Capacitor_SMD:C_0603_1608Metric
- C3: footprint Capacitor_SMD:C_0603_1608Metric_Pad1.05x0.95mm_HandSolder -> Capacitor_SMD:C_0603_1608Metric; Manufacturer Taiyo Yuden -> TDK; Manufacturer_No UMK107BJ105KA-T -> C1608X8L1C105K080AC
- C4: renamed from C5; footprint Capacitor_SMD:C_0603_1608Metric_Pad1.05x0.95mm_HandSolder -> Capacitor_SMD:C_0603_1608Metric
- C5: renamed from C4; footprint Capacitor_SMD:C_0603_1608Metric_Pad1.05x0.95mm_HandSolder -> Capacitor_SMD:C_0603_1608Metric; Manufacturer Taiyo Yuden -> TDK; Manufacturer_No UMK107BJ105KA-T -> C1608X8L1C105K080AC
- J1: renamed from J2; footprint Connector_PinHeader_2.00mm:PinHeader_1x04_P2.00mm_Horizontal -> Connector_JST:JST_PH_S4B-PH-SM4-TB_1x04-1MP_P2.00mm_Horizontal; Manufacturer Wurth -> JST; Manufacturer_No 61300411121 -> S4B-PH-SM4-TB(LF)(SN)
- J2: renamed from J1; footprint Connector_PinHeader_2.00mm:PinHeader_1x04_P2.00mm_Horizontal -> Connector_JST:JST_PH_S4B-PH-SM4-TB_1x04-1MP_P2.00mm_Horizontal; Manufacturer Wurth -> JST; Manufacturer_No 61300411121 -> S4B-PH-SM4-TB(LF)(SN)
- J3: renamed from J4; footprint Connector_PinHeader_2.00mm:PinHeader_1x04_P2.00mm_Horizontal -> Connector_FFC-FPC:Molex_200528-0040_1x04-1MP_P1.00mm_Horizontal; Manufacturer Wurth -> Molex; Manufacturer_No 61300411121 -> 200528-0040
- R1, R2, R3, R4: footprint Resistor_SMD:R_0603_1608Metric_Pad1.05x0.95mm_HandSolder -> Resistor_SMD:R_0603_1608Metric
- R5, R6: Manufacturer (none) -> Vishay Dale; Manufacturer_No (none) -> CRCW06034K70FKEAC
- SW83: renamed from SW91; Manufacturer CK -> C&K; Manufacturer_No KMR223NGULCLFG -> KMR221GLFS
- renumbered SW92 to SW84
Connections:
- net labels added: PWM
- net labels removed: AUX
- wire segments 83 -> 99
- no-connect marks 0 -> 2
Other:
- note added: "Only in standalone Keyboard"
