File: reform2-keyboard-pcb/reform-kbd-mcu.sch (KiCad schematic (older format))
At the start: 30 parts, among them J1 USB, J2 UART, J3 AUX, J4 USB_C_Receptacle_USB2.0, SW83 RESET, SW84 SW_DIP_x01, U1 ATMEGA32U4-AU, Y1 16MHz

Commit message: reform2-keyboard: version 2d5; add info badge; finalize connector positions; add optional 3v3 regulator for standalone
Parts:
- added C11, C12: 1uF, Capacitor_SMD:C_0603_1608Metric, symbol Device:C_Small
- added U3: MCP1700-3302E_SOT23, Package_TO_SOT_SMD:SOT-23, symbol Regulator_Linear:MCP1700-3302E_SOT23
- J4: Flags (none) -> DNP
- R13, R14: Flags (none) -> DNP; Manufacturer Yageo -> Panasonic; Manufacturer_No AC0603FR-135K1L -> ERJ-3EKF5101V
- R3: Manufacturer_No AF0603JR-0710KL -> RC0603FR-0710KL
- R5, R6: Manufacturer Vishay Dale -> Yageo; Manufacturer_No CRCW06034K70FKEAC -> RC0603FR-074K7L
- SW84: Manufacturer Omron -> Apem; Manufacturer_No A6S-1101-H -> DM01
- U1: symbol MCU_Microchip_ATmega:ATmega32U4-AU -> reform2-keyboard-rescue:ATmega32U4-AU-MCU_Microchip_ATmega
- Y1: footprint Crystals:Crystal_SMD_3225-4pin_3.2x2.5mm_HandSoldering -> Crystal:Crystal_SMD_3225-4Pin_3.2x2.5mm
Connections:
- wire segments 99 -> 111
Changed lines of the file:
@@
 Sheet 2 3
 Title "MNT Reform 2 Keyboard"
-Date "2020-04-12"
-Rev "2.0D-4"
+Date "2020-07-16"
+Rev "2.0D-5"
 Comp "Copyright 2017-2020 MNT Research GmbH"
 Comment1 "https://mntre.com"
@@
 F 3 "" H 3400 2800 50  0001 C CNN
 F 4 "Yageo" H 3400 2800 50  0001 C CNN "Manufacturer"
-F 5 "AF0603JR-0710KL" H 3400 2800 50  0001 C CNN "Manufacturer_No"
+F 5 "RC0603FR-0710KL" H 3400 2800 50  0001 C CNN "Manufacturer_No"
 	1    3400 2800
 	1    0    0    -1
@@
 F 0 "Y1" H 2475 3750 50  0000 L CNN
 F 1 "16MHz" H 2475 3675 50  0000 L CNN
-F 2 "Crystals:Crystal_SMD_3225-4pin_3.2x2.5mm_HandSoldering" H 2350 3550 50  0001 C CNN
+F 2 "Crystal:Crystal_SMD_3225-4Pin_3.2x2.5mm" H 2350 3550 50  0001 C CNN
 F 3 "" H 2350 3550 50  0001 C CNN
 F 4 "Abracon" H 2350 3550 50  0001 C CNN "Manufacturer"
@@
 	4100 6450 4100 6550
 $Comp
-L MCU_Microchip_ATmega:ATmega32U4-AU U1
+L reform2-keyboard-rescue:ATmega32U4-AU-MCU_Microchip_ATmega U1
 U 1 1 5A21306C
 P 4200 4650
+AR Path="/5A21306C" Ref="U1"  Part="1"
+AR Path="/5A2069AE/5A21306C" Ref="U1"  Part="1"
 F 0 "U1" H 4450 2900 50  0000 C CNN
 F 1 "ATMEGA32U4-AU" H 4700 2800 50  0000 C CNN
@@
 F 2 "Button_Switch_SMD:SW_DIP_SPSTx01_Slide_Omron_A6S-110x_W8.9mm_P2.54mm" H 1750 2200 50  0001 C CNN
 F 3 "~" H 1750 2200 50  0001 C CNN
-F 4 "Omron" H 1750 2200 50  0001 C CNN "Manufacturer"
-F 5 "A6S-1101-H" H 1750 2200 50  0001 C CNN "Manufacturer_No"
+F 4 "Apem" H 1750 2200 50  0001 C CNN "Manufacturer"
+F 5 "DM01" H 1750 2200 50  0001 C CNN "Manufacturer_No"
 	1    1750 2200
 	1    0    0    -1
@@
 F 2 "Resistor_SMD:R_0603_1608Metric" H 6400 3850 50  0001 C CNN
 F 3 "~" H 6400 3850 50  0001 C CNN
-F 4 "Vishay Dale" H 6400 3850 50  0001 C CNN "Manufacturer"
-F 5 "CRCW06034K70FKEAC" H 6400 3850 50  0001 C CNN "Manufacturer_No"
+F 4 "Yageo" H 6400 3850 50  0001 C CNN "Manufacturer"
+F 5 "RC0603FR-074K7L" H 6400 3850 50  0001 C CNN "Manufacturer_No"
 	1    6400 3850
 	1    0    0    -1
@@
 F 2 "Resistor_SMD:R_0603_1608Metric" H 6700 3850 50  0001 C CNN
 F 3 "~" H 6700 3850 50  0001 C CNN
-F 4 "Vishay Dale" H 6700 3850 50  0001 C CNN "Manufacturer"
-F 5 "CRCW06034K70FKEAC" H 6700 3850 50  0001 C CNN "Manufacturer_No"
+F 4 "Yageo" H 6700 3850 50  0001 C CNN "Manufacturer"
+F 5 "RC0603FR-074K7L" H 6700 3850 50  0001 C CNN "Manufacturer_No"
 	1    6700 3850
 	1    0    0    -1
@@
 F 4 "12401610E4#2A" H 7900 3050 50  0001 C CNN "Manufacturer_No"
 F 5 "Amphenol" H 7900 3050 50  0001 C CNN "Manufacturer"
+F 6 "DNP" H 7900 3050 50  0001 C CNN "Flags"
 	1    7900 3050
 	1    0    0    -1
@@
 F 2 "Resistor_SMD:R_0603_1608Metric" H 9050 2650 50  0001 C CNN
 F 3 "~" H 9050 2650 50  0001 C CNN
-F 4 "Yageo" H 9050 2650 50  0001 C CNN "Manufacturer"
-F 5 "AC0603FR-135K1L" H 9050 2650 50  0001 C CNN "Manufacturer_No"
+F 4 "Panasonic" H 9050 2650 50  0001 C CNN "Manufacturer"
+F 5 "ERJ-3EKF5101V" H 9050 2650 50  0001 C CNN "Manufacturer_No"
+F 6 "DNP" H 9050 2650 50  0001 C CNN "Flags"
 	1    9050 2650
 	0    1    1    0
@@
 F 2 "Resistor_SMD:R_0603_1608Metric" H 9300 2750 50  0001 C CNN
 F 3 "~" H 9300 2750 50  0001 C CNN
-F 4 "Yageo" H 9300 2750 50  0001 C CNN "Manufacturer"
-F 5 "AC0603FR-135K1L" H 9300 2750 50  0001 C CNN "Manufacturer_No"
+F 4 "Panasonic" H 9300 2750 50  0001 C CNN "Manufacturer"
+F 5 "ERJ-3EKF5101V" H 9300 2750 50  0001 C CNN "Manufacturer_No"
+F 6 "DNP" H 9300 2750 50  0001 C CNN "Flags"
 	1    9300 2750
 	0    -1   -1   0
@@
 Text Notes 7900 2050 0    60   ~ 0
 Only in standalone Keyboard
+$Comp
+L Regulator_Linear:MCP1700-3302E_SOT23 U3
+U 1 1 5F214B98
+P 9650 3800
+F 0 "U3" H 9650 4042 50  0000 C CNN
+F 1 "MCP1700-3302E_SOT23" H 9650 3951 50  0000 C CNN
+F 2 "Package_TO_SOT_SMD:SOT-23" H 9650 4025 50  0001 C CNN
+F 3 "http://ww1.microchip.com/downloads/en/DeviceDoc/20001826D.pdf" H 9650 3800 50  0001 C CNN
+F 4 "Microchip" H 9650 3800 50  0001 C CNN "Manufacturer"
+F 5 "MCP1700T-3302E/TT" H 9650 3800 50  0001 C CNN "Manufacturer_No"
+F 6 "DNP" H 9650 3800 50  0001 C CNN "Flags"
+	1    9650 3800
+	1    0    0    -1
+$EndComp
+$Comp
+L power:+5V #PWR0102
+U 1 1 5F215B65
+P 9100 3750
+F 0 "#PWR0102" H 9100 3600 50  0001 C CNN
+F 1 "+5V" H 9100 3890 50  0000 C CNN
+F 2 "" H 9100 3750 50  0001 C CNN
+F 3 "" H 9100 3750 50  0001 C CNN
+	1    9100 3750
+	1    0    0    -1
+$EndComp
+Wire Wire Line
+	9100 3750 9100 3800
+Wire Wire Line
+	9100 3800 9350 3800
+$Comp
+L power:GND #PWR0103
+U 1 1 5F2187C9
+P 9650 4200
+F 0 "#PWR0103" H 9650 3950 50  0001 C CNN
+F 1 "GND" H 9655 4027 50  0000 C CNN
+F 2 "" H 9650 4200 50  0001 C CNN
+F 3 "" H 9650 4200 50  0001 C CNN
+	1    9650 4200
+	1    0    0    -1
+$EndComp
+$Comp
+L power:+3V3 #PWR0104
+U 1 1 5F21B5B0
+P 10200 3750
+F 0 "#PWR0104" H 10200 3600 50  0001 C CNN
+F 1 "+3V3" H 10215 3923 50  0000 C CNN
+F 2 "" H 10200 3750 50  0001 C CNN
+F 3 "" H 10200 3750 50  0001 C CNN
+	1    10200 3750
+	1    0    0    -1
+$EndComp
+Wire Wire Line
+	10200 3750 10200 3800
+Wire Wire Line
+	10200 3800 9950 3800
+$Comp
+L Device:C_Small C11
+U 1 1 5F2226E4
+P 9100 3950
+F 0 "C11" H 9110 4020 50  0000 L CNN
+F 1 "1uF" H 9110 3870 50  0000 L CNN
+F 2 "Capacitor_SMD:C_0603_1608Metric" H 9100 3950 50  0001 C CNN
+F 3 "" H 9100 3950 50  0001 C CNN
+F 4 "TDK" H 9100 3950 50  0001 C CNN "Manufacturer"
+F 5 "C1608X8L1C105K080AC" H 9100 3950 50  0001 C CNN "Manufacturer_No"
+F 6 "DNP" H 9100 3950 50  0001 C CNN "Flags"
+	1    9100 3950
+	-1   0    0    -1
+$EndComp
+$Comp
+L Device:C_Small C12
+U 1 1 5F223065
+P 10200 3950
+F 0 "C12" H 10210 4020 50  0000 L CNN
+F 1 "1uF" H 10210 3870 50  0000 L CNN
+F 2 "Capacitor_SMD:C_0603_1608Metric" H 10200 3950 50  0001 C CNN
+F 3 "" H 10200 3950 50  0001 C CNN
+F 4 "TDK" H 10200 3950 50  0001 C CNN "Manufacturer"
+F 5 "C1608X8L1C105K080AC" H 10200 3950 50  0001 C CNN "Manufacturer_No"
+F 6 "DNP" H 10200 3950 50  0001 C CNN "Flags"
+	1    10200 3950
+	-1   0    0    -1
+$EndComp
+Wire Wire Line
+	10200 3850 10200 3800
+Connection ~ 10200 3800
+Wire Wire Line
+	9100 3800 9100 3850
+Connection ~ 9100 3800
+Wire Wire Line
+	9650 4100 9650 4150
+Wire Wire Line
+	9650 4150 9100 4150
+Wire Wire Line
+	9100 4150 9100 4050
+Connection ~ 9650 4150
+Wire Wire Line
+	9650 4150 9650 4200
+Wire Wire Line
+	9650 4150 10200 4150
+Wire Wire Line
+	10200 4150 10200 4050
 $EndSCHEMATC

Commit message: place left side
Parts:
- C1, C11, C12, C2, C3, C4, C5, C6: symbol Device:C_Small -> reform2-keyboard-rescue:C_Small-Device
- GFX1, GFX2: symbol Mechanical:MountingHole -> reform2-keyboard-rescue:MountingHole-Mechanical
- H1, H2, H3, H4, H5, H6: symbol Mechanical:MountingHole_Pad -> reform2-keyboard-rescue:MountingHole_Pad-Mechanical
- J4: symbol Connector:USB_C_Receptacle_USB2.0 -> reform2-keyboard-rescue:USB_C_Receptacle_USB2.0-Connector
- R1, R13, R14, R2, R3, R4, R5, R6: symbol Device:R_Small -> reform2-keyboard-rescue:R_Small-Device
- SW83: symbol Switch:SW_SPST -> reform2-keyboard-rescue:SW_SPST-Switch
- SW84: symbol Switch:SW_DIP_x01 -> reform2-keyboard-rescue:SW_DIP_x01-Switch
- U3: symbol Regulator_Linear:MCP1700-3302E_SOT23 -> reform2-keyboard-rescue:MCP1700-3302E_SOT23-Regulator_Linear
- Y1: symbol Device:Crystal_GND24 -> reform2-keyboard-rescue:Crystal_GND24-Device
Connections:
- net COL13: no longer names the net of U1.37 (PF6)
- net COL14 renamed RGB
- net ROW6: no longer names the net of U1.25 (PD4)
- no-connect marks 2 -> 4
Changed lines of the file:
@@
 $EndComp
 $Comp
-L Device:C_Small C1
+L reform2-keyboard-rescue:C_Small-Device C1
 U 1 1 5A2073AA
 P 2050 3850
+AR Path="/5A2073AA" Ref="C1"  Part="1"
+AR Path="/5A2069AE/5A2073AA" Ref="C1"  Part="1"
 F 0 "C1" H 2060 3920 50  0000 L CNN
 F 1 "18pF" H 2060 3770 50  0000 L CNN
@@
 $EndComp
 $Comp
-L Device:C_Small C2
+L reform2-keyboard-rescue:C_Small-Device C2
 U 1 1 5A2073F7
 P 2650 3850
+AR Path="/5A2073F7" Ref="C2"  Part="1"
+AR Path="/5A2069AE/5A2073F7" Ref="C2"  Part="1"
 F 0 "C2" H 2660 3920 50  0000 L CNN
 F 1 "18pF" H 2660 3770 50  0000 L CNN
@@
 $EndComp
 $Comp
-L Device:C_Small C3
+L reform2-keyboard-rescue:C_Small-Device C3
 U 1 1 5A20764E
 P 3450 4700
+AR Path="/5A20764E" Ref="C3"  Part="1"
+AR Path="/5A2069AE/5A20764E" Ref="C3"  Part="1"
 F 0 "C3" H 3460 4770 50  0000 L CNN
 F 1 "1uF" H 3460 4620 50  0000 L CNN
@@
 Text GLabel 4800 4950 2    60   Input ~ 0
 ROW5
-Text GLabel 4800 4750 2    60   Input ~ 0
-ROW6
 Text GLabel 4800 4850 2    60   Input ~ 0
 COL1
@@
 Text GLabel 4800 5850 2    60   Input ~ 0
 COL12
-Text GLabel 4800 5950 2    60   Input ~ 0
-COL13
-Text GLabel 4800 4050 2    60   Input ~ 0
-COL14
-$Comp
-L Device:R_Small R2
+$Comp
+L reform2-keyboard-rescue:R_Small-Device R2
 U 1 1 5A213EDF
 P 3150 4250
@@
 $EndComp
 $Comp
-L Device:R_Small R1
+L reform2-keyboard-rescue:R_Small-Device R1
 U 1 1 5A213F64
 P 3150 4150
@@
 $EndComp
 $Comp
-L Device:C_Small C5
+L reform2-keyboard-rescue:C_Small-Device C5
 U 1 1 5A2148C0
 P 4800 2400
+AR Path="/5A2148C0" Ref="C5"  Part="1"
+AR Path="/5A2069AE/5A2148C0" Ref="C5"  Part="1"
 F 0 "C5" H 4810 2470 50  0000 L CNN
 F 1 "1uF" H 4810 2320 50  0000 L CNN
@@
 $EndComp
 $Comp
-L Device:C_Small C4
+L reform2-keyboard-rescue:C_Small-Device C4
 U 1 1 5A214A09
 P 3800 2400
+AR Path="/5A214A09" Ref="C4"  Part="1"
+AR Path="/5A2069AE/5A214A09" Ref="C4"  Part="1"
 F 0 "C4" H 3810 2470 50  0000 L CNN
 F 1 "0.1uF" H 3810 2320 50  0000 L CNN
@@
 $EndComp
 $Comp
-L Device:R_Small R3
+L reform2-keyboard-rescue:R_Small-Device R3
 U 1 1 5A21443A
 P 3400 2800
@@
 $EndComp
 $Comp
-L Device:Crystal_GND24 Y1
+L reform2-keyboard-rescue:Crystal_GND24-Device Y1
 U 1 1 5A6378F6
 P 2350 3550
+AR Path="/5A6378F6" Ref="Y1"  Part="1"
+AR Path="/5A2069AE/5A6378F6" Ref="Y1"  Part="1"
 F 0 "Y1" H 2475 3750 50  0000 L CNN
 F 1 "16MHz" H 2475 3675 50  0000 L CNN
@@
 PROG
 $Comp
-L Switch:SW_SPST SW83
+L reform2-keyboard-rescue:SW_SPST-Switch SW83
 U 1 1 5CF3DA9E
 P 1750 1600
@@
 	2050 1600 1950 1600
 $Comp
-L Switch:SW_DIP_x01 SW84
+L reform2-keyboard-rescue:SW_DIP_x01-Switch SW84
 U 1 1 5CF54073
 P 1750 2200
@@
 	1400 2200 1450 2200
 $Comp
-L Device:R_Small R4
+L reform2-keyboard-rescue:R_Small-Device R4
 U 1 1 5CF5B5C6
 P 3500 3750
@@
 UART_RX
 $Comp
-L Mechanical:MountingHole_Pad H1
+L reform2-keyboard-rescue:MountingHole_Pad-Mechanical H1
 U 1 1 5CFAB6F9
 P 2750 7100
@@
 $EndComp
 $Comp
-L Mechanical:MountingHole_Pad H2
+L reform2-keyboard-rescue:MountingHole_Pad-Mechanical H2
 U 1 1 5CFABDD2
 P 3100 7100
@@
 $EndComp
 $Comp
-L Mechanical:MountingHole_Pad H3
+L reform2-keyboard-rescue:MountingHole_Pad-Mechanical H3
 U 1 1 5CFAC2C0
 P 3450 7100
@@
 $EndComp
 $Comp
-L Mechanical:MountingHole_Pad H4
+L reform2-keyboard-rescue:MountingHole_Pad-Mechanical H4
 U 1 1 5CFAC2CA
 P 3800 7100
@@
 	3450 7200 3800 7200
 $Comp
-L Mechanical:MountingHole GFX1
+L reform2-keyboard-rescue:MountingHole-Mechanical GFX1
 U 1 1 5CFBB66E
 P 5100 7100
@@
 $EndComp
 $Comp
-L Mechanical:MountingHole GFX2
+L reform2-keyboard-rescue:MountingHole-Mechanical GFX2
 U 1 1 5CFBBDCD
 P 5600 7100
@@
 	4200 2500 4200 2850
 $Comp
-L Device:C_Small C6
+L reform2-keyboard-rescue:C_Small-Device C6
 U 1 1 5DC43CAF
 P 5050 2400
+AR Path="/5DC43CAF" Ref="C6"  Part="1"
+AR Path="/5A2069AE/5DC43CAF" Ref="C6"  Part="1"
 F 0 "C6" H 5060 2470 50  0000 L CNN
 F 1 "0.1uF" H 5100 2300 50  0000 L CNN
@@
 DISP_SDA
 $Comp
-L Device:R_Small R5
+L reform2-keyboard-rescue:R_Small-Device R5
 U 1 1 5DCCE912
 P 6400 3850
@@
 $EndComp
 $Comp
-L Device:R_Small R6
+L reform2-keyboard-rescue:R_Small-Device R6
 U 1 1 5DCD0C98
 P 6700 3850
@@
 To SSD1306
 $Comp
-L Mechanical:MountingHole_Pad H5
+L reform2-keyboard-rescue:MountingHole_Pad-Mechanical H5
 U 1 1 5DC7F0C0
 P 4200 7100
@@
 $EndComp
 $Comp
-L Mechanical:MountingHole_Pad H6
+L reform2-keyboard-rescue:MountingHole_Pad-Mechanical H6
 U 1 1 5DC7F6F1
 P 4600 7100
@@
 	3400 2550 3400 2700
 $Comp
-L Connector:USB_C_Receptacle_USB2.0 J4
+L reform2-keyboard-rescue:USB_C_Receptacle_USB2.0-Connector J4
 U 1 1 5E62B709
 P 7900 3050
+AR Path="/5E62B709" Ref="J4"  Part="1"
+AR Path="/5A2069AE/5E62B709" Ref="J4"  Part="1"
 F 0 "J4" H 8007 3917 50  0000 C CNN
 F 1 "USB_C_Receptacle_USB2.0" H 8007 3826 50  0000 C CNN
@@
 	8650 3250 8500 3250
 $Comp
-L Device:R_Small R13
+L reform2-keyboard-rescue:R_Small-Device R13
 U 1 1 5E63CB6C
 P 9050 2650
@@
 $EndComp
 $Comp
-L Device:R_Small R14
+L reform2-keyboard-rescue:R_Small-Device R14
 U 1 1 5E63CE03
 P 9300 2750
@@
 Only in standalone Keyboard
 $Comp
-L Regulator_Linear:MCP1700-3302E_SOT23 U3
+L reform2-keyboard-rescue:MCP1700-3302E_SOT23-Regulator_Linear U3
 U 1 1 5F214B98
 P 9650 3800
@@
 	10200 3800 9950 3800
 $Comp
-L Device:C_Small C11
+L reform2-keyboard-rescue:C_Small-Device C11
 U 1 1 5F2226E4
 P 9100 3950
+AR Path="/5F2226E4" Ref="C11"  Part="1"
+AR Path="/5A2069AE/5F2226E4" Ref="C11"  Part="1"
 F 0 "C11" H 9110 4020 50  0000 L CNN
 F 1 "1uF" H 9110 3870 50  0000 L CNN
@@
 $EndComp
 $Comp
-L Device:C_Small C12
+L reform2-keyboard-rescue:C_Small-Device C12
 U 1 1 5F223065
 P 10200 3950
+AR Path="/5F223065" Ref="C12"  Part="1"
+AR Path="/5A2069AE/5F223065" Ref="C12"  Part="1"
 F 0 "C12" H 10210 4020 50  0000 L CNN
 F 1 "1uF" H 10210 3870 50  0000 L CNN
@@
 Wire Wire Line
 	10200 4150 10200 4050
+Text GLabel 4800 4050 2    60   Input ~ 0
+RGB
+NoConn ~ 4800 4750
+NoConn ~ 4800 5950
 $EndSCHEMATC
