File: reform2-keyboard-pcb/reform2-keyboard-backlight.sch (KiCad schematic (older format))
At the start: 93 parts, among them U2 TPS61185

Commit message: reform2-keyboard: version 2d5; add info badge; finalize connector positions; add optional 3v3 regulator for standalone
Parts:
- R11: Manufacturer Panasonic -> Yageo; Manufacturer_No ERJ-3EKF1004V -> RC0603FR-071ML
- U2: Manufacturer_No TPS61185 -> TPS61185RGET
Changed lines of the file:
@@
 Sheet 3 3
 Title "MNT Reform 2 Keyboard"
-Date "2020-04-12"
-Rev "2.0D-4"
+Date "2020-07-16"
+Rev "2.0D-5"
 Comp "Copyright 2017-2020 MNT Research GmbH"
 Comment1 "https://mntre.com"
@@
 F 3 "" H 4350 3700 60  0001 C CNN
 F 4 "Texas Instruments" H 4350 3700 50  0001 C CNN "Manufacturer"
-F 5 "TPS61185" H 4350 3700 50  0001 C CNN "Manufacturer_No"
+F 5 "TPS61185RGET" H 4350 3700 50  0001 C CNN "Manufacturer_No"
 	1    4350 3700
 	1    0    0    -1
@@
 F 2 "Resistor_SMD:R_0603_1608Metric" H 5700 1850 50  0001 C CNN
 F 3 "~" H 5700 1850 50  0001 C CNN
-F 4 "Panasonic" H 5700 1850 50  0001 C CNN "Manufacturer"
-F 5 "ERJ-3EKF1004V" H 5700 1850 50  0001 C CNN "Manufacturer_No"
+F 4 "Yageo" H 5700 1850 50  0001 C CNN "Manufacturer"
+F 5 "RC0603FR-071ML" H 5700 1850 50  0001 C CNN "Manufacturer_No"
 	1    5700 1850
 	1    0    0    -1

Commit message: place left side
Parts:
- removed D154, D155, D156, D157, D158, D159, D160, D161, D162, D163: WLED, LED_SMD:LED_0603_1608Metric, symbol Device:LED_Small
- C10, C7, C8, C9: symbol Device:C_Small -> reform2-keyboard-rescue:C_Small-Device
- D100, D101, D102, D103, D104, D105, D106, D107, D108, D109, D110, D111, D112, D113, D114, D115, D116, D117, D118, D119, D120, D121, D122, D123, D124, D125, D126, D127, D128, D129, D130, D131, D132, D133, D134, D135, D136, D137, D138, D139, D140, D141, D142, D143, D144, D145, D146, D147, D148, D149, D150, D151, D152, D153, D84, D85, D86, D87, D88, D89, D90, D91, D92, D93, D94, D95, D96, D97, D98, D99: symbol Device:LED_Small -> reform2-keyboard-rescue:LED_Small-Device
- D83: symbol Device:D_Schottky_Small -> reform2-keyboard-rescue:D_Schottky_Small-Device
- L1: symbol Device:L_Small -> reform2-keyboard-rescue:L_Small-Device
- R10, R11, R12, R7, R8, R9: symbol Device:R_Small -> reform2-keyboard-rescue:R_Small-Device
Connections:
- no-connect marks 2 -> 3

Commit message: first pass layout & routing
Parts:
- removed D124, D125, D126, D127, D128, D129, D130, D131, D132, D133: WLED, LED_SMD:LED_0603_1608Metric, symbol reform2-keyboard-rescue:LED_Small-Device
Connections:
- no-connect marks 3 -> 4
Changed lines of the file:
@@
-	0    -1   -1   0
-$EndComp
-Wire Wire Line
-	7850 1700 7850 1650
-$Comp
-L reform2-keyboard-rescue:LED_Small-Device D126
-U 1 1 5E69CF48
-P 7850 2200
-F 0 "D126" V 7896 2132 50  0000 R CNN
-F 1 "WLED" V 7805 2132 50  0000 R CNN
-F 2 "LED_SMD:LED_0603_1608Metric" V 7850 2200 50  0001 C CNN
-F 3 "~" V 7850 2200 50  0001 C CNN
-F 4 "OSRAM" H 7850 2200 50  0001 C CNN "Manufacturer"
-F 5 "LW Q38E-Q2OO-3K5L" H 7850 2200 50  0001 C CNN "Manufacturer_No"
-	1    7850 2200
-	0    -1   -1   0
-$EndComp
-$Comp
-L reform2-keyboard-rescue:LED_Small-Device D127
-U 1 1 5E69CF52
-P 7850 2400
-F 0 "D127" V 7896 2332 50  0000 R CNN
-F 1 "WLED" V 7805 2332 50  0000 R CNN
-F 2 "LED_SMD:LED_0603_1608Metric" V 7850 2400 50  0001 C CNN
-F 3 "~" V 7850 2400 50  0001 C CNN
-F 4 "OSRAM" H 7850 2400 50  0001 C CNN "Manufacturer"
-F 5 "LW Q38E-Q2OO-3K5L" H 7850 2400 50  0001 C CNN "Manufacturer_No"
-	1    7850 2400
-	0    -1   -1   0
-$EndComp
-$Comp
-L reform2-keyboard-rescue:LED_Small-Device D128
-U 1 1 5E69CF5C
-P 7850 2600
-F 0 "D128" V 7896 2532 50  0000 R CNN
-F 1 "WLED" V 7805 2532 50  0000 R CNN
-F 2 "LED_SMD:LED_0603_1608Metric" V 7850 2600 50  0001 C CNN
-F 3 "~" V 7850 2600 50  0001 C CNN
-F 4 "OSRAM" H 7850 2600 50  0001 C CNN "Manufacturer"
-F 5 "LW Q38E-Q2OO-3K5L" H 7850 2600 50  0001 C CNN "Manufacturer_No"
-	1    7850 2600
-	0    -1   -1   0
-$EndComp
-$Comp
-L reform2-keyboard-rescue:LED_Small-Device D129
-U 1 1 5E69CF66
-P 7850 2800
-F 0 "D129" V 7896 2732 50  0000 R CNN
-F 1 "WLED" V 7805 2732 50  0000 R CNN
-F 2 "LED_SMD:LED_0603_1608Metric" V 7850 2800 50  0001 C CNN
-F 3 "~" V 7850 2800 50  0001 C CNN
-F 4 "OSRAM" H 7850 2800 50  0001 C CNN "Manufacturer"
-F 5 "LW Q38E-Q2OO-3K5L" H 7850 2800 50  0001 C CNN "Manufacturer_No"
-	1    7850 2800
-	0    -1   -1   0
-$EndComp
-$Comp
-L reform2-keyboard-rescue:LED_Small-Device D130
-U 1 1 5E69CF70
-P 7850 3000
-F 0 "D130" V 7896 2932 50  0000 R CNN
-F 1 "WLED" V 7805 2932 50  0000 R CNN
-F 2 "LED_SMD:LED_0603_1608Metric" V 7850 3000 50  0001 C CNN
-F 3 "~" V 7850 3000 50  0001 C CNN
-F 4 "OSRAM" H 7850 3000 50  0001 C CNN "Manufacturer"
-F 5 "LW Q38E-Q2OO-3K5L" H 7850 3000 50  0001 C CNN "Manufacturer_No"
-	1    7850 3000
-	0    -1   -1   0
-$EndComp
-$Comp
-L reform2-keyboard-rescue:LED_Small-Device D131
-U 1 1 5E69CF7A
-P 7850 3200
-F 0 "D131" V 7896 3132 50  0000 R CNN
-F 1 "WLED" V 7805 3132 50  0000 R CNN
-F 2 "LED_SMD:LED_0603_1608Metric" V 7850 3200 50  0001 C CNN
-F 3 "~" V 7850 3200 50  0001 C CNN
-F 4 "OSRAM" H 7850 3200 50  0001 C CNN "Manufacturer"
-F 5 "LW Q38E-Q2OO-3K5L" H 7850 3200 50  0001 C CNN "Manufacturer_No"
-	1    7850 3200
 	0    -1   -1   0
 $EndComp
@@
 	7050 1650 7450 1650
 Connection ~ 7450 1650
-Wire Wire Line
-	7450 1650 7850 1650
-Connection ~ 7850 1650
-Wire Wire Line
-	7850 1650 8250 1650
 Connection ~ 8250 1650
 Wire Wire Line
@@
 Wire Wire Line
 	7450 3700 7450 4250
-Wire Wire Line
-	7850 3700 7850 4400
 Wire Wire Line
 	8250 3700 8250 4550
@@
 $EndComp
 $Comp
-L reform2-keyboard-rescue:LED_Small-Device D132
-U 1 1 5E819D55
-P 7850 3400
-F 0 "D132" V 7896 3332 50  0000 R CNN
-F 1 "WLED" V 7805 3332 50  0000 R CNN
-F 2 "LED_SMD:LED_0603_1608Metric" V 7850 3400 50  0001 C CNN
-F 3 "~" V 7850 3400 50  0001 C CNN
-F 4 "OSRAM" H 7850 3400 50  0001 C CNN "Manufacturer"
-F 5 "LW Q38E-Q2OO-3K5L" H 7850 3400 50  0001 C CNN "Manufacturer_No"
-	1    7850 3400
-	0    -1   -1   0
-$EndComp
-$Comp
-L reform2-keyboard-rescue:LED_Small-Device D133
-U 1 1 5E819D5F
-P 7850 3600
-F 0 "D133" V 7896 3532 50  0000 R CNN
-F 1 "WLED" V 7805 3532 50  0000 R CNN
-F 2 "LED_SMD:LED_0603_1608Metric" V 7850 3600 50  0001 C CNN
-F 3 "~" V 7850 3600 50  0001 C CNN
-F 4 "OSRAM" H 7850 3600 50  0001 C CNN "Manufacturer"
-F 5 "LW Q38E-Q2OO-3K5L" H 7850 3600 50  0001 C CNN "Manufacturer_No"
-	1    7850 3600
-	0    -1   -1   0
-$EndComp
-$Comp
 L reform2-keyboard-rescue:LED_Small-Device D142
 U 1 1 5E819D69
@@
 	8650 3700 8650 4700
 $Comp
-L reform2-keyboard-rescue:LED_Small-Device D125
-U 1 1 5E69CF3E
-P 7850 2000
-F 0 "D125" V 7896 1932 50  0000 R CNN
-F 1 "WLED" V 7805 1932 50  0000 R CNN
-F 2 "LED_SMD:LED_0603_1608Metric" V 7850 2000 50  0001 C CNN
-F 3 "~" V 7850 2000 50  0001 C CNN
-F 4 "OSRAM" H 7850 2000 50  0001 C CNN "Manufacturer"
-F 5 "LW Q38E-Q2OO-3K5L" H 7850 2000 50  0001 C CNN "Manufacturer_No"
-	1    7850 2000
-	0    -1   -1   0
-$EndComp
-$Comp
-L reform2-keyboard-rescue:LED_Small-Device D124
-U 1 1 5E69CF33
-P 7850 1800
-F 0 "D124" V 7896 1732 50  0000 R CNN
-F 1 "WLED" V 7805 1732 50  0000 R CNN
-F 2 "LED_SMD:LED_0603_1608Metric" V 7850 1800 50  0001 C CNN
-F 3 "~" V 7850 1800 50  0001 C CNN
-F 4 "OSRAM" H 7850 1800 50  0001 C CNN "Manufacturer"
-F 5 "LW Q38E-Q2OO-3K5L" H 7850 1800 50  0001 C CNN "Manufacturer_No"
-	1    7850 1800
-	0    -1   -1   0
-$EndComp
-$Comp
 L reform2-keyboard-rescue:LED_Small-Device D97
 U 1 1 5E69363F
@@
 Wire Wire Line
 	5000 4550 8250 4550
-Wire Wire Line
-	7850 4400 5000 4400
 Wire Wire Line
 	5000 4250 7450 4250
@@
 	1    0    0    -1
 $EndComp
+Wire Wire Line
+	7450 1650 8250 1650
+NoConn ~ 5000 4400
 $EndSCHEMATC
